Commit message: Fixed transform issue with hand cameras

File: spot_description/urdf/arm/spot_arm.urdf.xacro (robot description, xacro)
@@ -147,4 +147,10 @@
         <limit effort="1000" velocity="1000.00" lower="-1.57" upper="0.0"/>
     </joint>
+    <link name="${name}.link_wr1"/>
+    <joint name="${name}_link_wr1_to_wrist" type = "fixed">
+        <parent link = "${name}_wrist_roll"/>
+        <child  link = "${name}.link_wr1"/>
+        <origin xyz = "0 0 0"/>
+    </joint>
     </xacro:macro>
 </robot>

Commit message: Migrated collision and transmission from manipulation driver

File: spot_description/urdf/arm/spot_arm.urdf.xacro (robot description, xacro)
@@ -13,4 +13,13 @@
         </material>
         </visual>
+        <collision>
+        <origin xyz="0 0 0" rpy="0 0 0"/>
+        <geometry>
+            <mesh filename="package://spot_description/meshes/arm/arm0.link_sh0.obj"/>
+        </geometry>
+        <material name="arm0.link_sh0">
+            <color rgba="1 0.2 0.2 1"/>
+        </material>
+        </collision>
     </link>
     <joint name="${name}_shoulder_yaw" type="revolute">
@@ -31,4 +40,13 @@
         </material>
         </visual>
+        <collision>
+        <origin xyz="0 0 0" rpy="0 0 0"/>
+        <geometry>
+            <mesh filename="package://spot_description/meshes/arm/arm0.link_sh1.obj"/>
+        </geometry>
+        <material name="arm0.link_sh1">
+            <color rgba="1 0.2 0.2 1"/>
+        </material>
+        </collision>
     </link>
     <joint name="${name}_shoulder_pitch" type="revolute">
@@ -49,11 +67,20 @@
             </material>
         </visual>
-    </link>
-    <joint name="${name}_shoulder_roll" type="revolute">
+        <collision>
+        <origin xyz="0 0 0" rpy="0 0 0"/>
+        <geometry>
+            <mesh filename="package://spot_description/meshes/arm/arm0.link_hr0.obj"/>
+        </geometry>
+            <material name="arm0.link_hr0">
+            <color rgba="1 0.2 0.2 1"/>
+            </material>
+        </collision>
+    </link>
+    <joint name="${name}_shoulder_roll" type="fixed">
         <origin xyz="0.0 0.0 0.0" rpy="0 0 0"/>
         <axis xyz="1 0 0"/>
         <parent link="${name}_shoulder_pitch"/>
         <child link="${name}_shoulder_roll"/>
-        <limit effort="1000" velocity="1000.00" lower="-1e6" upper="1e6"/>
+	<limit effort="0" velocity="0" lower="0" upper="0"/>
     </joint>
     <link name="${name}_elbow_pitch">
@@ -67,4 +94,13 @@
             </material>
         </visual>
+        <collision>
+        <origin xyz="0 0 0" rpy="0 0 0"/>
+        <geometry>
+            <mesh filename="package://spot_description/meshes/arm/arm0.link_el0.obj"/>
+        </geometry>
+            <material name="arm0.link_el0">
+            <color rgba="1 0.2 0.2 1"/>
+            </material>
+        </collision>
     </link>
     <joint name="${name}_elbow_pitch" type="revolute">
@@ -85,4 +121,13 @@
             </material>
         </visual>
+        <collision>
+        <origin xyz="0 0 0" rpy="0 0 0"/>
+        <geometry>
+            <mesh filename="package://spot_description/meshes/arm/arm0.link_el1.obj"/>
+        </geometry>
+            <material name="arm0.link_el1">
+            <color rgba="1 0.2 0.2 1"/>
+            </material>
+        </collision>
     </link>
     <joint name="${name}_elbow_roll" type="revolute">
@@ -103,4 +148,13 @@
             </material>
         </visual>
+        <collision>
+        <origin xyz="0 0 0" rpy="0 0 0"/>
+        <geometry>
+            <mesh filename="package://spot_description/meshes/arm/arm0.link_wr0.obj"/>
+        </geometry>
+            <material name="arm0.link_wr0">
+            <color rgba="1 0.2 0.2 1"/>
+            </material>
+        </collision>
     </link>
     <joint name="${name}_wrist_pitch" type="revolute">
@@ -121,4 +175,13 @@
             </material>
         </visual>
+        <collision>
+        <origin xyz="0 0 0" rpy="0 0 0"/>
+        <geometry>
+            <mesh filename="package://spot_description/meshes/arm/arm0.link_wr1.obj"/>
+        </geometry>
+            <material name="arm0.link_wr1">
+            <color rgba="1 0.2 0.2 1"/>
+            </material>
+        </collision>
     </link>
     <joint name="${name}_wrist_roll" type="revolute">
@@ -139,4 +202,13 @@
         </material>
         </visual>
+        <collision>
+        <origin xyz="0 0 0" rpy="0 0 0"/>
+        <geometry>
+            <mesh filename="package://spot_description/meshes/arm/arm0.link_fngr.obj"/>
+        </geometry>
+        <material name="arm0.link_fngr">
+            <color rgba="0.2 0.2 0.2 1"/>
+        </material>
+        </collision>
     </link>
     <joint name="${name}_fingers" type="revolute">
@@ -154,3 +226,65 @@
     </joint>
     </xacro:macro>
+<!-- Transmissions -->
+  <transmission name="tran1">
+    <type>transmission_interface/SimpleTransmission</type>
+    <joint name="arm0_shoulder_yaw">
+      <hardwareInterface>hardware_interface/PositionJointInterface</hardwareInterface>
+    </joint>
+    <actuator name="motor1">
+      <hardwareInterface>hardware_interface/PositionJointInterface</hardwareInterface>
+      <mechanicalReduction>1</mechanicalReduction>
+    </actuator>
+  </transmission>
+  <transmission name="tran2">
+    <type>transmission_interface/SimpleTransmission</type>
+    <joint name="arm0_shoulder_pitch">
+      <hardwareInterface>hardware_interface/PositionJointInterface</hardwareInterface>
+    </joint>
+    <actuator name="motor2">
+      <hardwareInterface>hardware_interface/PositionJointInterface</hardwareInterface>
+      <mechanicalReduction>1</mechanicalReduction>
+    </actuator>
+  </transmission>
+  <transmission name="tran3">
+    <type>transmission_interface/SimpleTransmission</type>
+    <joint name="arm0_elbow_pitch">
+      <hardwareInterface>hardware_interface/PositionJointInterface</hardwareInterface>
+    </joint>
+    <actuator name="motor3">
+      <hardwareInterface>hardware_interface/PositionJointInterface</hardwareInterface>
+      <mechanicalReduction>1</mechanicalReduction>
+    </actuator>
+  </transmission>
+  <transmission name="tran4">
+    <type>transmission_interface/SimpleTransmission</type>
+    <joint name="arm0_elbow_roll">
+      <hardwareInterface>hardware_interface/PositionJointInterface</hardwareInterface>
+    </joint>
+    <actuator name="motor4">
+      <hardwareInterface>hardware_interface/PositionJointInterface</hardwareInterface>
+      <mechanicalReduction>1</mechanicalReduction>
+    </actuator>
+  </transmission>
+  <transmission name="tran5">
+    <type>transmission_interface/SimpleTransmission</type>
+    <joint name="arm0_wrist_pitch">
+      <hardwareInterface>hardware_interface/PositionJointInterface</hardwareInterface>
+    </joint>
+    <actuator name="motor5">
+      <hardwareInterface>hardware_interface/PositionJointInterface</hardwareInterface>
+      <mechanicalReduction>1</mechanicalReduction>
+    </actuator>
+  </transmission>
+  <transmission name="tran6">
+    <type>transmission_interface/SimpleTransmission</type>
+    <joint name="arm0_wrist_roll">
+      <hardwareInterface>hardware_interface/PositionJointInterface</hardwareInterface>
+    </joint>
+    <actuator name="motor6">
+      <hardwareInterface>hardware_interface/PositionJointInterface</hardwareInterface>
+      <mechanicalReduction>1</mechanicalReduction>
+    </actuator>
+  </transmission>
+<!-- EOF Transmissions -->
 </robot>

Commit message: Changed camera color frame source to urdf

File: spot_description/urdf/arm/spot_arm.urdf.xacro (robot description, xacro)
@@ -225,4 +225,10 @@
         <origin xyz = "0 0 0"/>
     </joint>
+    <link name="hand_color_image_sensor"/>
+    <joint name="color_image_joint" type="fixed">
+        <parent link = "${name}_wrist_roll"/>
+        <child  link = "hand_color_image_sensor"/>
+        <origin xyz  = "0.14 0.02 0.022" rpy="-1.57 0 -1.54"/>
+    </joint>
     </xacro:macro>
 <!-- Transmissions -->

Commit message: Added hand frame

File: spot_description/urdf/arm/spot_arm.urdf.xacro (robot description, xacro)
@@ -225,4 +225,10 @@
         <origin xyz = "0 0 0"/>
     </joint>
+    <link name="${name}_hand"/>
+    <joint nam="${name}_wrist_to_hand" type="fixed">
+        <parent link = "${name}_wrist_roll"/>
+        <child  link = "${name}_hand"/>
+        <origin xyz = "0.19557 0.0 0.0"/>
+    </joint>
     <link name="hand_color_image_sensor"/>
     <joint name="color_image_joint" type="fixed">

Commit message: Fixed typo in hand link

File: spot_description/urdf/arm/spot_arm.urdf.xacro (robot description, xacro)
@@ -226,5 +226,5 @@
     </joint>
     <link name="${name}_hand"/>
-    <joint nam="${name}_wrist_to_hand" type="fixed">
+    <joint name="${name}_wrist_to_hand" type="fixed">
         <parent link = "${name}_wrist_roll"/>
         <child  link = "${name}_hand"/>

Commit message: Fixed issues with hand camera

File: spot_description/urdf/arm/spot_arm.urdf.xacro (robot description, xacro)
@@ -235,5 +235,11 @@
         <parent link = "${name}_wrist_roll"/>
         <child  link = "hand_color_image_sensor"/>
-        <origin xyz  = "0.14 0.02 0.022" rpy="-1.57 0 -1.54"/>
+        <origin xyz  = "0.14 0.02 0.022" rpy="-1.42 0 -1.57"/>
+    </joint>
+    <link name="hand_depth_sensor"/>
+    <joint name="depth_sensor_joint" type="fixed">
+        <parent link = "${name}_wrist_roll"/>
+        <child  link = "hand_depth_sensor"/>
+        <origin xyz  = "0.14 0.0 0.01" rpy="0 1.42 0"/>
     </joint>
     </xacro:macro>

Commit message: remove superfluous wrist link

File: spot_description/urdf/arm/spot_arm.urdf.xacro (robot description, xacro)
@@ -219,10 +219,4 @@
         <limit effort="1000" velocity="1000.00" lower="-1.57" upper="0.0"/>
     </joint>
-    <link name="${name}.link_wr1"/>
-    <joint name="${name}_link_wr1_to_wrist" type = "fixed">
-        <parent link = "${name}_wrist_roll"/>
-        <child  link = "${name}.link_wr1"/>
-        <origin xyz = "0 0 0"/>
-    </joint>
     <link name="hand_color_image_sensor"/>
     <joint name="color_image_joint" type="fixed">

Commit message: add tool link and virtual ee joint

File: spot_description/urdf/arm/spot_arm.urdf.xacro (robot description, xacro)
@@ -192,4 +192,11 @@
         <limit effort="1000" velocity="1000.00" lower="-2.87979326579064354163" upper="2.87979326579064354163"/>
     </joint>
+    <link name="${name}_tool0"/>
+    <joint name="${name}_ee_virtual_joint" type="fixed">
+        <origin xyz="0.19557 0 0" rpy="0 0 0"/>
+        <axis xyz="0.0 0.0 0.0"/>
+        <parent link="${name}_wrist_roll"/>
+        <child link="${name}_tool0"/>
+    </joint>
     <link name="${name}_fingers">
         <visual>
