Commit message: spot_ros in catkin_ws on spot

File: spot_description/urdf/arm/spot_arm.urdf.xacro (robot description, xacro)
@@ -82,5 +82,5 @@
         <parent link="${name}_shoulder_pitch"/>
         <child link="${name}_shoulder_roll"/>
-	<limit effort="0" velocity="0" lower="0" upper="0"/>
+        <!--limit effort="1000" velocity="1000.00" lower="-1e6" upper="1e6"/-->
     </joint>
     <link name="${name}_elbow_pitch">
@@ -192,5 +192,6 @@
         <limit effort="1000" velocity="1000.00" lower="-2.87979326579064354163" upper="2.87979326579064354163"/>
     </joint>
-    <link name="${name}_tool0"/>
+    <link name="${name}_tool0">
+    </link>
     <joint name="${name}_ee_virtual_joint" type="fixed">
         <origin xyz="0.19557 0 0" rpy="0 0 0"/>
@@ -226,28 +227,4 @@
         <limit effort="1000" velocity="1000.00" lower="-1.57" upper="0.0"/>
     </joint>
-    <link name="${name}.link_wr1"/>
-    <joint name="${name}_link_wr1_to_wrist" type = "fixed">
-        <parent link = "${name}_wrist_roll"/>
-        <child  link = "${name}.link_wr1"/>
-        <origin xyz = "0 0 0"/>
-    </joint>
-    <link name="${name}_hand"/>
-    <joint name="${name}_wrist_to_hand" type="fixed">
-        <parent link = "${name}_wrist_roll"/>
-        <child  link = "${name}_hand"/>
-        <origin xyz = "0.19557 0.0 0.0"/>
-    </joint>
-    <link name="hand_color_image_sensor"/>
-    <joint name="color_image_joint" type="fixed">
-        <parent link = "${name}_wrist_roll"/>
-        <child  link = "hand_color_image_sensor"/>
-        <origin xyz  = "0.14 0.02 0.022" rpy="-1.42 0 -1.57"/>
-    </joint>
-    <link name="hand_depth_sensor"/>
-    <joint name="depth_sensor_joint" type="fixed">
-        <parent link = "${name}_wrist_roll"/>
-        <child  link = "hand_depth_sensor"/>
-        <origin xyz  = "0.14 0.0 0.01" rpy="0 1.42 0"/>
-    </joint>
     </xacro:macro>
 <!-- Transmissions -->

File: spot_description/urdf/spot.urdf.xacro (robot description, xacro)
@@ -4,7 +4,6 @@
          published by the driver (see spot_driver package) during runtime, so that the transforms
          include calibration adjustments. -->
-    <xacro:arg name="has_arm" default="False" />
-    <xacro:arg name="has_eap" default="False" />
-    <!-- Fixed links -->
+    <xacro:arg name="has_arm" default="true" />
+    <xacro:arg name="has_velodyne" default="false" />
     <link name="body">
         <visual>
@@ -18,8 +17,4 @@
             </geometry>
         </collision>
-        <inertial>
-             <mass value="16.25" />
-             <inertia  ixx="0.085" ixy="0.0"  ixz="0.0"  iyy="1.045"  iyz="0.0"  izz="1.042" />
-    	</inertial>
     </link>
     <link name="base_link"/>
@@ -41,5 +36,4 @@
         <child link="rear_rail" />
     </joint>
-    <!-- Front Left -->
     <link name="front_left_hip">
         <visual>
@@ -53,8 +47,4 @@
             </geometry>
         </collision>
-        <inertial>
-            <mass value="1.5" />
-    	    <inertia  ixx="0.0605" ixy="0.0"  ixz="0.0"  iyy="0.0"  iyz="0.0"  izz="0.0" />
-    	</inertial>
     </link>
     <joint name="front_left_hip_x" type="revolute">
@@ -63,17 +53,6 @@
         <parent link="body" />
         <child link="front_left_hip" />
-        <dynamics damping="0.1" friction="0.1"/>
         <limit effort="1000" velocity="1000.00" lower="-0.78539816339744827899" upper="0.78539816339744827899" />
     </joint>
-    <transmission name="front_left_hip_x_trans">
-	    <type>transmission_interface/SimpleTransmission</type>
-	    <joint name="front_left_hip_x">
-            <hardwareInterface>EffortJointInterface</hardwareInterface>
-        </joint>
-	    <actuator name="front_left_hip_x">
-          	<mechanicalReduction>50</mechanicalReduction>
-          	<hardwareInterface>EffortJointInterface</hardwareInterface>
-	    </actuator>
-    </transmission>
     <link name="front_left_upper_leg">
         <visual>
@@ -87,8 +66,4 @@
             </geometry>
         </collision>
-        <inertial>
-            <mass value="1.5" />
-    	    <inertia  ixx="0.0" ixy="0.0"  ixz="0.0"  iyy="0.05"  iyz="0.0"  izz="0.0" />
-    	</inertial>
     </link>
     <joint name="front_left_hip_y" type="revolute">
@@ -97,17 +72,6 @@
         <parent link="front_left_hip" />
         <child link="front_left_upper_leg" />
-        <dynamics damping="0.1" friction="0.1"/>
         <limit effort="1000" velocity="1000.00" lower="-0.89884456477707963539" upper="2.2951079663725435509" />
     </joint>
-    <transmission name="front_left_hip_y_trans">
-        <type>transmission_interface/SimpleTransmission</type>
-        <joint name="front_left_hip_y">
-            <hardwareInterface>EffortJointInterface</hardwareInterface>
-        </joint>
-        <actuator name="front_left_hip_y">
-            <mechanicalReduction>50</mechanicalReduction>
-            <hardwareInterface>EffortJointInterface</hardwareInterface>
-        </actuator>
-    </transmission>
     <link name="front_left_lower_leg">
         <visual>
@@ -121,8 +85,4 @@
             </geometry>
         </collision>
-        <inertial>
-            <mass value="1.0" />
-    	    <inertia  ixx="0.0" ixy="0.0"  ixz="0.0"  iyy="0.045"  iyz="0.0"  izz="0.0" />
-    	</inertial>
     </link>
     <joint name="front_left_knee" type="revolute">
@@ -131,30 +91,6 @@
         <parent link="front_left_upper_leg" />
         <child link="front_left_lower_leg" />
-        <dynamics damping="0.1" friction="0.1"/>
         <limit effort="1000" velocity="1000.00" lower="-2.7929" upper="-0.254801" />
     </joint>
-    <gazebo reference="front_left_lower_leg">
-        <sensor name="front_left_lower_leg_contactsensor_sensor" type="contact">
-        <always_on>true</always_on>
-        <contact>
-            <collision>front_left_lower_leg_fixed_joint_lump__front_bump_sensor_collision</collision>
-        </contact>
-        <plugin filename="libgazebo_ros_bumper.so" name="front_left_lower_leg_plugin">
-            <bumperTopicName>front_left_lower_leg_contact</bumperTopicName>
-            <frameName>front_left_lower_leg</frameName>
-        </plugin>
-        </sensor>
-    </gazebo>
-    <transmission name="front_left_knee_trans">
-	  <type>transmission_interface/SimpleTransmission</type>
-	  <joint name="front_left_knee">
-          	<hardwareInterface>EffortJointInterface</hardwareInterface>
-      </joint>
-	  <actuator name="front_left_knee">
-          	<mechanicalReduction>50</mechanicalReduction>
-          	<hardwareInterface>EffortJointInterface</hardwareInterface>
-	  </actuator>
-    </transmission>
-    <!-- Front Right -->
     <link name="front_right_hip">
         <visual>
@@ -168,8 +104,4 @@
             </geometry>
         </collision>
-        <inertial>
-            <mass value="1.5" />
-    	    <inertia  ixx="0.0605" ixy="0.0"  ixz="0.0"  iyy="0.0"  iyz="0.0"  izz="0.0" />
-    	</inertial>
     </link>
     <joint name="front_right_hip_x" type="revolute">
@@ -178,17 +110,6 @@
         <parent link="body" />
         <child link="front_right_hip" />
-        <dynamics damping="0.1" friction="0.1"/>
         <limit effort="1000" velocity="1000.00" lower="-0.78539816339744827899" upper="0.78539816339744827899" />
     </joint>
-    <transmission name="front_right_hip_x_trans">
-	  <type>transmission_interface/SimpleTransmission</type>
-	  <joint name="front_right_hip_x">
-          	<hardwareInterface>EffortJointInterface</hardwareInterface>
-      </joint>
-	  <actuator name="front_right_hip_x">
-          	<mechanicalReduction>50</mechanicalReduction>
-          	<hardwareInterface>EffortJointInterface</hardwareInterface>
-	  </actuator>
-    </transmission>
     <link name="front_right_upper_leg">
         <visual>
@@ -202,8 +123,4 @@
             </geometry>
         </collision>
-        <inertial>
-            <mass value="1.5" />
-    	    <inertia  ixx="0.0" ixy="0.0"  ixz="0.0"  iyy="0.05"  iyz="0.0"  izz="0.0" />
-    	</inertial>
     </link>
     <joint name="front_right_hip_y" type="revolute">
@@ -212,17 +129,6 @@
         <parent link="front_right_hip" />
         <child link="front_right_upper_leg" />
-        <dynamics damping="0.1" friction="0.1"/>
         <limit effort="1000" velocity="1000.00" lower="-0.89884456477707963539" upper="2.2951079663725435509" />
     </joint>
-    <transmission name="front_right_hip_y_trans">
-        <type>transmission_interface/SimpleTransmission</type>
-        <joint name="front_right_hip_y">
-            <hardwareInterface>EffortJointInterface</hardwareInterface>
-        </joint>
-        <actuator name="front_right_hip_y">
-            <mechanicalReduction>50</mechanicalReduction>
-            <hardwareInterface>EffortJointInterface</hardwareInterface>
-        </actuator>
-    </transmission>
     <link name="front_right_lower_leg">
         <visual>
@@ -236,8 +142,4 @@
             </geometry>
         </collision>
-        <inertial>
-            <mass value="1.0" />
-    	    <inertia  ixx="0.0" ixy="0.0"  ixz="0.0"  iyy="0.045"  iyz="0.0"  izz="0.0" />
-    	</inertial>
     </link>
     <joint name="front_right_knee" type="revolute">
@@ -246,30 +148,6 @@
         <parent link="front_right_upper_leg" />
         <child link="front_right_lower_leg" />
-        <dynamics damping="0.1" friction="0.1"/>
         <limit effort="1000" velocity="1000.00" lower="-2.7929" upper="-0.247563" />
     </joint>
-    <gazebo reference="front_right_lower_leg">
-        <sensor name="front_right_lower_leg_contactsensor_sensor" type="contact">
-        <always_on>true</always_on>
-        <contact>
-            <collision>front_right_lower_leg_fixed_joint_lump__front_bump_sensor_collision</collision>
-        </contact>
-        <plugin filename="libgazebo_ros_bumper.so" name="front_right_lower_leg_plugin">
-            <bumperTopicName>front_right_lower_leg_contact</bumperTopicName>
-            <frameName>front_right_lower_leg</frameName>
-        </plugin>
-        </sensor>
-    </gazebo>
-    <transmission name="front_right_knee_trans">
-        <type>transmission_interface/SimpleTransmission</type>
-        <joint name="front_right_knee">
-            <hardwareInterface>EffortJointInterface</hardwareInterface>
-        </joint>
-        <actuator name="front_right_knee">
-            <mechanicalReduction>50</mechanicalReduction>
-            <hardwareInterface>EffortJointInterface</hardwareInterface>
-        </actuator>
-    </transmission>
-    <!-- Rear Left -->
     <link name="rear_left_hip">
         <visual>
@@ -283,8 +161,4 @@
             </geometry>
         </collision>
-        <inertial>
-            <mass value="1.5" />
-    	    <inertia  ixx="0.0605" ixy="0.0"  ixz="0.0"  iyy="0.0"  iyz="0.0"  izz="0.0" />
-    	</inertial>
     </link>
     <joint name="rear_left_hip_x" type="revolute">
@@ -293,17 +167,6 @@
         <parent link="body" />
         <child link="rear_left_hip" />
-        <dynamics damping="0.1" friction="0.1"/>
         <limit effort="1000" velocity="1000.00" lower="-0.78539816339744827899" upper="0.78539816339744827899" />
     </joint>
-    <transmission name="rear_left_hip_x_trans">
-        <type>transmission_interface/SimpleTransmission</type>
-        <joint name="rear_left_hip_x">
-            <hardwareInterface>EffortJointInterface</hardwareInterface>
-        </joint>
-        <actuator name="rear_left_hip_x">
-            <mechanicalReduction>50</mechanicalReduction>
-            <hardwareInterface>EffortJointInterface</hardwareInterface>
-        </actuator>
-    </transmission>
     <link name="rear_left_upper_leg">
         <visual>
@@ -317,8 +180,4 @@
             </geometry>
         </collision>
-        <inertial>
-           <mass value="1.5" />
-    	   <inertia  ixx="0.0" ixy="0.0"  ixz="0.0"  iyy="0.05"  iyz="0.0"  izz="0.0" />
-    	</inertial>
     </link>
     <joint name="rear_left_hip_y" type="revolute">
@@ -327,17 +186,6 @@
         <parent link="rear_left_hip" />
         <child link="rear_left_upper_leg" />
-        <dynamics damping="0.1" friction="0.1"/>
         <limit effort="1000" velocity="1000.00" lower="-0.89884456477707963539" upper="2.2951079663725435509" />
     </joint>
-    <transmission name="rear_left_hip_y_trans">
-        <type>transmission_interface/SimpleTransmission</type>
-        <joint name="rear_left_hip_y">
-            <hardwareInterface>EffortJointInterface</hardwareInterface>
-        </joint>
-        <actuator name="rear_left_hip_y">
-            <mechanicalReduction>50</mechanicalReduction>
-            <hardwareInterface>EffortJointInterface</hardwareInterface>
-        </actuator>
-    </transmission>
     <link name="rear_left_lower_leg">
         <visual>
@@ -351,8 +199,4 @@
             </geometry>
         </collision>
-        <inertial>
-            <mass value="1.0" />
-    	    <inertia  ixx="0.0" ixy="0.0"  ixz="0.0"  iyy="0.045"  iyz="0.0"  izz="0.0" />
-    	</inertial>
     </link>
     <joint name="rear_left_knee" type="revolute">
@@ -361,30 +205,6 @@
         <parent link="rear_left_upper_leg" />
         <child link="rear_left_lower_leg" />
-        <dynamics damping="0.1" friction="0.1"/>
         <limit effort="1000" velocity="1000.00" lower="-2.7929" upper="-0.267153" />
     </joint>
-    <gazebo reference="rear_left_lower_leg">
-        <sensor name="rear_left_lower_leg_contactsensor_sensor" type="contact">
-        <always_on>true</always_on>
-        <contact>
-            <collision>rear_left_lower_leg_fixed_joint_lump__rear_bump_sensor_collision</collision>
-        </contact>
-        <plugin filename="libgazebo_ros_bumper.so" name="rear_left_lower_leg_plugin">
-            <bumperTopicName>rear_left_lower_leg_contact</bumperTopicName>
-            <frameName>rear_left_lower_leg</frameName>
-        </plugin>
-        </sensor>
-    </gazebo>
-    <transmission name="rear_left_knee_trans">
-        <type>transmission_interface/SimpleTransmission</type>
-        <joint name="rear_left_knee">
-             <hardwareInterface>EffortJointInterface</hardwareInterface>
-        </joint>
-        <actuator name="rear_left_knee">
-            <mechanicalReduction>50</mechanicalReduction>
-            <hardwareInterface>EffortJointInterface</hardwareInterface>
-        </actuator>
-    </transmission>
-    <!-- Rear Right -->
     <link name="rear_right_hip">
         <visual>
@@ -398,8 +218,4 @@
             </geometry>
         </collision>
-        <inertial>
-            <mass value="1.5" />
-    	    <inertia  ixx="0.0605" ixy="0.0"  ixz="0.0"  iyy="0.0"  iyz="0.0"  izz="0.0" />
-    	</inertial>
     </link>
     <joint name="rear_right_hip_x" type="revolute">
@@ -408,17 +224,6 @@
         <parent link="body" />
         <child link="rear_right_hip" />
-        <dynamics damping="0.1" friction="0.1"/>
         <limit effort="1000" velocity="1000.00" lower="-0.78539816339744827899" upper="0.78539816339744827899" />
     </joint>
-    <transmission name="rear_right_hip_x_trans">
-        <type>transmission_interface/SimpleTransmission</type>
-        <joint name="rear_right_hip_x">
-            <hardwareInterface>EffortJointInterface</hardwareInterface>
-        </joint>
-        <actuator name="rear_right_hip_x">
-            <mechanicalReduction>50</mechanicalReduction>
-            <hardwareInterface>EffortJointInterface</hardwareInterface>
-        </actuator>
-    </transmission>
     <link name="rear_right_upper_leg">
         <visual>
@@ -432,8 +237,4 @@
             </geometry>
         </collision>
-        <inertial>
-            <mass value="1.5" />
-    	    <inertia  ixx="0.0" ixy="0.0"  ixz="0.0"  iyy="0.05"  iyz="0.0"  izz="0.0" />
-    	</inertial>
     </link>
     <joint name="rear_right_hip_y" type="revolute">
@@ -442,17 +243,6 @@
         <parent link="rear_right_hip" />
         <child link="rear_right_upper_leg" />
-        <dynamics damping="0.1" friction="0.1"/>
         <limit effort="1000" velocity="1000.00" lower="-0.89884456477707963539" upper="2.2951079663725435509" />
     </joint>
-    <transmission name="rear_right_hip_y_trans">
-        <type>transmission_interface/SimpleTransmission</type>
-        <joint name="rear_right_hip_y">
-            <hardwareInterface>EffortJointInterface</hardwareInterface>
-            </joint>
-        <actuator name="rear_right_hip_y">
-            <mechanicalReduction>50</mechanicalReduction>
-            <hardwareInterface>EffortJointInterface</hardwareInterface>
-        </actuator>
-    </transmission>
     <link name="rear_right_lower_leg">
         <visual>
@@ -466,8 +256,4 @@
             </geometry>
         </collision>
-        <inertial>
-            <mass value="1.0" />
-    	    <inertia  ixx="0.0" ixy="0.0"  ixz="0.0"  iyy="0.045"  iyz="0.0"  izz="0.0" />
-    	</inertial>
     </link>
     <joint name="rear_right_knee" type="revolute">
@@ -476,32 +262,6 @@
         <parent link="rear_right_upper_leg" />
         <child link="rear_right_lower_leg" />
-        <dynamics damping="0.1" friction="0.1"/>
         <limit effort="1000" velocity="1000.00" lower="-2.7929" upper="-0.257725" />
     </joint>
-    <gazebo reference="rear_right_lower_leg">
-        <sensor name="rear_right_lower_leg_contactsensor_sensor" type="contact">
-        <always_on>true</always_on>
-        <contact>
-            <collision>rear_right_lower_leg_fixed_joint_lump__rear_bump_sensor_collision</collision>
-        </contact>
-        <plugin filename="libgazebo_ros_bumper.so" name="rear_right_lower_leg_plugin">
-            <bumperTopicName>rear_right_lower_leg_contact</bumperTopicName>
-            <frameName>rear_right_lower_leg</frameName>
-        </plugin>
-        </sensor>
-    </gazebo>
-    <transmission name="rear_right_knee_trans">
-        <type>transmission_interface/SimpleTransmission</type>
-        <joint name="rear_right_knee">
-            <hardwareInterface>EffortJointInterface</hardwareInterface>
-            </joint>
-        <actuator name="rear_right_knee">
-            <mechanicalReduction>50</mechanicalReduction>
-            <hardwareInterface>EffortJointInterface</hardwareInterface>
-        </actuator>
-    </transmission>
-    <gazebo>
-    	<plugin name="gazebo_ros_control" filename="libgazebo_ros_control.so"/>
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