Commit message: Revert "spot_ros in catkin_ws on spot"
This reverts commit fe6b80d88789fd8da3bb13667d48cfc86882e563.

File: spot_description/urdf/arm/spot_arm.urdf.xacro (robot description, xacro)
@@ -82,5 +82,5 @@
         <parent link="${name}_shoulder_pitch"/>
         <child link="${name}_shoulder_roll"/>
-        <!--limit effort="1000" velocity="1000.00" lower="-1e6" upper="1e6"/-->
+	<limit effort="0" velocity="0" lower="0" upper="0"/>
     </joint>
     <link name="${name}_elbow_pitch">
@@ -192,6 +192,5 @@
         <limit effort="1000" velocity="1000.00" lower="-2.87979326579064354163" upper="2.87979326579064354163"/>
     </joint>
-    <link name="${name}_tool0">
-    </link>
+    <link name="${name}_tool0"/>
     <joint name="${name}_ee_virtual_joint" type="fixed">
         <origin xyz="0.19557 0 0" rpy="0 0 0"/>
@@ -227,4 +226,28 @@
         <limit effort="1000" velocity="1000.00" lower="-1.57" upper="0.0"/>
     </joint>
+    <link name="${name}.link_wr1"/>
+    <joint name="${name}_link_wr1_to_wrist" type = "fixed">
+        <parent link = "${name}_wrist_roll"/>
+        <child  link = "${name}.link_wr1"/>
+        <origin xyz = "0 0 0"/>
+    </joint>
+    <link name="${name}_hand"/>
+    <joint name="${name}_wrist_to_hand" type="fixed">
+        <parent link = "${name}_wrist_roll"/>
+        <child  link = "${name}_hand"/>
+        <origin xyz = "0.19557 0.0 0.0"/>
+    </joint>
+    <link name="hand_color_image_sensor"/>
+    <joint name="color_image_joint" type="fixed">
+        <parent link = "${name}_wrist_roll"/>
+        <child  link = "hand_color_image_sensor"/>
+        <origin xyz  = "0.14 0.02 0.022" rpy="-1.42 0 -1.57"/>
+    </joint>
+    <link name="hand_depth_sensor"/>
+    <joint name="depth_sensor_joint" type="fixed">
+        <parent link = "${name}_wrist_roll"/>
+        <child  link = "hand_depth_sensor"/>
+        <origin xyz  = "0.14 0.0 0.01" rpy="0 1.42 0"/>
+    </joint>
     </xacro:macro>
 <!-- Transmissions -->

File: spot_description/urdf/spot.urdf.xacro (robot description, xacro)
@@ -4,6 +4,7 @@
          published by the driver (see spot_driver package) during runtime, so that the transforms
          include calibration adjustments. -->
-    <xacro:arg name="has_arm" default="true" />
-    <xacro:arg name="has_velodyne" default="false" />
+    <xacro:arg name="has_arm" default="False" />
+    <xacro:arg name="has_eap" default="False" />
+    <!-- Fixed links -->
     <link name="body">
         <visual>
@@ -17,4 +18,8 @@
             </geometry>
         </collision>
+        <inertial>
+             <mass value="16.25" />
+             <inertia  ixx="0.085" ixy="0.0"  ixz="0.0"  iyy="1.045"  iyz="0.0"  izz="1.042" />
+    	</inertial>
     </link>
     <link name="base_link"/>
@@ -36,4 +41,5 @@
         <child link="rear_rail" />
     </joint>
+    <!-- Front Left -->
     <link name="front_left_hip">
         <visual>
@@ -47,4 +53,8 @@
             </geometry>
         </collision>
+        <inertial>
+            <mass value="1.5" />
+    	    <inertia  ixx="0.0605" ixy="0.0"  ixz="0.0"  iyy="0.0"  iyz="0.0"  izz="0.0" />
+    	</inertial>
     </link>
     <joint name="front_left_hip_x" type="revolute">
@@ -53,6 +63,17 @@
         <parent link="body" />
         <child link="front_left_hip" />
+        <dynamics damping="0.1" friction="0.1"/>
         <limit effort="1000" velocity="1000.00" lower="-0.78539816339744827899" upper="0.78539816339744827899" />
     </joint>
+    <transmission name="front_left_hip_x_trans">
+	    <type>transmission_interface/SimpleTransmission</type>
+	    <joint name="front_left_hip_x">
+            <hardwareInterface>EffortJointInterface</hardwareInterface>
+        </joint>
+	    <actuator name="front_left_hip_x">
+          	<mechanicalReduction>50</mechanicalReduction>
+          	<hardwareInterface>EffortJointInterface</hardwareInterface>
+	    </actuator>
+    </transmission>
     <link name="front_left_upper_leg">
         <visual>
@@ -66,4 +87,8 @@
             </geometry>
         </collision>
+        <inertial>
+            <mass value="1.5" />
+    	    <inertia  ixx="0.0" ixy="0.0"  ixz="0.0"  iyy="0.05"  iyz="0.0"  izz="0.0" />
+    	</inertial>
     </link>
     <joint name="front_left_hip_y" type="revolute">
@@ -72,6 +97,17 @@
         <parent link="front_left_hip" />
         <child link="front_left_upper_leg" />
+        <dynamics damping="0.1" friction="0.1"/>
         <limit effort="1000" velocity="1000.00" lower="-0.89884456477707963539" upper="2.2951079663725435509" />
     </joint>
+    <transmission name="front_left_hip_y_trans">
+        <type>transmission_interface/SimpleTransmission</type>
+        <joint name="front_left_hip_y">
+            <hardwareInterface>EffortJointInterface</hardwareInterface>
+        </joint>
+        <actuator name="front_left_hip_y">
+            <mechanicalReduction>50</mechanicalReduction>
+            <hardwareInterface>EffortJointInterface</hardwareInterface>
+        </actuator>
+    </transmission>
     <link name="front_left_lower_leg">
         <visual>
@@ -85,4 +121,8 @@
             </geometry>
         </collision>
+        <inertial>
+            <mass value="1.0" />
+    	    <inertia  ixx="0.0" ixy="0.0"  ixz="0.0"  iyy="0.045"  iyz="0.0"  izz="0.0" />
+    	</inertial>
     </link>
     <joint name="front_left_knee" type="revolute">
@@ -91,6 +131,30 @@
         <parent link="front_left_upper_leg" />
         <child link="front_left_lower_leg" />
+        <dynamics damping="0.1" friction="0.1"/>
         <limit effort="1000" velocity="1000.00" lower="-2.7929" upper="-0.254801" />
     </joint>
+    <gazebo reference="front_left_lower_leg">
+        <sensor name="front_left_lower_leg_contactsensor_sensor" type="contact">
+        <always_on>true</always_on>
+        <contact>
+            <collision>front_left_lower_leg_fixed_joint_lump__front_bump_sensor_collision</collision>
+        </contact>
+        <plugin filename="libgazebo_ros_bumper.so" name="front_left_lower_leg_plugin">
+            <bumperTopicName>front_left_lower_leg_contact</bumperTopicName>
+            <frameName>front_left_lower_leg</frameName>
+        </plugin>
+        </sensor>
+    </gazebo>
+    <transmission name="front_left_knee_trans">
+	  <type>transmission_interface/SimpleTransmission</type>
+	  <joint name="front_left_knee">
+          	<hardwareInterface>EffortJointInterface</hardwareInterface>
+      </joint>
+	  <actuator name="front_left_knee">
+          	<mechanicalReduction>50</mechanicalReduction>
+          	<hardwareInterface>EffortJointInterface</hardwareInterface>
+	  </actuator>
+    </transmission>
+    <!-- Front Right -->
     <link name="front_right_hip">
         <visual>
@@ -104,4 +168,8 @@
             </geometry>
         </collision>
+        <inertial>
+            <mass value="1.5" />
+    	    <inertia  ixx="0.0605" ixy="0.0"  ixz="0.0"  iyy="0.0"  iyz="0.0"  izz="0.0" />
+    	</inertial>
     </link>
     <joint name="front_right_hip_x" type="revolute">
@@ -110,6 +178,17 @@
         <parent link="body" />
         <child link="front_right_hip" />
+        <dynamics damping="0.1" friction="0.1"/>
         <limit effort="1000" velocity="1000.00" lower="-0.78539816339744827899" upper="0.78539816339744827899" />
     </joint>
+    <transmission name="front_right_hip_x_trans">
+	  <type>transmission_interface/SimpleTransmission</type>
+	  <joint name="front_right_hip_x">
+          	<hardwareInterface>EffortJointInterface</hardwareInterface>
+      </joint>
+	  <actuator name="front_right_hip_x">
+          	<mechanicalReduction>50</mechanicalReduction>
+          	<hardwareInterface>EffortJointInterface</hardwareInterface>
+	  </actuator>
+    </transmission>
     <link name="front_right_upper_leg">
         <visual>
@@ -123,4 +202,8 @@
             </geometry>
         </collision>
+        <inertial>
+            <mass value="1.5" />
+    	    <inertia  ixx="0.0" ixy="0.0"  ixz="0.0"  iyy="0.05"  iyz="0.0"  izz="0.0" />
+    	</inertial>
     </link>
     <joint name="front_right_hip_y" type="revolute">
@@ -129,6 +212,17 @@
         <parent link="front_right_hip" />
         <child link="front_right_upper_leg" />
+        <dynamics damping="0.1" friction="0.1"/>
         <limit effort="1000" velocity="1000.00" lower="-0.89884456477707963539" upper="2.2951079663725435509" />
     </joint>
+    <transmission name="front_right_hip_y_trans">
+        <type>transmission_interface/SimpleTransmission</type>
+        <joint name="front_right_hip_y">
+            <hardwareInterface>EffortJointInterface</hardwareInterface>
+        </joint>
+        <actuator name="front_right_hip_y">
+            <mechanicalReduction>50</mechanicalReduction>
+            <hardwareInterface>EffortJointInterface</hardwareInterface>
+        </actuator>
+    </transmission>
     <link name="front_right_lower_leg">
         <visual>
@@ -142,4 +236,8 @@
             </geometry>
         </collision>
+        <inertial>
+            <mass value="1.0" />
+    	    <inertia  ixx="0.0" ixy="0.0"  ixz="0.0"  iyy="0.045"  iyz="0.0"  izz="0.0" />
+    	</inertial>
     </link>
     <joint name="front_right_knee" type="revolute">
@@ -148,6 +246,30 @@
         <parent link="front_right_upper_leg" />
         <child link="front_right_lower_leg" />
+        <dynamics damping="0.1" friction="0.1"/>
         <limit effort="1000" velocity="1000.00" lower="-2.7929" upper="-0.247563" />
     </joint>
+    <gazebo reference="front_right_lower_leg">
+        <sensor name="front_right_lower_leg_contactsensor_sensor" type="contact">
+        <always_on>true</always_on>
+        <contact>
+            <collision>front_right_lower_leg_fixed_joint_lump__front_bump_sensor_collision</collision>
+        </contact>
+        <plugin filename="libgazebo_ros_bumper.so" name="front_right_lower_leg_plugin">
+            <bumperTopicName>front_right_lower_leg_contact</bumperTopicName>
+            <frameName>front_right_lower_leg</frameName>
+        </plugin>
+        </sensor>
+    </gazebo>
+    <transmission name="front_right_knee_trans">
+        <type>transmission_interface/SimpleTransmission</type>
+        <joint name="front_right_knee">
+            <hardwareInterface>EffortJointInterface</hardwareInterface>
+        </joint>
+        <actuator name="front_right_knee">
+            <mechanicalReduction>50</mechanicalReduction>
+            <hardwareInterface>EffortJointInterface</hardwareInterface>
+        </actuator>
+    </transmission>
+    <!-- Rear Left -->
     <link name="rear_left_hip">
         <visual>
@@ -161,4 +283,8 @@
             </geometry>
         </collision>
+        <inertial>
+            <mass value="1.5" />
+    	    <inertia  ixx="0.0605" ixy="0.0"  ixz="0.0"  iyy="0.0"  iyz="0.0"  izz="0.0" />
+    	</inertial>
     </link>
     <joint name="rear_left_hip_x" type="revolute">
@@ -167,6 +293,17 @@
         <parent link="body" />
         <child link="rear_left_hip" />
+        <dynamics damping="0.1" friction="0.1"/>
         <limit effort="1000" velocity="1000.00" lower="-0.78539816339744827899" upper="0.78539816339744827899" />
     </joint>
+    <transmission name="rear_left_hip_x_trans">
+        <type>transmission_interface/SimpleTransmission</type>
+        <joint name="rear_left_hip_x">
+            <hardwareInterface>EffortJointInterface</hardwareInterface>
+        </joint>
+        <actuator name="rear_left_hip_x">
+            <mechanicalReduction>50</mechanicalReduction>
+            <hardwareInterface>EffortJointInterface</hardwareInterface>
+        </actuator>
+    </transmission>
     <link name="rear_left_upper_leg">
         <visual>
@@ -180,4 +317,8 @@
             </geometry>
         </collision>
+        <inertial>
+           <mass value="1.5" />
+    	   <inertia  ixx="0.0" ixy="0.0"  ixz="0.0"  iyy="0.05"  iyz="0.0"  izz="0.0" />
+    	</inertial>
     </link>
     <joint name="rear_left_hip_y" type="revolute">
@@ -186,6 +327,17 @@
         <parent link="rear_left_hip" />
         <child link="rear_left_upper_leg" />
+        <dynamics damping="0.1" friction="0.1"/>
         <limit effort="1000" velocity="1000.00" lower="-0.89884456477707963539" upper="2.2951079663725435509" />
     </joint>
+    <transmission name="rear_left_hip_y_trans">
+        <type>transmission_interface/SimpleTransmission</type>
+        <joint name="rear_left_hip_y">
+            <hardwareInterface>EffortJointInterface</hardwareInterface>
+        </joint>
+        <actuator name="rear_left_hip_y">
+            <mechanicalReduction>50</mechanicalReduction>
+            <hardwareInterface>EffortJointInterface</hardwareInterface>
+        </actuator>
+    </transmission>
     <link name="rear_left_lower_leg">
         <visual>
@@ -199,4 +351,8 @@
             </geometry>
         </collision>
+        <inertial>
+            <mass value="1.0" />
+    	    <inertia  ixx="0.0" ixy="0.0"  ixz="0.0"  iyy="0.045"  iyz="0.0"  izz="0.0" />
+    	</inertial>
     </link>
     <joint name="rear_left_knee" type="revolute">
@@ -205,6 +361,30 @@
         <parent link="rear_left_upper_leg" />
         <child link="rear_left_lower_leg" />
+        <dynamics damping="0.1" friction="0.1"/>
         <limit effort="1000" velocity="1000.00" lower="-2.7929" upper="-0.267153" />
     </joint>
+    <gazebo reference="rear_left_lower_leg">
+        <sensor name="rear_left_lower_leg_contactsensor_sensor" type="contact">
+        <always_on>true</always_on>
+        <contact>
+            <collision>rear_left_lower_leg_fixed_joint_lump__rear_bump_sensor_collision</collision>
+        </contact>
+        <plugin filename="libgazebo_ros_bumper.so" name="rear_left_lower_leg_plugin">
+            <bumperTopicName>rear_left_lower_leg_contact</bumperTopicName>
+            <frameName>rear_left_lower_leg</frameName>
+        </plugin>
+        </sensor>
+    </gazebo>
+    <transmission name="rear_left_knee_trans">
+        <type>transmission_interface/SimpleTransmission</type>
+        <joint name="rear_left_knee">
+             <hardwareInterface>EffortJointInterface</hardwareInterface>
+        </joint>
+        <actuator name="rear_left_knee">
+            <mechanicalReduction>50</mechanicalReduction>
+            <hardwareInterface>EffortJointInterface</hardwareInterface>
+        </actuator>
+    </transmission>
+    <!-- Rear Right -->
     <link name="rear_right_hip">
         <visual>
@@ -218,4 +398,8 @@
             </geometry>
         </collision>
+        <inertial>
+            <mass value="1.5" />
+    	    <inertia  ixx="0.0605" ixy="0.0"  ixz="0.0"  iyy="0.0"  iyz="0.0"  izz="0.0" />
+    	</inertial>
     </link>
     <joint name="rear_right_hip_x" type="revolute">
@@ -224,6 +408,17 @@
         <parent link="body" />
         <child link="rear_right_hip" />
+        <dynamics damping="0.1" friction="0.1"/>
         <limit effort="1000" velocity="1000.00" lower="-0.78539816339744827899" upper="0.78539816339744827899" />
     </joint>
+    <transmission name="rear_right_hip_x_trans">
+        <type>transmission_interface/SimpleTransmission</type>
+        <joint name="rear_right_hip_x">
+            <hardwareInterface>EffortJointInterface</hardwareInterface>
+        </joint>
+        <actuator name="rear_right_hip_x">
+            <mechanicalReduction>50</mechanicalReduction>
+            <hardwareInterface>EffortJointInterface</hardwareInterface>
+        </actuator>
+    </transmission>
     <link name="rear_right_upper_leg">
         <visual>
@@ -237,4 +432,8 @@
             </geometry>
         </collision>
+        <inertial>
+            <mass value="1.5" />
+    	    <inertia  ixx="0.0" ixy="0.0"  ixz="0.0"  iyy="0.05"  iyz="0.0"  izz="0.0" />
+    	</inertial>
     </link>
     <joint name="rear_right_hip_y" type="revolute">
@@ -243,6 +442,17 @@
         <parent link="rear_right_hip" />
         <child link="rear_right_upper_leg" />
+        <dynamics damping="0.1" friction="0.1"/>
         <limit effort="1000" velocity="1000.00" lower="-0.89884456477707963539" upper="2.2951079663725435509" />
     </joint>
+    <transmission name="rear_right_hip_y_trans">
+        <type>transmission_interface/SimpleTransmission</type>
+        <joint name="rear_right_hip_y">
+            <hardwareInterface>EffortJointInterface</hardwareInterface>
+            </joint>
+        <actuator name="rear_right_hip_y">
+            <mechanicalReduction>50</mechanicalReduction>
+            <hardwareInterface>EffortJointInterface</hardwareInterface>
+        </actuator>
+    </transmission>
     <link name="rear_right_lower_leg">
         <visual>
@@ -256,4 +466,8 @@
             </geometry>
         </collision>
+        <inertial>
+            <mass value="1.0" />
+    	    <inertia  ixx="0.0" ixy="0.0"  ixz="0.0"  iyy="0.045"  iyz="0.0"  izz="0.0" />
+    	</inertial>
     </link>
     <joint name="rear_right_knee" type="revolute">
@@ -262,6 +476,32 @@
         <parent link="rear_right_upper_leg" />
         <child link="rear_right_lower_leg" />
+        <dynamics damping="0.1" friction="0.1"/>
         <limit effort="1000" velocity="1000.00" lower="-2.7929" upper="-0.257725" />
     </joint>
+    <gazebo reference="rear_right_lower_leg">
+        <sensor name="rear_right_lower_leg_contactsensor_sensor" type="contact">
+        <always_on>true</always_on>
+        <contact>
+            <collision>rear_right_lower_leg_fixed_joint_lump__rear_bump_sensor_collision</collision>
+        </contact>
+        <plugin filename="libgazebo_ros_bumper.so" name="rear_right_lower_leg_plugin">
+            <bumperTopicName>rear_right_lower_leg_contact</bumperTopicName>
+            <frameName>rear_right_lower_leg</frameName>
+        </plugin>
+        </sensor>
+    </gazebo>
+    <transmission name="rear_right_knee_trans">
+        <type>transmission_interface/SimpleTransmission</type>
+        <joint name="rear_right_knee">
+            <hardwareInterface>EffortJointInterface</hardwareInterface>
+            </joint>
+        <actuator name="rear_right_knee">
+            <mechanicalReduction>50</mechanicalReduction>
+            <hardwareInterface>EffortJointInterface</hardwareInterface>
+        </actuator>
+    </transmission>
+    <gazebo>
+    	<plugin name="gazebo_ros_control" filename="libgazebo_ros_control.so"/>
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
Commit message: made realsense optional

File: spot_description/urdf/arm/spot_arm.urdf.xacro (robot description, xacro)
@@ -2,4 +2,5 @@
 <robot xmlns:xacro="http://www.ros.org/wiki/xacro">
     <xacro:macro name="spot_arm" params="name" >
+    <xacro:arg name="has_realsense" default="False" />
     <link name="${name}_base_link"/>
     <link name="${name}_shoulder_yaw">
@@ -313,3 +314,9 @@
   </transmission>
 <!-- EOF Transmissions -->
+  <xacro:if value="$(arg has_realsense)">
+    <xacro:include filename="$(find spot_description)/urdf/realsense_mount.urdf.xacro"/>
+    <xacro:realsense_mount parent = "arm0_wrist_roll">
+      <origin xyz = "0.145 0 -0.06" rpy = "3.1416 0 -1.57"/>
+    </xacro:realsense_mount>
+  </xacro:if>
 </robot>

File: spot_description/urdf/spot.urdf.xacro (robot description, xacro)
@@ -538,8 +538,4 @@
         </xacro:VLP-16>
     </xacro:if>
-    <xacro:include filename="$(find spot_description)/urdf/realsense_mount.urdf.xacro"/>
-    <xacro:realsense_mount parent = "arm0_wrist_roll">
-        <origin xyz = "0.145 0 -0.06" rpy = "3.1416 0 -1.57"/>
-    </xacro:realsense_mount>
     <!-- Optional custom includes. -->
     <xacro:include filename="$(optenv SPOT_URDF_EXTRAS empty.urdf)" />

Commit message: Updated arm URDF to use high quality colored meshes

File: spot_description/urdf/arm/spot_arm.urdf.xacro (robot description, xacro)
@@ -8,5 +8,5 @@
         <origin xyz="0 0 0" rpy="0 0 0"/>
         <geometry>
-            <mesh filename="package://spot_description/meshes/arm/arm0.link_sh0.obj"/>
+            <mesh filename="package://spot_description/meshes/arm/arm0.link_sh0.dae"/>
         </geometry>
         <material name="arm0.link_sh0">
@@ -62,5 +62,5 @@
         <origin xyz="0 0 0" rpy="0 0 0"/>
         <geometry>
-            <mesh filename="package://spot_description/meshes/arm/arm0.link_hr0.obj"/>
+            <mesh filename="package://spot_description/meshes/arm/arm0.link_hr0.dae"/>
         </geometry>
             <material name="arm0.link_hr0">
@@ -89,5 +89,5 @@
         <origin xyz="0 0 0" rpy="0 0 0"/>
         <geometry>
-            <mesh filename="package://spot_description/meshes/arm/arm0.link_el0.obj"/>
+            <mesh filename="package://spot_description/meshes/arm/arm0.link_el0.dae"/>
         </geometry>
             <material name="arm0.link_el0">
@@ -116,5 +116,5 @@
         <origin xyz="0 0 0" rpy="0 0 0"/>
         <geometry>
-            <mesh filename="package://spot_description/meshes/arm/arm0.link_el1.obj"/>
+            <mesh filename="package://spot_description/meshes/arm/arm0.link_el1.dae"/>
         </geometry>
             <material name="arm0.link_el1">
@@ -143,5 +143,5 @@
         <origin xyz="0 0 0" rpy="0 0 0"/>
         <geometry>
-            <mesh filename="package://spot_description/meshes/arm/arm0.link_wr0.obj"/>
+            <mesh filename="package://spot_description/meshes/arm/arm0.link_wr0.dae"/>
         </geometry>
             <material name="arm0.link_wr0">
@@ -170,5 +170,5 @@
         <origin xyz="0 0 0" rpy="0 0 0"/>
         <geometry>
-            <mesh filename="package://spot_description/meshes/arm/arm0.link_wr1.obj"/>
+            <mesh filename="package://spot_description/meshes/arm/arm0.link_wr1.dae"/>
         </geometry>
             <material name="arm0.link_wr1">
@@ -204,5 +204,5 @@
         <origin xyz="0 0 0" rpy="0 0 0"/>
         <geometry>
-            <mesh filename="package://spot_description/meshes/arm/arm0.link_fngr.obj"/>
+            <mesh filename="package://spot_description/meshes/arm/arm0.link_fngr.dae"/>
         </geometry>
         <material name="arm0.link_fngr">
