Commit message: Fixed indentation on spot arm xacro file

File: spot_description/urdf/arm/spot_arm.urdf.xacro (robot description, xacro)
@@ -6,20 +6,20 @@
     <link name="${name}_shoulder_yaw">
         <visual>
-        <origin xyz="0 0 0" rpy="0 0 0"/>
-        <geometry>
-            <mesh filename="package://spot_description/meshes/arm/arm0.link_sh0.dae"/>
-        </geometry>
-        <material name="arm0.link_sh0">
-            <color rgba="0.2 0.2 0.2 1"/>
-        </material>
-        </visual>
-        <collision>
-        <origin xyz="0 0 0" rpy="0 0 0"/>
-        <geometry>
-            <mesh filename="package://spot_description/meshes/arm/arm0.link_sh0.obj"/>
-        </geometry>
-        <material name="arm0.link_sh0">
-            <color rgba="1 0.2 0.2 1"/>
-        </material>
+            <origin xyz="0 0 0" rpy="0 0 0"/>
+            <geometry>
+                <mesh filename="package://spot_description/meshes/arm/arm0.link_sh0.dae"/>
+            </geometry>
+            <material name="arm0.link_sh0">
+                <color rgba="0.2 0.2 0.2 1"/>
+            </material>
+        </visual>
+        <collision>
+            <origin xyz="0 0 0" rpy="0 0 0"/>
+            <geometry>
+                <mesh filename="package://spot_description/meshes/arm/arm0.link_sh0.obj"/>
+            </geometry>
+            <material name="arm0.link_sh0">
+                <color rgba="1 0.2 0.2 1"/>
+            </material>
         </collision>
     </link>
@@ -33,20 +33,20 @@
     <link name="${name}_shoulder_pitch">
         <visual>
-        <origin xyz="0 0 0" rpy="0 0 0"/>
-        <geometry>
-            <mesh filename="package://spot_description/meshes/arm/arm0.link_sh1.obj"/>
-        </geometry>
-        <material name="arm0.link_sh1">
-            <color rgba="0.2 0.2 0.2 1"/>
-        </material>
-        </visual>
-        <collision>
-        <origin xyz="0 0 0" rpy="0 0 0"/>
-        <geometry>
-            <mesh filename="package://spot_description/meshes/arm/arm0.link_sh1.obj"/>
-        </geometry>
-        <material name="arm0.link_sh1">
-            <color rgba="1 0.2 0.2 1"/>
-        </material>
+            <origin xyz="0 0 0" rpy="0 0 0"/>
+            <geometry>
+                <mesh filename="package://spot_description/meshes/arm/arm0.link_sh1.obj"/>
+            </geometry>
+            <material name="arm0.link_sh1">
+                <color rgba="0.2 0.2 0.2 1"/>
+            </material>
+        </visual>
+        <collision>
+            <origin xyz="0 0 0" rpy="0 0 0"/>
+            <geometry>
+                <mesh filename="package://spot_description/meshes/arm/arm0.link_sh1.obj"/>
+            </geometry>
+            <material name="arm0.link_sh1">
+                <color rgba="1 0.2 0.2 1"/>
+            </material>
         </collision>
     </link>
@@ -60,19 +60,19 @@
     <link name="${name}_shoulder_roll">
         <visual>
-        <origin xyz="0 0 0" rpy="0 0 0"/>
-        <geometry>
-            <mesh filename="package://spot_description/meshes/arm/arm0.link_hr0.dae"/>
-        </geometry>
+            <origin xyz="0 0 0" rpy="0 0 0"/>
+            <geometry>
+                <mesh filename="package://spot_description/meshes/arm/arm0.link_hr0.dae"/>
+            </geometry>
+                <material name="arm0.link_hr0">
+                    <color rgba="0.2 0.2 0.2 1"/>
+                </material>
+        </visual>
+        <collision>
+            <origin xyz="0 0 0" rpy="0 0 0"/>
+            <geometry>
+                <mesh filename="package://spot_description/meshes/arm/arm0.link_hr0.obj"/>
+            </geometry>
             <material name="arm0.link_hr0">
-            <color rgba="0.2 0.2 0.2 1"/>
-            </material>
-        </visual>
-        <collision>
-        <origin xyz="0 0 0" rpy="0 0 0"/>
-        <geometry>
-            <mesh filename="package://spot_description/meshes/arm/arm0.link_hr0.obj"/>
-        </geometry>
-            <material name="arm0.link_hr0">
-            <color rgba="1 0.2 0.2 1"/>
+                <color rgba="1 0.2 0.2 1"/>
             </material>
         </collision>
@@ -83,23 +83,23 @@
         <parent link="${name}_shoulder_pitch"/>
         <child link="${name}_shoulder_roll"/>
-	<limit effort="0" velocity="0" lower="0" upper="0"/>
+        <limit effort="0" velocity="0" lower="0" upper="0"/>
     </joint>
     <link name="${name}_elbow_pitch">
         <visual>
-        <origin xyz="0 0 0" rpy="0 0 0"/>
-        <geometry>
-            <mesh filename="package://spot_description/meshes/arm/arm0.link_el0.dae"/>
-        </geometry>
+            <origin xyz="0 0 0" rpy="0 0 0"/>
+            <geometry>
+                <mesh filename="package://spot_description/meshes/arm/arm0.link_el0.dae"/>
+            </geometry>
             <material name="arm0.link_el0">
-            <color rgba="0.2 0.2 0.2 1"/>
-            </material>
-        </visual>
-        <collision>
-        <origin xyz="0 0 0" rpy="0 0 0"/>
-        <geometry>
-            <mesh filename="package://spot_description/meshes/arm/arm0.link_el0.obj"/>
-        </geometry>
+                <color rgba="0.2 0.2 0.2 1"/>
+            </material>
+        </visual>
+        <collision>
+            <origin xyz="0 0 0" rpy="0 0 0"/>
+            <geometry>
+                <mesh filename="package://spot_description/meshes/arm/arm0.link_el0.obj"/>
+            </geometry>
             <material name="arm0.link_el0">
-            <color rgba="1 0.2 0.2 1"/>
+                <color rgba="1 0.2 0.2 1"/>
             </material>
         </collision>
@@ -114,19 +114,19 @@
     <link name="${name}_elbow_roll">
         <visual>
-        <origin xyz="0 0 0" rpy="0 0 0"/>
-        <geometry>
-            <mesh filename="package://spot_description/meshes/arm/arm0.link_el1.dae"/>
-        </geometry>
+            <origin xyz="0 0 0" rpy="0 0 0"/>
+            <geometry>
+                <mesh filename="package://spot_description/meshes/arm/arm0.link_el1.dae"/>
+            </geometry>
             <material name="arm0.link_el1">
-            <color rgba="0.2 0.2 0.2 1"/>
-            </material>
-        </visual>
-        <collision>
-        <origin xyz="0 0 0" rpy="0 0 0"/>
-        <geometry>
-            <mesh filename="package://spot_description/meshes/arm/arm0.link_el1.obj"/>
-        </geometry>
+                <color rgba="0.2 0.2 0.2 1"/>
+            </material>
+        </visual>
+        <collision>
+            <origin xyz="0 0 0" rpy="0 0 0"/>
+            <geometry>
+                <mesh filename="package://spot_description/meshes/arm/arm0.link_el1.obj"/>
+            </geometry>
             <material name="arm0.link_el1">
-            <color rgba="1 0.2 0.2 1"/>
+                <color rgba="1 0.2 0.2 1"/>
             </material>
         </collision>
@@ -141,19 +141,19 @@
     <link name="${name}_wrist_pitch">
         <visual>
-        <origin xyz="0 0 0" rpy="0 0 0"/>
-        <geometry>
-            <mesh filename="package://spot_description/meshes/arm/arm0.link_wr0.dae"/>
-        </geometry>
+            <origin xyz="0 0 0" rpy="0 0 0"/>
+            <geometry>
+                <mesh filename="package://spot_description/meshes/arm/arm0.link_wr0.dae"/>
+            </geometry>
             <material name="arm0.link_wr0">
-            <color rgba="0.2 0.2 0.2 1"/>
-            </material>
-        </visual>
-        <collision>
-        <origin xyz="0 0 0" rpy="0 0 0"/>
-        <geometry>
-            <mesh filename="package://spot_description/meshes/arm/arm0.link_wr0.obj"/>
-        </geometry>
+                <color rgba="0.2 0.2 0.2 1"/>
+            </material>
+        </visual>
+        <collision>
+            <origin xyz="0 0 0" rpy="0 0 0"/>
+            <geometry>
+                <mesh filename="package://spot_description/meshes/arm/arm0.link_wr0.obj"/>
+            </geometry>
             <material name="arm0.link_wr0">
-            <color rgba="1 0.2 0.2 1"/>
+                <color rgba="1 0.2 0.2 1"/>
             </material>
         </collision>
@@ -168,19 +168,19 @@
     <link name="${name}_wrist_roll">
         <visual>
-        <origin xyz="0 0 0" rpy="0 0 0"/>
-        <geometry>
-            <mesh filename="package://spot_description/meshes/arm/arm0.link_wr1.dae"/>
-        </geometry>
+            <origin xyz="0 0 0" rpy="0 0 0"/>
+            <geometry>
+                <mesh filename="package://spot_description/meshes/arm/arm0.link_wr1.dae"/>
+            </geometry>
             <material name="arm0.link_wr1">
-            <color rgba="0.2 0.2 0.2 1"/>
-            </material>
-        </visual>
-        <collision>
-        <origin xyz="0 0 0" rpy="0 0 0"/>
-        <geometry>
-            <mesh filename="package://spot_description/meshes/arm/arm0.link_wr1.obj"/>
-        </geometry>
+                <color rgba="0.2 0.2 0.2 1"/>
+            </material>
+        </visual>
+            <collision>
+            <origin xyz="0 0 0" rpy="0 0 0"/>
+            <geometry>
+                <mesh filename="package://spot_description/meshes/arm/arm0.link_wr1.obj"/>
+            </geometry>
             <material name="arm0.link_wr1">
-            <color rgba="1 0.2 0.2 1"/>
+                <color rgba="1 0.2 0.2 1"/>
             </material>
         </collision>
@@ -202,20 +202,20 @@
     <link name="${name}_fingers">
         <visual>
-        <origin xyz="0 0 0" rpy="0 0 0"/>
-        <geometry>
-            <mesh filename="package://spot_description/meshes/arm/arm0.link_fngr.dae"/>
-        </geometry>
-        <material name="arm0.link_fngr">
-            <color rgba="0.2 0.2 0.2 1"/>
-        </material>
-        </visual>
-        <collision>
-        <origin xyz="0 0 0" rpy="0 0 0"/>
-        <geometry>
-            <mesh filename="package://spot_description/meshes/arm/arm0.link_fngr.obj"/>
-        </geometry>
-        <material name="arm0.link_fngr">
-            <color rgba="0.2 0.2 0.2 1"/>
-        </material>
+            <origin xyz="0 0 0" rpy="0 0 0"/>
+            <geometry>
+                <mesh filename="package://spot_description/meshes/arm/arm0.link_fngr.dae"/>
+            </geometry>
+            <material name="arm0.link_fngr">
+                <color rgba="0.2 0.2 0.2 1"/>
+            </material>
+        </visual>
+        <collision>
+            <origin xyz="0 0 0" rpy="0 0 0"/>
+            <geometry>
+                <mesh filename="package://spot_description/meshes/arm/arm0.link_fngr.obj"/>
+            </geometry>
+            <material name="arm0.link_fngr">
+                <color rgba="0.2 0.2 0.2 1"/>
+            </material>
         </collision>
     </link>

Commit message: Added visual and collision for the arm base

File: spot_description/urdf/arm/spot_arm.urdf.xacro (robot description, xacro)
@@ -3,5 +3,19 @@
     <xacro:macro name="spot_arm" params="name" >
     <xacro:arg name="has_realsense" default="False" />
-    <link name="${name}_base_link"/>
+    <link name="${name}_base_link">
+        <visual>
+            <geometry>
+                <!-- Add a small scale increase to cover up body mesh imperfections -->
+                <mesh filename="package://spot_description/meshes/arm/arm0.base_link.dae" scale="1.02 1.02 1.02"/>
+            </geometry>
+            <origin xyz="-0.001 0.0002 -0.116" rpy="0 0.03 0"/>
+        </visual>
+        <collision>
+            <geometry>
+                <cylinder radius="0.08" length="0.05"/>
+            </geometry>
+            <origin xyz="-0.02 0 -0.08"/>
+        </collision>
+    </link>
     <link name="${name}_shoulder_yaw">
         <visual>

Commit message: adds a dedicated image server to alleviate processing-time burden from the drivers
* Added parameters for image server

* SpotImageServer initial commit

* Added node and fixed bugs to make runnable

* Added services to get single shot images from the robot

* Updated parameter defaults and configs

* Added static transform publisher for calibrated cameras

* Removed image handling references in the body wrapper and ros wrapper

* Added optional namespace for velodyne points

* Added image publisher with default settings to bringup launch

* Incorporated hand static transforms to image publisher

* Added option for image publisher config file

* Made pointcloud source configurable

* Updated to new camera topics

* Added check for empty image requests

* Added missing body image requests

* Updated RGB pixel format to be explicitly stated

File: spot_description/urdf/arm/spot_arm.urdf.xacro (robot description, xacro)
@@ -252,16 +252,4 @@
         <child  link = "${name}_hand"/>
         <origin xyz = "0.19557 0.0 0.0"/>
-    </joint>
-    <link name="hand_color_image_sensor"/>
-    <joint name="color_image_joint" type="fixed">
-        <parent link = "${name}_wrist_roll"/>
-        <child  link = "hand_color_image_sensor"/>
-        <origin xyz  = "0.14 0.02 0.022" rpy="-1.42 0 -1.57"/>
-    </joint>
-    <link name="hand_depth_sensor"/>
-    <joint name="depth_sensor_joint" type="fixed">
-        <parent link = "${name}_wrist_roll"/>
-        <child  link = "hand_depth_sensor"/>
-        <origin xyz  = "0.14 0.0 0.01" rpy="0 1.42 0"/>
     </joint>
     </xacro:macro>

Commit message: Added a frame at the median point of the hand mounting holes for payload registration

File: spot_description/urdf/arm/spot_arm.urdf.xacro (robot description, xacro)
@@ -252,4 +252,10 @@
         <child  link = "${name}_hand"/>
         <origin xyz = "0.19557 0.0 0.0"/>
+    </joint>
+    <link name="${name}_mounting_frame"/>
+    <joint name="${name}_wrist_to_mounting_frame" type="fixed">
+        <parent link = "${name}_wrist_roll"/>
+        <child  link = "${name}_mounting_frame"/>
+        <origin xyz = "0.1103 0 -0.036"/>
     </joint>
     </xacro:macro>

Commit message: add args to the arm xacro to use prop meshes and format

File: spot_description/urdf/arm/spot_arm.urdf.xacro (robot description, xacro)
@@ -3,9 +3,14 @@
     <xacro:macro name="spot_arm" params="name" >
     <xacro:arg name="has_realsense" default="False" />
+    <xacro:arg name="use_proprietary_meshes" default="false" />
+    <xacro:arg name="proprietary_format" default="dae" />
+    <!-- Determine mesh source -->
+  <xacro:property name="mesh_pkg" value="$(eval 'spot_propriety_description' if use_proprietary_meshes else 'spot_description')"/>
+  <xacro:property name="mesh_ext" value="$(eval proprietary_format if use_proprietary_meshes else 'obj')" />
     <link name="${name}_base_link">
         <visual>
             <geometry>
                 <!-- Add a small scale increase to cover up body mesh imperfections -->
-                <mesh filename="package://spot_description/meshes/arm/arm0.base_link.dae" scale="1.02 1.02 1.02"/>
+                <mesh filename="package://$(var mesh_pkg)/meshes/arm/arm0.base_link.$(var mesh_ext)" scale="1.02 1.02 1.02"/>
             </geometry>
             <origin xyz="-0.001 0.0002 -0.116" rpy="0 0.03 0"/>
@@ -22,5 +27,5 @@
             <origin xyz="0 0 0" rpy="0 0 0"/>
             <geometry>
-                <mesh filename="package://spot_description/meshes/arm/arm0.link_sh0.dae"/>
+                <mesh filename="package://$(var mesh_pkg)/meshes/arm/arm0.link_sh0.$(var mesh_ext)"/>
             </geometry>
             <material name="arm0.link_sh0">
@@ -76,5 +81,5 @@
             <origin xyz="0 0 0" rpy="0 0 0"/>
             <geometry>
-                <mesh filename="package://spot_description/meshes/arm/arm0.link_hr0.dae"/>
+                <mesh filename="package://$(var mesh_pkg)/meshes/arm/arm0.link_hr0.$(var mesh_ext)"/>
             </geometry>
                 <material name="arm0.link_hr0">
@@ -103,5 +108,5 @@
             <origin xyz="0 0 0" rpy="0 0 0"/>
             <geometry>
-                <mesh filename="package://spot_description/meshes/arm/arm0.link_el0.dae"/>
+                <mesh filename="package://$(var mesh_pkg)/meshes/arm/arm0.link_el0.$(var mesh_ext)"/>
             </geometry>
             <material name="arm0.link_el0">
@@ -130,5 +135,5 @@
             <origin xyz="0 0 0" rpy="0 0 0"/>
             <geometry>
-                <mesh filename="package://spot_description/meshes/arm/arm0.link_el1.dae"/>
+                <mesh filename="package://$(var mesh_pkg)/meshes/arm/arm0.link_el1.$(var mesh_ext)"/>
             </geometry>
             <material name="arm0.link_el1">
@@ -157,5 +162,5 @@
             <origin xyz="0 0 0" rpy="0 0 0"/>
             <geometry>
-                <mesh filename="package://spot_description/meshes/arm/arm0.link_wr0.dae"/>
+                <mesh filename="package://$(var mesh_pkg)/meshes/arm/arm0.link_wr0.$(var mesh_ext)"/>
             </geometry>
             <material name="arm0.link_wr0">
@@ -184,5 +189,5 @@
             <origin xyz="0 0 0" rpy="0 0 0"/>
             <geometry>
-                <mesh filename="package://spot_description/meshes/arm/arm0.link_wr1.dae"/>
+                <mesh filename="package://$(var mesh_pkg)/meshes/arm/arm0.link_wr1.$(var mesh_ext)"/>
             </geometry>
             <material name="arm0.link_wr1">
@@ -218,5 +223,5 @@
             <origin xyz="0 0 0" rpy="0 0 0"/>
             <geometry>
-                <mesh filename="package://spot_description/meshes/arm/arm0.link_fngr.dae"/>
+                <mesh filename="package://$(var mesh_pkg)/meshes/arm/arm0.link_fngr.$(var mesh_ext)"/>
             </geometry>
             <material name="arm0.link_fngr">

Commit message: fix syntax for xacro variable

File: spot_description/urdf/arm/spot_arm.urdf.xacro (robot description, xacro)
@@ -12,5 +12,5 @@
             <geometry>
                 <!-- Add a small scale increase to cover up body mesh imperfections -->
-                <mesh filename="package://$(var mesh_pkg)/meshes/arm/arm0.base_link.$(var mesh_ext)" scale="1.02 1.02 1.02"/>
+                <mesh filename="package://${mesh_pkg}/meshes/arm/arm0.base_link.${mesh_ext}" scale="1.02 1.02 1.02"/>
             </geometry>
             <origin xyz="-0.001 0.0002 -0.116" rpy="0 0.03 0"/>
@@ -27,5 +27,5 @@
             <origin xyz="0 0 0" rpy="0 0 0"/>
             <geometry>
-                <mesh filename="package://$(var mesh_pkg)/meshes/arm/arm0.link_sh0.$(var mesh_ext)"/>
+                <mesh filename="package://${mesh_pkg}/meshes/arm/arm0.link_sh0.${mesh_ext}"/>
             </geometry>
             <material name="arm0.link_sh0">
@@ -81,5 +81,5 @@
             <origin xyz="0 0 0" rpy="0 0 0"/>
             <geometry>
-                <mesh filename="package://$(var mesh_pkg)/meshes/arm/arm0.link_hr0.$(var mesh_ext)"/>
+                <mesh filename="package://${mesh_pkg}/meshes/arm/arm0.link_hr0.${mesh_ext}"/>
             </geometry>
                 <material name="arm0.link_hr0">
@@ -108,5 +108,5 @@
             <origin xyz="0 0 0" rpy="0 0 0"/>
             <geometry>
-                <mesh filename="package://$(var mesh_pkg)/meshes/arm/arm0.link_el0.$(var mesh_ext)"/>
+                <mesh filename="package://${mesh_pkg}/meshes/arm/arm0.link_el0.${mesh_ext}"/>
             </geometry>
             <material name="arm0.link_el0">
@@ -135,5 +135,5 @@
             <origin xyz="0 0 0" rpy="0 0 0"/>
             <geometry>
-                <mesh filename="package://$(var mesh_pkg)/meshes/arm/arm0.link_el1.$(var mesh_ext)"/>
+                <mesh filename="package://${mesh_pkg}/meshes/arm/arm0.link_el1.${mesh_ext}"/>
             </geometry>
             <material name="arm0.link_el1">
@@ -162,5 +162,5 @@
             <origin xyz="0 0 0" rpy="0 0 0"/>
             <geometry>
-                <mesh filename="package://$(var mesh_pkg)/meshes/arm/arm0.link_wr0.$(var mesh_ext)"/>
+                <mesh filename="package://${mesh_pkg}/meshes/arm/arm0.link_wr0.${mesh_ext}"/>
             </geometry>
             <material name="arm0.link_wr0">
@@ -189,5 +189,5 @@
             <origin xyz="0 0 0" rpy="0 0 0"/>
             <geometry>
-                <mesh filename="package://$(var mesh_pkg)/meshes/arm/arm0.link_wr1.$(var mesh_ext)"/>
+                <mesh filename="package://${mesh_pkg}/meshes/arm/arm0.link_wr1.${mesh_ext}"/>
             </geometry>
             <material name="arm0.link_wr1">
@@ -223,5 +223,5 @@
             <origin xyz="0 0 0" rpy="0 0 0"/>
             <geometry>
-                <mesh filename="package://$(var mesh_pkg)/meshes/arm/arm0.link_fngr.$(var mesh_ext)"/>
+                <mesh filename="package://${mesh_pkg}/meshes/arm/arm0.link_fngr.${mesh_ext}"/>
             </geometry>
             <material name="arm0.link_fngr">
