Commit message: make propriety pkg name and extension args

File: spot_description/urdf/arm/spot_arm.urdf.xacro (robot description, xacro)
@@ -4,7 +4,8 @@
     <xacro:arg name="has_realsense" default="False" />
     <xacro:arg name="use_proprietary_meshes" default="false" />
+    <xacro:arg name="proprietary_pkg" default="spot_propreity_description" />
     <xacro:arg name="proprietary_format" default="dae" />
     <!-- Determine mesh source -->
-  <xacro:property name="mesh_pkg" value="$(eval 'spot_propriety_description' if use_proprietary_meshes else 'spot_description')"/>
+  <xacro:property name="mesh_pkg" value="$(eval proprietary_pkg if use_proprietary_meshes else 'spot_description')"/>
   <xacro:property name="mesh_ext" value="$(eval proprietary_format if use_proprietary_meshes else 'obj')" />
     <link name="${name}_base_link">

File: spot_description/urdf/spot.urdf.xacro (robot description, xacro)
@@ -11,5 +11,10 @@
     <xacro:arg name="kinematic_model" default="none"/>
     <xacro:arg name="use_proprietary_meshes" default="false" />
+    <xacro:arg name="proprietary_pkg" default="spot_propreity_description" />
+    <xacro:arg name="proprietary_format" default="dae" />
     <xacro:property name="kinematic_model" value="$(arg kinematic_model)"/>
+    <!-- Determine mesh source -->
+    <xacro:property name="mesh_pkg" value="$(eval proprietary_pkg if use_proprietary_meshes else 'spot_description')"/>
+    <xacro:property name="mesh_ext" value="$(eval proprietary_format if use_proprietary_meshes else 'obj')" />
     <xacro:unless value="${kinematic_model == 'none'}">
         <link name="base_footprint"/>
@@ -596,10 +601,10 @@
             <visual>
               <geometry>
-                <mesh filename="package://spot_propriety_description/meshes/accessories/eap_lidar.stl"/>
+		<mesh filename="package://${mesh_pkg}/meshes/accessories/eap_lidar.${mesh_ext}"/>
               </geometry>
             </visual>
             <collision>
               <geometry>
-                <mesh filename="package://spot_propriety_description/meshes/accessories/eap_lidar.stl"/>
+                <mesh filename="package://${mesh_pkg}/meshes/accessories/eap_lidar.${mesh_ext}"/>
               </geometry>
             </collision>
@@ -636,10 +641,10 @@
             <visual>
               <geometry>
-                <mesh filename="package://spot_propriety_description/meshes/accessories/EAP2.dae" />
+                <mesh filename="package://${mesh_pkg}/meshes/accessories/EAP2.${mesh_ext}" />
               </geometry>
             </visual>
             <collision>
               <geometry>
-                <mesh filename="package://spot_propriety_description/meshes/accessories/EAP2_compressed.stl" />
+                <mesh filename="package://${mesh_pkg}/meshes/accessories/EAP2.${mesh_ext}" />
               </geometry>
             </collision>

Commit message: lower gripper joint limit to allow numerical drift

File: spot_description/urdf/arm/spot_arm.urdf.xacro (robot description, xacro)
@@ -258,5 +258,5 @@
         <parent link="${name}_wrist_roll"/>
         <child link="${name}_fingers"/>
-        <limit effort="1000" velocity="1000.00" lower="-1.57" upper="0.0"/>
+        <limit effort="1000" velocity="1000.00" lower="-1.58" upper="0.0"/>
     </joint>
     <link name="${name}.link_wr1"/>
