Commit message: Added arm to robot description and visualization.

File: spot_description/urdf/spot_with_arm.urdf.xacro (robot description, xacro)
@@ -1,7 +1,9 @@
 <?xml version="1.0" ?>
 <robot name="spot" xmlns:xacro="http://www.ros.org/wiki/xacro">
-    <!-- We do not specify links for the cameras in the URDF. Instead, transforms for those are
-         published by the driver (see spot_driver package) during runtime, so that the transforms
-         include calibration adjustments. -->
+    <!--
+        We do not specify links for the cameras in the URDF. Instead, transforms for those are
+        published by the driver (see spot_driver package), so that the transforms can
+        include calibration adjustments.
+    -->
     <link name="body">
         <visual>
@@ -262,5 +264,8 @@
         <limit effort="1000" velocity="1000.00" lower="-2.7929" upper="-0.257725" />
     </joint>
-    <!-- Optional custom includes. -->
-    <xacro:include filename="$(optenv SPOT_URDF_EXTRAS empty.urdf)" />
+    <xacro:include filename="$(find spot_description)/urdf/arm/spot_arm_include.urdf.xacro"/>
+    <xacro:spot_arm
+        name="arm" base_frame="front_rail"
+        x="0.06" y="0.0" z="0.0"
+        roll="0.0" pitch="0.0" yaw="0.0"/>
 </robot>

Commit message: Friendly link names for Spot arm.

File: spot_description/urdf/spot_with_arm.urdf.xacro (robot description, xacro)
@@ -265,10 +265,10 @@
     </joint>
     <!-- Spot Arm -->
-    <xacro:include filename="$(find spot_description)/urdf/arm/spot_arm_include.urdf.xacro"/>
-    <xacro:spot_arm name="arm"/>
+    <xacro:include filename="$(find spot_description)/urdf/arm/spot_arm.urdf.xacro"/>
+    <xacro:spot_arm name="arm0"/>
     <joint name="arm0_mount" type="fixed">
         <origin xyz="0.292 0 0.188" rpy="0 0 0"/>
         <parent link="base_link"/>
-        <child link="arm0.base_link"/>
+        <child link="arm0_base_link"/>
     </joint>
 </robot>

Commit message: Removed unnecessary copy and paste

File: spot_description/urdf/spot_with_arm.urdf.xacro (robot description, xacro)
@@ -1,267 +1,5 @@
 <?xml version="1.0" ?>
 <robot name="spot" xmlns:xacro="http://www.ros.org/wiki/xacro">
-    <!--
-        We do not specify links for the cameras in the URDF. Instead, transforms for those are
-        published by the driver (see spot_driver package), so that the transforms can
-        include calibration adjustments.
-    -->
-    <link name="body">
-        <visual>
-            <geometry>
-                <mesh filename="package://spot_description/meshes/body/body.dae" />
-            </geometry>
-        </visual>
-        <collision>
-            <geometry>
-                <mesh filename="package://spot_description/meshes/body/body_collision.stl" />
-            </geometry>
-        </collision>
-    </link>
-    <link name="base_link"/>
-    <joint name="base_link_joint" type="fixed">
-        <origin xyz="0 0 0" rpy="0 0 0" />
-        <parent link="body" />
-        <child link="base_link" />
-    </joint>
-    <link name="front_rail"/>
-    <joint name="front_rail_joint" type="fixed">
-        <origin xyz="0.223 0 0.0805" rpy="0 0 0" />
-        <parent link="body" />
-        <child link="front_rail" />
-    </joint>
-    <link name="rear_rail"/>
-    <joint name="rear_rail_joint" type="fixed">
-        <origin xyz="-0.223 0 0.0805" rpy="0 0 0" />
-        <parent link="body" />
-        <child link="rear_rail" />
-    </joint>
-    <link name="front_left_hip">
-        <visual>
-            <geometry>
-                <mesh filename="package://spot_description/meshes/body/front_left_hip.dae" />
-            </geometry>
-        </visual>
-        <collision>
-            <geometry>
-                <mesh filename="package://spot_description/meshes/body/front_left_hip_collision.stl" />
-            </geometry>
-        </collision>
-    </link>
-    <joint name="front_left_hip_x" type="revolute">
-        <origin xyz="0.29785 0.05500 0.00000" rpy="0 0 0" />
-        <axis xyz="1 0 0" />
-        <parent link="body" />
-        <child link="front_left_hip" />
-        <limit effort="1000" velocity="1000.00" lower="-0.78539816339744827899" upper="0.78539816339744827899" />
-    </joint>
-    <link name="front_left_upper_leg">
-        <visual>
-            <geometry>
-                <mesh filename="package://spot_description/meshes/body/front_left_upper_leg.dae" />
-            </geometry>
-        </visual>
-        <collision>
-            <geometry>
-                <mesh filename="package://spot_description/meshes/body/front_left_upper_leg_collision.stl" />
-            </geometry>
-        </collision>
-    </link>
-    <joint name="front_left_hip_y" type="revolute">
-        <origin xyz="0.0 0.110945 0.0" rpy="0 0 0" />
-        <axis xyz="0 1 0" />
-        <parent link="front_left_hip" />
-        <child link="front_left_upper_leg" />
-        <limit effort="1000" velocity="1000.00" lower="-0.89884456477707963539" upper="2.2951079663725435509" />
-    </joint>
-    <link name="front_left_lower_leg">
-        <visual>
-            <geometry>
-                <mesh filename="package://spot_description/meshes/body/front_left_lower_leg.dae" />
-            </geometry>
-        </visual>
-        <collision>
-            <geometry>
-                <mesh filename="package://spot_description/meshes/body/front_left_lower_leg_collision.stl" />
-            </geometry>
-        </collision>
-    </link>
-    <joint name="front_left_knee" type="revolute">
-        <origin xyz="0.025 0.000 -0.3205" rpy="0 0 0" />
-        <axis xyz="0 1 0" />
-        <parent link="front_left_upper_leg" />
-        <child link="front_left_lower_leg" />
-        <limit effort="1000" velocity="1000.00" lower="-2.7929" upper="-0.254801" />
-    </joint>
-    <link name="front_right_hip">
-        <visual>
-            <geometry>
-                <mesh filename="package://spot_description/meshes/body/front_right_hip.dae" />
-            </geometry>
-        </visual>
-        <collision>
-            <geometry>
-                <mesh filename="package://spot_description/meshes/body/front_right_hip_collision.stl" />
-            </geometry>
-        </collision>
-    </link>
-    <joint name="front_right_hip_x" type="revolute">
-        <origin xyz="0.29785 -0.05500 0.00000" rpy="0 0 0" />
-        <axis xyz="1 0 0" />
-        <parent link="body" />
-        <child link="front_right_hip" />
-        <limit effort="1000" velocity="1000.00" lower="-0.78539816339744827899" upper="0.78539816339744827899" />
-    </joint>
-    <link name="front_right_upper_leg">
-        <visual>
-            <geometry>
-                <mesh filename="package://spot_description/meshes/body/front_right_upper_leg.dae" />
-            </geometry>
-        </visual>
-        <collision>
-            <geometry>
-                <mesh filename="package://spot_description/meshes/body/front_right_upper_leg_collision.stl" />
-            </geometry>
-        </collision>
-    </link>
-    <joint name="front_right_hip_y" type="revolute">
-        <origin xyz="0.0 -0.110945 0.0" rpy="0 0 0" />
-        <axis xyz="0 1 0" />
-        <parent link="front_right_hip" />
-        <child link="front_right_upper_leg" />
-        <limit effort="1000" velocity="1000.00" lower="-0.89884456477707963539" upper="2.2951079663725435509" />
-    </joint>
-    <link name="front_right_lower_leg">
-        <visual>
-            <geometry>
-                <mesh filename="package://spot_description/meshes/body/front_right_lower_leg.dae" />
-            </geometry>
-        </visual>
-        <collision>
-            <geometry>
-                <mesh filename="package://spot_description/meshes/body/front_right_lower_leg_collision.stl" />
-            </geometry>
-        </collision>
-    </link>
-    <joint name="front_right_knee" type="revolute">
-        <origin xyz="0.025 0.000 -0.3205" rpy="0 0 0" />
-        <axis xyz="0 1 0" />
-        <parent link="front_right_upper_leg" />
-        <child link="front_right_lower_leg" />
-        <limit effort="1000" velocity="1000.00" lower="-2.7929" upper="-0.247563" />
-    </joint>
-    <link name="rear_left_hip">
-        <visual>
-            <geometry>
-                <mesh filename="package://spot_description/meshes/body/rear_left_hip.dae" />
-            </geometry>
-        </visual>
-        <collision>
-            <geometry>
-                <mesh filename="package://spot_description/meshes/body/rear_left_hip_collision.stl" />
-            </geometry>
-        </collision>
-    </link>
-    <joint name="rear_left_hip_x" type="revolute">
-        <origin xyz="-0.29785 0.05500 0.00000" rpy="0 0 0" />
-        <axis xyz="1 0 0" />
-        <parent link="body" />
-        <child link="rear_left_hip" />
-        <limit effort="1000" velocity="1000.00" lower="-0.78539816339744827899" upper="0.78539816339744827899" />
-    </joint>
-    <link name="rear_left_upper_leg">
-        <visual>
-            <geometry>
-                <mesh filename="package://spot_description/meshes/body/rear_left_upper_leg.dae" />
-            </geometry>
-        </visual>
-        <collision>
-            <geometry>
-                <mesh filename="package://spot_description/meshes/body/rear_left_upper_leg_collision.stl" />
-            </geometry>
-        </collision>
-    </link>
-    <joint name="rear_left_hip_y" type="revolute">
-        <origin xyz="0.0 0.110945 0.0" rpy="0 0 0" />
-        <axis xyz="0 1 0" />
-        <parent link="rear_left_hip" />
-        <child link="rear_left_upper_leg" />
-        <limit effort="1000" velocity="1000.00" lower="-0.89884456477707963539" upper="2.2951079663725435509" />
-    </joint>
-    <link name="rear_left_lower_leg">
-        <visual>
-            <geometry>
-                <mesh filename="package://spot_description/meshes/body/rear_left_lower_leg.dae" />
-            </geometry>
-        </visual>
-        <collision>
-            <geometry>
-                <mesh filename="package://spot_description/meshes/body/rear_left_lower_leg_collision.stl" />
-            </geometry>
-        </collision>
-    </link>
-    <joint name="rear_left_knee" type="revolute">
-        <origin xyz="0.025 0.000 -0.3205" rpy="0 0 0" />
-        <axis xyz="0 1 0" />
-        <parent link="rear_left_upper_leg" />
-        <child link="rear_left_lower_leg" />
-        <limit effort="1000" velocity="1000.00" lower="-2.7929" upper="-0.267153" />
-    </joint>
-    <link name="rear_right_hip">
-        <visual>
-            <geometry>
-                <mesh filename="package://spot_description/meshes/body/rear_right_hip.dae" />
-            </geometry>
-        </visual>
-        <collision>
-            <geometry>
-                <mesh filename="package://spot_description/meshes/body/rear_right_hip_collision.stl" />
-            </geometry>
-        </collision>
-    </link>
-    <joint name="rear_right_hip_x" type="revolute">
-        <origin xyz="-0.29785 -0.05500 0.00000" rpy="0 0 0" />
-        <axis xyz="1 0 0" />
-        <parent link="body" />
-        <child link="rear_right_hip" />
-        <limit effort="1000" velocity="1000.00" lower="-0.78539816339744827899" upper="0.78539816339744827899" />
-    </joint>
-    <link name="rear_right_upper_leg">
-        <visual>
-            <geometry>
-                <mesh filename="package://spot_description/meshes/body/rear_right_upper_leg.dae" />
-            </geometry>
-        </visual>
-        <collision>
-            <geometry>
-                <mesh filename="package://spot_description/meshes/body/rear_right_upper_leg_collision.stl" />
-            </geometry>
-        </collision>
-    </link>
-    <joint name="rear_right_hip_y" type="revolute">
-        <origin xyz="0.0 -0.110945 0.0" rpy="0 0 0" />
-        <axis xyz="0 1 0" />
-        <parent link="rear_right_hip" />
-        <child link="rear_right_upper_leg" />
-        <limit effort="1000" velocity="1000.00" lower="-0.89884456477707963539" upper="2.2951079663725435509" />
-    </joint>
-    <link name="rear_right_lower_leg">
-        <visual>
-            <geometry>
-                <mesh filename="package://spot_description/meshes/body/rear_right_lower_leg.dae" />
-            </geometry>
-        </visual>
-        <collision>
-            <geometry>
-                <mesh filename="package://spot_description/meshes/body/rear_right_lower_leg_collision.stl" />
-            </geometry>
-        </collision>
-    </link>
-    <joint name="rear_right_knee" type="revolute">
-        <origin xyz="0.025 0.000 -0.3205" rpy="0 0 0" />
-        <axis xyz="0 1 0" />
-        <parent link="rear_right_upper_leg" />
-        <child link="rear_right_lower_leg" />
-        <limit effort="1000" velocity="1000.00" lower="-2.7929" upper="-0.257725" />
-    </joint>
+    <xacro:include filename="$(find spot_description)/urdf/spot.urdf.xacro"/>
     <!-- Spot Arm -->
     <xacro:include filename="$(find spot_description)/urdf/arm/spot_arm.urdf.xacro"/>
