Commit message: Converted realsense mount to a xacro:macro

File: spot_description/urdf/realsense_mount.urdf.xacro (robot description, xacro)
@@ -1,4 +1,5 @@
 <robot xmlns:xacro="http://www.ros.org/wiki/xacro">
     <!-- Original STLs at https://utexas.app.box.com/folder/226702516436 -->
+    <xacro:macro name = "realsense_mount" params = "*origin parent:=arm0_wrist_roll">
     <link name = "realsense_mount_chin">
         <visual name = "realsense_mount_chin_visual">
@@ -14,7 +15,7 @@
     </link>
     <joint name = "joint_chin_to_arm" type = "fixed">
-        <parent link = "arm0_wrist_roll"/>
+        <parent link = "${parent}"/>
         <child  link = "realsense_mount_chin"/>
-        <origin xyz = "0.145 0 -0.06" rpy = "3.1416 0 -1.57"/>
+        <xacro:insert_block name="origin" />
     </joint>
     <link name = "realsense_mount_chin_top">
@@ -73,3 +74,4 @@
         <origin xyz="0 0.0125 0.01" rpy = "0 -1.57 1.57"/>
     </xacro:sensor_d435>
+    </xacro:macro>
 </robot>

File: spot_description/urdf/spot.urdf.xacro (robot description, xacro)
@@ -539,4 +539,7 @@
     </xacro:if>
     <xacro:include filename="$(find spot_description)/urdf/realsense_mount.urdf.xacro"/>
+    <xacro:realsense_mount parent = "arm0_wrist_roll">
+        <origin xyz = "0.145 0 -0.06" rpy = "3.1416 0 -1.57"/>
+    </xacro:realsense_mount>
     <!-- Optional custom includes. -->
     <xacro:include filename="$(optenv SPOT_URDF_EXTRAS empty.urdf)" />
