Commit message: Incorporate Velodyne VLP-16.

File: spot_description/urdf/spot.urdf.xacro (robot description, xacro)
@@ -4,4 +4,6 @@
          published by the driver (see spot_driver package) during runtime, so that the transforms
          include calibration adjustments. -->
+    <xacro:arg name="has_arm" default="false" />
+    <xacro:arg name="has_velodyne" default="false" />
     <link name="body">
         <visual>
@@ -262,4 +264,21 @@
         <limit effort="1000" velocity="1000.00" lower="-2.7929" upper="-0.257725" />
     </joint>
+    <!-- Spot Arm -->
+    <xacro:if value="$(arg has_arm)">
+        <xacro:include filename="$(find spot_description)/urdf/arm/spot_arm.urdf.xacro"/>
+        <xacro:spot_arm name="arm0"/>
+        <joint name="arm0_mount" type="fixed">
+            <origin xyz="0.292 0 0.188" rpy="0 0 0"/>
+            <parent link="base_link"/>
+            <child link="arm0_base_link"/>
+        </joint>
+    </xacro:if>
+    <!-- Spot Arm -->
+    <xacro:if value="$(arg has_velodyne)">
+        <xacro:include filename="$(find velodyne_description)/urdf/VLP-16.urdf.xacro"/>
+        <xacro:VLP-16 parent="base_link" name="velodyne">
+            <origin xyz="0 0 1.0" rpy="0 0 0" />
+        </xacro:VLP-16>
+    </xacro:if>
     <!-- Optional custom includes. -->
     <xacro:include filename="$(optenv SPOT_URDF_EXTRAS empty.urdf)" />

Commit message: Adjust Velodyne URDF position.

File: spot_description/urdf/spot.urdf.xacro (robot description, xacro)
@@ -278,5 +278,5 @@
         <xacro:include filename="$(find velodyne_description)/urdf/VLP-16.urdf.xacro"/>
         <xacro:VLP-16 parent="base_link" name="velodyne">
-            <origin xyz="0 0 1.0" rpy="0 0 0" />
+            <origin xyz="-0.24 0 0.16" rpy="0 0 0" />
         </xacro:VLP-16>
     </xacro:if>

Commit message: Adding dynamics to URDF for simulation.

File: spot_description/urdf/spot.urdf.xacro (robot description, xacro)
@@ -17,4 +17,8 @@
             </geometry>
         </collision>
+        <inertial>
+             <mass value="16.25" />
+             <inertia  ixx="0.085" ixy="0.0"  ixz="0.0"  iyy="1.045"  iyz="0.0"  izz="1.042" />
+    	</inertial>
     </link>
     <link name="base_link"/>
@@ -47,4 +51,8 @@
             </geometry>
         </collision>
+        <inertial>
+            <mass value="1.5" />
+    	    <inertia  ixx="0.0605" ixy="0.0"  ixz="0.0"  iyy="0.0"  iyz="0.0"  izz="0.0" />
+    	</inertial>
     </link>
     <joint name="front_left_hip_x" type="revolute">
@@ -53,6 +61,17 @@
         <parent link="body" />
         <child link="front_left_hip" />
+        <dynamics damping="0.1" friction="0.1"/>
         <limit effort="1000" velocity="1000.00" lower="-0.78539816339744827899" upper="0.78539816339744827899" />
     </joint>
+    <transmission name="front_left_hip_x_trans">
+	    <type>transmission_interface/SimpleTransmission</type>
+	    <joint name="front_left_hip_x">
+            <hardwareInterface>EffortJointInterface</hardwareInterface>
+        </joint>
+	    <actuator name="front_left_hip_x">
+          	<mechanicalReduction>50</mechanicalReduction>
+          	<hardwareInterface>EffortJointInterface</hardwareInterface>
+	    </actuator>
+    </transmission>
     <link name="front_left_upper_leg">
         <visual>
@@ -66,4 +85,8 @@
             </geometry>
         </collision>
+        <inertial>
+            <mass value="1.5" />
+    	    <inertia  ixx="0.0" ixy="0.0"  ixz="0.0"  iyy="0.05"  iyz="0.0"  izz="0.0" />
+    	</inertial>
     </link>
     <joint name="front_left_hip_y" type="revolute">
@@ -72,6 +95,17 @@
         <parent link="front_left_hip" />
         <child link="front_left_upper_leg" />
+        <dynamics damping="0.1" friction="0.1"/>
         <limit effort="1000" velocity="1000.00" lower="-0.89884456477707963539" upper="2.2951079663725435509" />
     </joint>
+    <transmission name="front_left_hip_y_trans">
+        <type>transmission_interface/SimpleTransmission</type>
+        <joint name="front_left_hip_y">
+            <hardwareInterface>EffortJointInterface</hardwareInterface>
+        </joint>
+        <actuator name="front_left_hip_y">
+            <mechanicalReduction>50</mechanicalReduction>
+            <hardwareInterface>EffortJointInterface</hardwareInterface>
+        </actuator>
+    </transmission>
     <link name="front_left_lower_leg">
         <visual>
@@ -85,4 +119,8 @@
             </geometry>
         </collision>
+        <inertial>
+            <mass value="1.0" />
+    	    <inertia  ixx="0.0" ixy="0.0"  ixz="0.0"  iyy="0.045"  iyz="0.0"  izz="0.0" />
+    	</inertial>
     </link>
     <joint name="front_left_knee" type="revolute">
@@ -91,6 +129,30 @@
         <parent link="front_left_upper_leg" />
         <child link="front_left_lower_leg" />
+        <dynamics damping="0.1" friction="0.1"/>
         <limit effort="1000" velocity="1000.00" lower="-2.7929" upper="-0.254801" />
     </joint>
+    <!-- Contact Sensor -->
+    <gazebo reference="front_left_lower_leg">
+        <sensor name="front_left_lower_leg_contactsensor_sensor" type="contact">
+        <always_on>true</always_on>
+        <contact>
+            <collision>front_left_lower_leg_fixed_joint_lump__front_bump_sensor_collision</collision>
+        </contact>
+        <plugin filename="libgazebo_ros_bumper.so" name="front_left_lower_leg_plugin">
+            <bumperTopicName>front_left_lower_leg_contact</bumperTopicName>
+            <frameName>front_left_lower_leg</frameName>
+        </plugin>
+        </sensor>
+    </gazebo>
+    <transmission name="front_left_knee_trans">
+	  <type>transmission_interface/SimpleTransmission</type>
+	  <joint name="front_left_knee">
+          	<hardwareInterface>EffortJointInterface</hardwareInterface>
+      </joint>
+	  <actuator name="front_left_knee">
+          	<mechanicalReduction>50</mechanicalReduction>
+          	<hardwareInterface>EffortJointInterface</hardwareInterface>
+	  </actuator>
+    </transmission>
     <link name="front_right_hip">
         <visual>
@@ -104,4 +166,8 @@
             </geometry>
         </collision>
+        <inertial>
+            <mass value="1.5" />
+    	    <inertia  ixx="0.0605" ixy="0.0"  ixz="0.0"  iyy="0.0"  iyz="0.0"  izz="0.0" />
+    	</inertial>
     </link>
     <joint name="front_right_hip_x" type="revolute">
@@ -110,6 +176,17 @@
         <parent link="body" />
         <child link="front_right_hip" />
+        <dynamics damping="0.1" friction="0.1"/>
         <limit effort="1000" velocity="1000.00" lower="-0.78539816339744827899" upper="0.78539816339744827899" />
     </joint>
+    <transmission name="front_right_hip_x_trans">
+	  <type>transmission_interface/SimpleTransmission</type>
+	  <joint name="front_right_hip_x">
+          	<hardwareInterface>EffortJointInterface</hardwareInterface>
+      </joint>
+	  <actuator name="front_right_hip_x">
+          	<mechanicalReduction>50</mechanicalReduction>
+          	<hardwareInterface>EffortJointInterface</hardwareInterface>
+	  </actuator>
+    </transmission>
     <link name="front_right_upper_leg">
         <visual>
@@ -123,4 +200,8 @@
             </geometry>
         </collision>
+        <inertial>
+            <mass value="1.5" />
+    	    <inertia  ixx="0.0" ixy="0.0"  ixz="0.0"  iyy="0.05"  iyz="0.0"  izz="0.0" />
+    	</inertial>
     </link>
     <joint name="front_right_hip_y" type="revolute">
@@ -129,6 +210,17 @@
         <parent link="front_right_hip" />
         <child link="front_right_upper_leg" />
+        <dynamics damping="0.1" friction="0.1"/>
         <limit effort="1000" velocity="1000.00" lower="-0.89884456477707963539" upper="2.2951079663725435509" />
     </joint>
+    <transmission name="front_right_hip_y_trans">
+        <type>transmission_interface/SimpleTransmission</type>
+        <joint name="front_right_hip_y">
+            <hardwareInterface>EffortJointInterface</hardwareInterface>
+        </joint>
+        <actuator name="front_right_hip_y">
+            <mechanicalReduction>50</mechanicalReduction>
+            <hardwareInterface>EffortJointInterface</hardwareInterface>
+        </actuator>
+    </transmission>
     <link name="front_right_lower_leg">
         <visual>
@@ -142,4 +234,8 @@
             </geometry>
         </collision>
+        <inertial>
+            <mass value="1.0" />
+    	    <inertia  ixx="0.0" ixy="0.0"  ixz="0.0"  iyy="0.045"  iyz="0.0"  izz="0.0" />
+    	</inertial>
     </link>
     <joint name="front_right_knee" type="revolute">
@@ -148,6 +244,30 @@
         <parent link="front_right_upper_leg" />
         <child link="front_right_lower_leg" />
+        <dynamics damping="0.1" friction="0.1"/>
         <limit effort="1000" velocity="1000.00" lower="-2.7929" upper="-0.247563" />
     </joint>
+     <!-- Contact Sensor -->
+    <gazebo reference="front_right_lower_leg">
+        <sensor name="front_right_lower_leg_contactsensor_sensor" type="contact">
+        <always_on>true</always_on>
+        <contact>
+            <collision>front_right_lower_leg_fixed_joint_lump__front_bump_sensor_collision</collision>
+        </contact>
+        <plugin filename="libgazebo_ros_bumper.so" name="front_right_lower_leg_plugin">
+            <bumperTopicName>front_right_lower_leg_contact</bumperTopicName>
+            <frameName>front_right_lower_leg</frameName>
+        </plugin>
+        </sensor>
+    </gazebo>
+    <transmission name="front_right_knee_trans">
+        <type>transmission_interface/SimpleTransmission</type>
+        <joint name="front_right_knee">
+            <hardwareInterface>EffortJointInterface</hardwareInterface>
+        </joint>
+        <actuator name="front_right_knee">
+            <mechanicalReduction>50</mechanicalReduction>
+            <hardwareInterface>EffortJointInterface</hardwareInterface>
+        </actuator>
+    </transmission>
     <link name="rear_left_hip">
         <visual>
@@ -161,4 +281,8 @@
             </geometry>
         </collision>
+        <inertial>
+            <mass value="1.5" />
+    	    <inertia  ixx="0.0605" ixy="0.0"  ixz="0.0"  iyy="0.0"  iyz="0.0"  izz="0.0" />
+    	</inertial>
     </link>
     <joint name="rear_left_hip_x" type="revolute">
@@ -167,6 +291,17 @@
         <parent link="body" />
         <child link="rear_left_hip" />
+        <dynamics damping="0.1" friction="0.1"/>
         <limit effort="1000" velocity="1000.00" lower="-0.78539816339744827899" upper="0.78539816339744827899" />
     </joint>
+    <transmission name="rear_left_hip_x_trans">
+        <type>transmission_interface/SimpleTransmission</type>
+        <joint name="rear_left_hip_x">
+            <hardwareInterface>EffortJointInterface</hardwareInterface>
+        </joint>
+        <actuator name="rear_left_hip_x">
+            <mechanicalReduction>50</mechanicalReduction>
+            <hardwareInterface>EffortJointInterface</hardwareInterface>
+        </actuator>
+    </transmission>
     <link name="rear_left_upper_leg">
         <visual>
@@ -180,4 +315,8 @@
             </geometry>
         </collision>
+        <inertial>
+           <mass value="1.5" />
+    	   <inertia  ixx="0.0" ixy="0.0"  ixz="0.0"  iyy="0.05"  iyz="0.0"  izz="0.0" />
+    	</inertial>
     </link>
     <joint name="rear_left_hip_y" type="revolute">
@@ -186,6 +325,17 @@
         <parent link="rear_left_hip" />
         <child link="rear_left_upper_leg" />
+        <dynamics damping="0.1" friction="0.1"/>
         <limit effort="1000" velocity="1000.00" lower="-0.89884456477707963539" upper="2.2951079663725435509" />
     </joint>
+    <transmission name="rear_left_hip_y_trans">
+        <type>transmission_interface/SimpleTransmission</type>
+        <joint name="rear_left_hip_y">
+            <hardwareInterface>EffortJointInterface</hardwareInterface>
+        </joint>
+        <actuator name="rear_left_hip_y">
+            <mechanicalReduction>50</mechanicalReduction>
+            <hardwareInterface>EffortJointInterface</hardwareInterface>
+        </actuator>
+    </transmission>
     <link name="rear_left_lower_leg">
         <visual>
@@ -199,4 +349,8 @@
             </geometry>
         </collision>
+        <inertial>
+            <mass value="1.0" />
+    	    <inertia  ixx="0.0" ixy="0.0"  ixz="0.0"  iyy="0.045"  iyz="0.0"  izz="0.0" />
+    	</inertial>
     </link>
     <joint name="rear_left_knee" type="revolute">
@@ -205,6 +359,30 @@
         <parent link="rear_left_upper_leg" />
         <child link="rear_left_lower_leg" />
+        <dynamics damping="0.1" friction="0.1"/>
         <limit effort="1000" velocity="1000.00" lower="-2.7929" upper="-0.267153" />
     </joint>
+    <!-- Contact Sensor -->
+    <gazebo reference="rear_left_lower_leg">
+        <sensor name="rear_left_lower_leg_contactsensor_sensor" type="contact">
+        <always_on>true</always_on>
+        <contact>
+            <collision>rear_left_lower_leg_fixed_joint_lump__rear_bump_sensor_collision</collision>
+        </contact>
+        <plugin filename="libgazebo_ros_bumper.so" name="rear_left_lower_leg_plugin">
+            <bumperTopicName>rear_left_lower_leg_contact</bumperTopicName>
+            <frameName>rear_left_lower_leg</frameName>
+        </plugin>
+        </sensor>
+    </gazebo>
+    <transmission name="rear_left_knee_trans">
+        <type>transmission_interface/SimpleTransmission</type>
+        <joint name="rear_left_knee">
+             <hardwareInterface>EffortJointInterface</hardwareInterface>
+        </joint>
+        <actuator name="rear_left_knee">
+            <mechanicalReduction>50</mechanicalReduction>
+            <hardwareInterface>EffortJointInterface</hardwareInterface>
+        </actuator>
+    </transmission>
     <link name="rear_right_hip">
         <visual>
@@ -218,4 +396,8 @@
             </geometry>
         </collision>
+        <inertial>
+            <mass value="1.5" />
+    	    <inertia  ixx="0.0605" ixy="0.0"  ixz="0.0"  iyy="0.0"  iyz="0.0"  izz="0.0" />
+    	</inertial>
     </link>
     <joint name="rear_right_hip_x" type="revolute">
@@ -224,6 +406,17 @@
         <parent link="body" />
         <child link="rear_right_hip" />
+        <dynamics damping="0.1" friction="0.1"/>
         <limit effort="1000" velocity="1000.00" lower="-0.78539816339744827899" upper="0.78539816339744827899" />
     </joint>
+    <transmission name="rear_right_hip_x_trans">
+        <type>transmission_interface/SimpleTransmission</type>
+        <joint name="rear_right_hip_x">
+            <hardwareInterface>EffortJointInterface</hardwareInterface>
+        </joint>
+        <actuator name="rear_right_hip_x">
+            <mechanicalReduction>50</mechanicalReduction>
+            <hardwareInterface>EffortJointInterface</hardwareInterface>
+        </actuator>
+    </transmission>
     <link name="rear_right_upper_leg">
         <visual>
@@ -237,4 +430,8 @@
             </geometry>
         </collision>
+        <inertial>
+            <mass value="1.5" />
+    	    <inertia  ixx="0.0" ixy="0.0"  ixz="0.0"  iyy="0.05"  iyz="0.0"  izz="0.0" />
+    	</inertial>
     </link>
     <joint name="rear_right_hip_y" type="revolute">
@@ -243,6 +440,17 @@
         <parent link="rear_right_hip" />
         <child link="rear_right_upper_leg" />
+        <dynamics damping="0.1" friction="0.1"/>
         <limit effort="1000" velocity="1000.00" lower="-0.89884456477707963539" upper="2.2951079663725435509" />
     </joint>
+    <transmission name="rear_right_hip_y_trans">
+        <type>transmission_interface/SimpleTransmission</type>
+        <joint name="rear_right_hip_y">
+            <hardwareInterface>EffortJointInterface</hardwareInterface>
+            </joint>
+        <actuator name="rear_right_hip_y">
+            <mechanicalReduction>50</mechanicalReduction>
+            <hardwareInterface>EffortJointInterface</hardwareInterface>
+        </actuator>
+    </transmission>
     <link name="rear_right_lower_leg">
         <visual>
@@ -256,4 +464,8 @@
             </geometry>
         </collision>
+        <inertial>
+            <mass value="1.0" />
+    	    <inertia  ixx="0.0" ixy="0.0"  ixz="0.0"  iyy="0.045"  iyz="0.0"  izz="0.0" />
+    	</inertial>
     </link>
     <joint name="rear_right_knee" type="revolute">
@@ -262,6 +474,33 @@
         <parent link="rear_right_upper_leg" />
         <child link="rear_right_lower_leg" />
+        <dynamics damping="0.1" friction="0.1"/>
         <limit effort="1000" velocity="1000.00" lower="-2.7929" upper="-0.257725" />
     </joint>
+    <!-- Contact Sensor -->
+    <gazebo reference="rear_right_lower_leg">
+        <sensor name="rear_right_lower_leg_contactsensor_sensor" type="contact">
+        <always_on>true</always_on>
+        <contact>
+            <collision>rear_right_lower_leg_fixed_joint_lump__rear_bump_sensor_collision</collision>
+        </contact>
+        <plugin filename="libgazebo_ros_bumper.so" name="rear_right_lower_leg_plugin">
+            <bumperTopicName>rear_right_lower_leg_contact</bumperTopicName>
+            <frameName>rear_right_lower_leg</frameName>
+        </plugin>
+        </sensor>
+    </gazebo>
+    <transmission name="rear_right_knee_trans">
+        <type>transmission_interface/SimpleTransmission</type>
+        <joint name="rear_right_knee">
+            <hardwareInterface>EffortJointInterface</hardwareInterface>
+            </joint>
+        <actuator name="rear_right_knee">
+            <mechanicalReduction>50</mechanicalReduction>
+            <hardwareInterface>EffortJointInterface</hardwareInterface>
+        </actuator>
+    </transmission>
+    <gazebo>
+    	<plugin name="gazebo_ros_control" filename="libgazebo_ros_control.so"/>
+    </gazebo>
     <!-- Spot Arm -->
     <xacro:if value="$(arg has_arm)">

Commit message: Add some comments to URDF

File: spot_description/urdf/spot.urdf.xacro (robot description, xacro)
@@ -6,4 +6,5 @@
     <xacro:arg name="has_arm" default="false" />
     <xacro:arg name="has_velodyne" default="false" />
+    <!-- Fixed links -->
     <link name="body">
         <visual>
@@ -40,4 +41,5 @@
         <child link="rear_rail" />
     </joint>
+    <!-- Front Left -->
     <link name="front_left_hip">
         <visual>
@@ -132,5 +134,4 @@
         <limit effort="1000" velocity="1000.00" lower="-2.7929" upper="-0.254801" />
     </joint>
-    <!-- Contact Sensor -->
     <gazebo reference="front_left_lower_leg">
         <sensor name="front_left_lower_leg_contactsensor_sensor" type="contact">
@@ -155,4 +156,5 @@
 	  </actuator>
     </transmission>
+    <!-- Front Right -->
     <link name="front_right_hip">
         <visual>
@@ -247,5 +249,4 @@
         <limit effort="1000" velocity="1000.00" lower="-2.7929" upper="-0.247563" />
     </joint>
-     <!-- Contact Sensor -->
     <gazebo reference="front_right_lower_leg">
         <sensor name="front_right_lower_leg_contactsensor_sensor" type="contact">
@@ -270,4 +271,5 @@
         </actuator>
     </transmission>
+    <!-- Rear Left -->
     <link name="rear_left_hip">
         <visual>
@@ -362,5 +364,4 @@
         <limit effort="1000" velocity="1000.00" lower="-2.7929" upper="-0.267153" />
     </joint>
-    <!-- Contact Sensor -->
     <gazebo reference="rear_left_lower_leg">
         <sensor name="rear_left_lower_leg_contactsensor_sensor" type="contact">
@@ -385,4 +386,5 @@
         </actuator>
     </transmission>
+    <!-- Rear Right -->
     <link name="rear_right_hip">
         <visual>
@@ -477,5 +479,4 @@
         <limit effort="1000" velocity="1000.00" lower="-2.7929" upper="-0.257725" />
     </joint>
-    <!-- Contact Sensor -->
     <gazebo reference="rear_right_lower_leg">
         <sensor name="rear_right_lower_leg_contactsensor_sensor" type="contact">

Commit message: Improved launch files for description and viz.

File: spot_description/urdf/spot.urdf.xacro (robot description, xacro)
@@ -4,6 +4,6 @@
          published by the driver (see spot_driver package) during runtime, so that the transforms
          include calibration adjustments. -->
-    <xacro:arg name="has_arm" default="false" />
-    <xacro:arg name="has_velodyne" default="false" />
+    <xacro:arg name="has_arm" default="False" />
+    <xacro:arg name="has_eap" default="False" />
     <!-- Fixed links -->
     <link name="body">
@@ -514,6 +514,6 @@
         </joint>
     </xacro:if>
-    <!-- Spot Arm -->
-    <xacro:if value="$(arg has_velodyne)">
+    <!-- Spot Enhanced Autonomy package (EAP) -->
+    <xacro:if value="$(arg has_eap)">
         <xacro:include filename="$(find velodyne_description)/urdf/VLP-16.urdf.xacro"/>
         <xacro:VLP-16 parent="base_link" name="velodyne">

Commit message: Add EAP lidar mount to model.

File: spot_description/urdf/spot.urdf.xacro (robot description, xacro)
@@ -516,7 +516,24 @@
     <!-- Spot Enhanced Autonomy package (EAP) -->
     <xacro:if value="$(arg has_eap)">
+        <link name="lidar_assembly">
+            <visual>
+                <geometry>
+                    <mesh filename="package://spot_description/meshes/accessories/eap_lidar.stl" />
+                </geometry>
+            </visual>
+            <collision>
+                <geometry>
+                    <mesh filename="package://spot_description/meshes/accessories/eap_lidar.stl" />
+                </geometry>
+            </collision>
+        </link>
+        <joint name="lidar_mount" type="fixed">
+            <origin xyz="-0.03 0.0 0.0" rpy="0 0 0" />
+            <parent link="rear_rail" />
+            <child link="lidar_assembly" />
+        </joint>
         <xacro:include filename="$(find velodyne_description)/urdf/VLP-16.urdf.xacro"/>
-        <xacro:VLP-16 parent="base_link" name="velodyne">
-            <origin xyz="-0.24 0 0.16" rpy="0 0 0" />
+        <xacro:VLP-16 parent="lidar_assembly" name="velodyne">
+            <origin xyz="0.0 0 0.08" rpy="0 0 0" />
         </xacro:VLP-16>
     </xacro:if>
