Commit message: Change URDF filepath syntax to play nice with Gazebo.

File: spot_description/urdf/spot.urdf.xacro (robot description, xacro)
@@ -10,10 +10,10 @@
         <visual>
             <geometry>
-                <mesh filename="package://spot_description/meshes/body/body.dae" />
-            </geometry>
-        </visual>
-        <collision>
-            <geometry>
-                <mesh filename="package://spot_description/meshes/body/body_collision.stl" />
+                <mesh filename="file://$(find spot_description)/meshes/body/body.dae" />
+            </geometry>
+        </visual>
+        <collision>
+            <geometry>
+                <mesh filename="file://$(find spot_description)/meshes/body/body_collision.stl" />
             </geometry>
         </collision>
@@ -45,10 +45,10 @@
         <visual>
             <geometry>
-                <mesh filename="package://spot_description/meshes/body/front_left_hip.dae" />
-            </geometry>
-        </visual>
-        <collision>
-            <geometry>
-                <mesh filename="package://spot_description/meshes/body/front_left_hip_collision.stl" />
+                <mesh filename="file://$(find spot_description)/meshes/body/front_left_hip.dae" />
+            </geometry>
+        </visual>
+        <collision>
+            <geometry>
+                <mesh filename="file://$(find spot_description)/meshes/body/front_left_hip_collision.stl" />
             </geometry>
         </collision>
@@ -79,10 +79,10 @@
         <visual>
             <geometry>
-                <mesh filename="package://spot_description/meshes/body/front_left_upper_leg.dae" />
-            </geometry>
-        </visual>
-        <collision>
-            <geometry>
-                <mesh filename="package://spot_description/meshes/body/front_left_upper_leg_collision.stl" />
+                <mesh filename="file://$(find spot_description)/meshes/body/front_left_upper_leg.dae" />
+            </geometry>
+        </visual>
+        <collision>
+            <geometry>
+                <mesh filename="file://$(find spot_description)/meshes/body/front_left_upper_leg_collision.stl" />
             </geometry>
         </collision>
@@ -113,10 +113,10 @@
         <visual>
             <geometry>
-                <mesh filename="package://spot_description/meshes/body/front_left_lower_leg.dae" />
-            </geometry>
-        </visual>
-        <collision>
-            <geometry>
-                <mesh filename="package://spot_description/meshes/body/front_left_lower_leg_collision.stl" />
+                <mesh filename="file://$(find spot_description)/meshes/body/front_left_lower_leg.dae" />
+            </geometry>
+        </visual>
+        <collision>
+            <geometry>
+                <mesh filename="file://$(find spot_description)/meshes/body/front_left_lower_leg_collision.stl" />
             </geometry>
         </collision>
@@ -160,10 +160,10 @@
         <visual>
             <geometry>
-                <mesh filename="package://spot_description/meshes/body/front_right_hip.dae" />
-            </geometry>
-        </visual>
-        <collision>
-            <geometry>
-                <mesh filename="package://spot_description/meshes/body/front_right_hip_collision.stl" />
+                <mesh filename="file://$(find spot_description)/meshes/body/front_right_hip.dae" />
+            </geometry>
+        </visual>
+        <collision>
+            <geometry>
+                <mesh filename="file://$(find spot_description)/meshes/body/front_right_hip_collision.stl" />
             </geometry>
         </collision>
@@ -194,10 +194,10 @@
         <visual>
             <geometry>
-                <mesh filename="package://spot_description/meshes/body/front_right_upper_leg.dae" />
-            </geometry>
-        </visual>
-        <collision>
-            <geometry>
-                <mesh filename="package://spot_description/meshes/body/front_right_upper_leg_collision.stl" />
+                <mesh filename="file://$(find spot_description)/meshes/body/front_right_upper_leg.dae" />
+            </geometry>
+        </visual>
+        <collision>
+            <geometry>
+                <mesh filename="file://$(find spot_description)/meshes/body/front_right_upper_leg_collision.stl" />
             </geometry>
         </collision>
@@ -228,10 +228,10 @@
         <visual>
             <geometry>
-                <mesh filename="package://spot_description/meshes/body/front_right_lower_leg.dae" />
-            </geometry>
-        </visual>
-        <collision>
-            <geometry>
-                <mesh filename="package://spot_description/meshes/body/front_right_lower_leg_collision.stl" />
+                <mesh filename="file://$(find spot_description)/meshes/body/front_right_lower_leg.dae" />
+            </geometry>
+        </visual>
+        <collision>
+            <geometry>
+                <mesh filename="file://$(find spot_description)/meshes/body/front_right_lower_leg_collision.stl" />
             </geometry>
         </collision>
@@ -275,10 +275,10 @@
         <visual>
             <geometry>
-                <mesh filename="package://spot_description/meshes/body/rear_left_hip.dae" />
-            </geometry>
-        </visual>
-        <collision>
-            <geometry>
-                <mesh filename="package://spot_description/meshes/body/rear_left_hip_collision.stl" />
+                <mesh filename="file://$(find spot_description)/meshes/body/rear_left_hip.dae" />
+            </geometry>
+        </visual>
+        <collision>
+            <geometry>
+                <mesh filename="file://$(find spot_description)/meshes/body/rear_left_hip_collision.stl" />
             </geometry>
         </collision>
@@ -309,10 +309,10 @@
         <visual>
             <geometry>
-                <mesh filename="package://spot_description/meshes/body/rear_left_upper_leg.dae" />
-            </geometry>
-        </visual>
-        <collision>
-            <geometry>
-                <mesh filename="package://spot_description/meshes/body/rear_left_upper_leg_collision.stl" />
+                <mesh filename="file://$(find spot_description)/meshes/body/rear_left_upper_leg.dae" />
+            </geometry>
+        </visual>
+        <collision>
+            <geometry>
+                <mesh filename="file://$(find spot_description)/meshes/body/rear_left_upper_leg_collision.stl" />
             </geometry>
         </collision>
@@ -343,10 +343,10 @@
         <visual>
             <geometry>
-                <mesh filename="package://spot_description/meshes/body/rear_left_lower_leg.dae" />
-            </geometry>
-        </visual>
-        <collision>
-            <geometry>
-                <mesh filename="package://spot_description/meshes/body/rear_left_lower_leg_collision.stl" />
+                <mesh filename="file://$(find spot_description)/meshes/body/rear_left_lower_leg.dae" />
+            </geometry>
+        </visual>
+        <collision>
+            <geometry>
+                <mesh filename="file://$(find spot_description)/meshes/body/rear_left_lower_leg_collision.stl" />
             </geometry>
         </collision>
@@ -390,10 +390,10 @@
         <visual>
             <geometry>
-                <mesh filename="package://spot_description/meshes/body/rear_right_hip.dae" />
-            </geometry>
-        </visual>
-        <collision>
-            <geometry>
-                <mesh filename="package://spot_description/meshes/body/rear_right_hip_collision.stl" />
+                <mesh filename="file://$(find spot_description)/meshes/body/rear_right_hip.dae" />
+            </geometry>
+        </visual>
+        <collision>
+            <geometry>
+                <mesh filename="file://$(find spot_description)/meshes/body/rear_right_hip_collision.stl" />
             </geometry>
         </collision>
@@ -424,10 +424,10 @@
         <visual>
             <geometry>
-                <mesh filename="package://spot_description/meshes/body/rear_right_upper_leg.dae" />
-            </geometry>
-        </visual>
-        <collision>
-            <geometry>
-                <mesh filename="package://spot_description/meshes/body/rear_right_upper_leg_collision.stl" />
+                <mesh filename="file://$(find spot_description)/meshes/body/rear_right_upper_leg.dae" />
+            </geometry>
+        </visual>
+        <collision>
+            <geometry>
+                <mesh filename="file://$(find spot_description)/meshes/body/rear_right_upper_leg_collision.stl" />
             </geometry>
         </collision>
@@ -458,10 +458,10 @@
         <visual>
             <geometry>
-                <mesh filename="package://spot_description/meshes/body/rear_right_lower_leg.dae" />
-            </geometry>
-        </visual>
-        <collision>
-            <geometry>
-                <mesh filename="package://spot_description/meshes/body/rear_right_lower_leg_collision.stl" />
+                <mesh filename="file://$(find spot_description)/meshes/body/rear_right_lower_leg.dae" />
+            </geometry>
+        </visual>
+        <collision>
+            <geometry>
+                <mesh filename="file://$(find spot_description)/meshes/body/rear_right_lower_leg_collision.stl" />
             </geometry>
         </collision>
@@ -519,10 +519,10 @@
             <visual>
                 <geometry>
-                    <mesh filename="package://spot_description/meshes/accessories/eap_lidar.stl" />
+                    <mesh filename="file://$(find spot_description)/meshes/accessories/eap_lidar.stl" />
                 </geometry>
             </visual>
             <collision>
                 <geometry>
-                    <mesh filename="package://spot_description/meshes/accessories/eap_lidar.stl" />
+                    <mesh filename="file://$(find spot_description)/meshes/accessories/eap_lidar.stl" />
                 </geometry>
             </collision>

Commit message: replaced all file:// calls with package://

File: spot_description/urdf/spot.urdf.xacro (robot description, xacro)
@@ -10,10 +10,10 @@
         <visual>
             <geometry>
-                <mesh filename="file://$(find spot_description)/meshes/body/body.dae" />
-            </geometry>
-        </visual>
-        <collision>
-            <geometry>
-                <mesh filename="file://$(find spot_description)/meshes/body/body_collision.stl" />
+                <mesh filename="package://spot_description/meshes/body/body.dae" />
+            </geometry>
+        </visual>
+        <collision>
+            <geometry>
+                <mesh filename="package://spot_description/meshes/body/body_collision.stl" />
             </geometry>
         </collision>
@@ -45,10 +45,10 @@
         <visual>
             <geometry>
-                <mesh filename="file://$(find spot_description)/meshes/body/front_left_hip.dae" />
-            </geometry>
-        </visual>
-        <collision>
-            <geometry>
-                <mesh filename="file://$(find spot_description)/meshes/body/front_left_hip_collision.stl" />
+                <mesh filename="package://spot_description/meshes/body/front_left_hip.dae" />
+            </geometry>
+        </visual>
+        <collision>
+            <geometry>
+                <mesh filename="package://spot_description/meshes/body/front_left_hip_collision.stl" />
             </geometry>
         </collision>
@@ -79,10 +79,10 @@
         <visual>
             <geometry>
-                <mesh filename="file://$(find spot_description)/meshes/body/front_left_upper_leg.dae" />
-            </geometry>
-        </visual>
-        <collision>
-            <geometry>
-                <mesh filename="file://$(find spot_description)/meshes/body/front_left_upper_leg_collision.stl" />
+                <mesh filename="package://spot_description/meshes/body/front_left_upper_leg.dae" />
+            </geometry>
+        </visual>
+        <collision>
+            <geometry>
+                <mesh filename="package://spot_description/meshes/body/front_left_upper_leg_collision.stl" />
             </geometry>
         </collision>
@@ -113,10 +113,10 @@
         <visual>
             <geometry>
-                <mesh filename="file://$(find spot_description)/meshes/body/front_left_lower_leg.dae" />
-            </geometry>
-        </visual>
-        <collision>
-            <geometry>
-                <mesh filename="file://$(find spot_description)/meshes/body/front_left_lower_leg_collision.stl" />
+                <mesh filename="package://spot_description/meshes/body/front_left_lower_leg.dae" />
+            </geometry>
+        </visual>
+        <collision>
+            <geometry>
+                <mesh filename="package://spot_description/meshes/body/front_left_lower_leg_collision.stl" />
             </geometry>
         </collision>
@@ -160,10 +160,10 @@
         <visual>
             <geometry>
-                <mesh filename="file://$(find spot_description)/meshes/body/front_right_hip.dae" />
-            </geometry>
-        </visual>
-        <collision>
-            <geometry>
-                <mesh filename="file://$(find spot_description)/meshes/body/front_right_hip_collision.stl" />
+                <mesh filename="package://spot_description/meshes/body/front_right_hip.dae" />
+            </geometry>
+        </visual>
+        <collision>
+            <geometry>
+                <mesh filename="package://spot_description/meshes/body/front_right_hip_collision.stl" />
             </geometry>
         </collision>
@@ -194,10 +194,10 @@
         <visual>
             <geometry>
-                <mesh filename="file://$(find spot_description)/meshes/body/front_right_upper_leg.dae" />
-            </geometry>
-        </visual>
-        <collision>
-            <geometry>
-                <mesh filename="file://$(find spot_description)/meshes/body/front_right_upper_leg_collision.stl" />
+                <mesh filename="package://spot_description/meshes/body/front_right_upper_leg.dae" />
+            </geometry>
+        </visual>
+        <collision>
+            <geometry>
+                <mesh filename="package://spot_description/meshes/body/front_right_upper_leg_collision.stl" />
             </geometry>
         </collision>
@@ -228,10 +228,10 @@
         <visual>
             <geometry>
-                <mesh filename="file://$(find spot_description)/meshes/body/front_right_lower_leg.dae" />
-            </geometry>
-        </visual>
-        <collision>
-            <geometry>
-                <mesh filename="file://$(find spot_description)/meshes/body/front_right_lower_leg_collision.stl" />
+                <mesh filename="package://spot_description/meshes/body/front_right_lower_leg.dae" />
+            </geometry>
+        </visual>
+        <collision>
+            <geometry>
+                <mesh filename="package://spot_description/meshes/body/front_right_lower_leg_collision.stl" />
             </geometry>
         </collision>
@@ -275,10 +275,10 @@
         <visual>
             <geometry>
-                <mesh filename="file://$(find spot_description)/meshes/body/rear_left_hip.dae" />
-            </geometry>
-        </visual>
-        <collision>
-            <geometry>
-                <mesh filename="file://$(find spot_description)/meshes/body/rear_left_hip_collision.stl" />
+                <mesh filename="package://spot_description/meshes/body/rear_left_hip.dae" />
+            </geometry>
+        </visual>
+        <collision>
+            <geometry>
+                <mesh filename="package://spot_description/meshes/body/rear_left_hip_collision.stl" />
             </geometry>
         </collision>
@@ -309,10 +309,10 @@
         <visual>
             <geometry>
-                <mesh filename="file://$(find spot_description)/meshes/body/rear_left_upper_leg.dae" />
-            </geometry>
-        </visual>
-        <collision>
-            <geometry>
-                <mesh filename="file://$(find spot_description)/meshes/body/rear_left_upper_leg_collision.stl" />
+                <mesh filename="package://spot_description/meshes/body/rear_left_upper_leg.dae" />
+            </geometry>
+        </visual>
+        <collision>
+            <geometry>
+                <mesh filename="package://spot_description/meshes/body/rear_left_upper_leg_collision.stl" />
             </geometry>
         </collision>
@@ -343,10 +343,10 @@
         <visual>
             <geometry>
-                <mesh filename="file://$(find spot_description)/meshes/body/rear_left_lower_leg.dae" />
-            </geometry>
-        </visual>
-        <collision>
-            <geometry>
-                <mesh filename="file://$(find spot_description)/meshes/body/rear_left_lower_leg_collision.stl" />
+                <mesh filename="package://spot_description/meshes/body/rear_left_lower_leg.dae" />
+            </geometry>
+        </visual>
+        <collision>
+            <geometry>
+                <mesh filename="package://spot_description/meshes/body/rear_left_lower_leg_collision.stl" />
             </geometry>
         </collision>
@@ -390,10 +390,10 @@
         <visual>
             <geometry>
-                <mesh filename="file://$(find spot_description)/meshes/body/rear_right_hip.dae" />
-            </geometry>
-        </visual>
-        <collision>
-            <geometry>
-                <mesh filename="file://$(find spot_description)/meshes/body/rear_right_hip_collision.stl" />
+                <mesh filename="package://spot_description/meshes/body/rear_right_hip.dae" />
+            </geometry>
+        </visual>
+        <collision>
+            <geometry>
+                <mesh filename="package://spot_description/meshes/body/rear_right_hip_collision.stl" />
             </geometry>
         </collision>
@@ -424,10 +424,10 @@
         <visual>
             <geometry>
-                <mesh filename="file://$(find spot_description)/meshes/body/rear_right_upper_leg.dae" />
-            </geometry>
-        </visual>
-        <collision>
-            <geometry>
-                <mesh filename="file://$(find spot_description)/meshes/body/rear_right_upper_leg_collision.stl" />
+                <mesh filename="package://spot_description/meshes/body/rear_right_upper_leg.dae" />
+            </geometry>
+        </visual>
+        <collision>
+            <geometry>
+                <mesh filename="package://spot_description/meshes/body/rear_right_upper_leg_collision.stl" />
             </geometry>
         </collision>
@@ -458,10 +458,10 @@
         <visual>
             <geometry>
-                <mesh filename="file://$(find spot_description)/meshes/body/rear_right_lower_leg.dae" />
-            </geometry>
-        </visual>
-        <collision>
-            <geometry>
-                <mesh filename="file://$(find spot_description)/meshes/body/rear_right_lower_leg_collision.stl" />
+                <mesh filename="package://spot_description/meshes/body/rear_right_lower_leg.dae" />
+            </geometry>
+        </visual>
+        <collision>
+            <geometry>
+                <mesh filename="package://spot_description/meshes/body/rear_right_lower_leg_collision.stl" />
             </geometry>
         </collision>
@@ -519,10 +519,10 @@
             <visual>
                 <geometry>
-                    <mesh filename="file://$(find spot_description)/meshes/accessories/eap_lidar.stl" />
+                    <mesh filename="package://spot_description/meshes/accessories/eap_lidar.stl" />
                 </geometry>
             </visual>
             <collision>
                 <geometry>
-                    <mesh filename="file://$(find spot_description)/meshes/accessories/eap_lidar.stl" />
+                    <mesh filename="package://spot_description/meshes/accessories/eap_lidar.stl" />
                 </geometry>
             </collision>

Commit message: Added realsense and mount to description

File: spot_description/urdf/spot.urdf.xacro (robot description, xacro)
@@ -538,4 +538,5 @@
         </xacro:VLP-16>
     </xacro:if>
+    <xacro:include filename="$(find spot_description)/urdf/realsense_mount.urdf.xacro"/>
     <!-- Optional custom includes. -->
     <xacro:include filename="$(optenv SPOT_URDF_EXTRAS empty.urdf)" />

Commit message: Added virtual links and joints to URDF

File: spot_description/urdf/spot.urdf.xacro (robot description, xacro)
@@ -6,4 +6,26 @@
     <xacro:arg name="has_arm" default="False" />
     <xacro:arg name="has_eap" default="False" />
+    <!-- Virtual links -->
+    <link name="base_footprint"/>
+    <link name="body_height"/>
+    <link name="body_with_yaw"/>
+    <!-- Virtual Joints -->
+    <joint name="body_height_joint" type="prismatic">
+        <parent link = "base_footprint"/>
+        <child  link = "body_height"/>
+        <limit lower = "0.4" upper = "0.6"/>    <!-- TODO: Test what the real values are -->
+    </joint>
+    <joint name="body_yaw_joint" type="revolute">
+        <parent link = "body_height"/>
+        <child  link = "body_with_yaw"/>
+        <limit lower = "${-pi/6}" upper = "${pi/6}"/>
+        <axis    xyz = "0 0 1"/>
+    </joint>
+    <joint name="body_pitch_joint" type="revolute">
+        <parent link = "body_with_yaw"/>
+        <child  link = "body"/>
+        <limit lower = "${-pi/9}" upper = "${pi/9}"/>
+        <axis    xyz = "0 1 0"/>
+    </joint>
     <!-- Fixed links -->
     <link name="body">

Commit message: Added virtual joints to TF tree

File: spot_description/urdf/spot.urdf.xacro (robot description, xacro)
@@ -10,20 +10,28 @@
     <link name="body_height"/>
     <link name="body_with_yaw"/>
+    <link name="body_with_pitch_and_yaw"/>
     <!-- Virtual Joints -->
     <joint name="body_height_joint" type="prismatic">
         <parent link = "base_footprint"/>
         <child  link = "body_height"/>
-        <limit lower = "0.4" upper = "0.6"/>    <!-- TODO: Test what the real values are -->
+        <axis xyz = "0 0 1"/>
+        <limit lower = "0.37" upper = "0.60" velocity="0.1" effort="1e9"/>    <!-- TODO: Test what the real values are -->
     </joint>
     <joint name="body_yaw_joint" type="revolute">
         <parent link = "body_height"/>
         <child  link = "body_with_yaw"/>
-        <limit lower = "${-pi/6}" upper = "${pi/6}"/>
+        <limit lower = "${-pi/6}" upper = "${pi/6}" velocity="0.1" effort="1e9"/>
         <axis    xyz = "0 0 1"/>
     </joint>
     <joint name="body_pitch_joint" type="revolute">
         <parent link = "body_with_yaw"/>
+        <child  link = "body_with_pitch_and_yaw"/>
+        <limit lower = "${-pi/9}" upper = "${pi/9}"  velocity="0.1" effort="1e9"/>
+        <axis    xyz = "0 1 0"/>
+    </joint>
+    <joint name="body_roll_joint" type="revolute">
+        <parent link = "body_with_pitch_and_yaw"/>
         <child  link = "body"/>
-        <limit lower = "${-pi/9}" upper = "${pi/9}"/>
+        <limit lower = "${-pi/9}" upper = "${pi/9}"  velocity="0.1" effort="1e9"/>
         <axis    xyz = "0 1 0"/>
     </joint>
