Commit message: Removed TODO comment

File: spot_description/urdf/spot.urdf.xacro (robot description, xacro)
@@ -16,5 +16,5 @@
         <child  link = "body_height"/>
         <axis xyz = "0 0 1"/>
-        <limit lower = "0.37" upper = "0.60" velocity="0.1" effort="1e9"/>    <!-- TODO: Test what the real values are -->
+        <limit lower = "0.37" upper = "0.60" velocity="0.1" effort="1e9"/>
     </joint>
     <joint name="body_yaw_joint" type="revolute">

Commit message: Fixed body roll axis

File: spot_description/urdf/spot.urdf.xacro (robot description, xacro)
@@ -34,5 +34,5 @@
         <child  link = "body"/>
         <limit lower = "${-pi/9}" upper = "${pi/9}"  velocity="0.1" effort="1e9"/>
-        <axis    xyz = "0 1 0"/>
+        <axis    xyz = "1 0 0"/>
     </joint>
     <!-- Fixed links -->

Commit message: Fixed joint limits on virtual joints

File: spot_description/urdf/spot.urdf.xacro (robot description, xacro)
@@ -21,5 +21,5 @@
         <parent link = "body_height"/>
         <child  link = "body_with_yaw"/>
-        <limit lower = "${-pi/6}" upper = "${pi/6}" velocity="0.1" effort="1e9"/>
+        <limit lower = "${-pi/9}" upper = "${pi/9}" velocity="0.1" effort="1e9"/>
         <axis    xyz = "0 0 1"/>
     </joint>
@@ -33,5 +33,5 @@
         <parent link = "body_with_pitch_and_yaw"/>
         <child  link = "body"/>
-        <limit lower = "${-pi/9}" upper = "${pi/9}"  velocity="0.1" effort="1e9"/>
+        <limit lower = "${-pi/18}" upper = "${pi/18}"  velocity="0.1" effort="1e9"/>
         <axis    xyz = "1 0 0"/>
     </joint>

Commit message: Updated joint limits on virtual joints

File: spot_description/urdf/spot.urdf.xacro (robot description, xacro)
@@ -27,5 +27,5 @@
         <parent link = "body_with_yaw"/>
         <child  link = "body_with_pitch_and_yaw"/>
-        <limit lower = "${-pi/9}" upper = "${pi/9}"  velocity="0.1" effort="1e9"/>
+        <limit lower = "${-pi/12}" upper = "${pi/12}"  velocity="0.1" effort="1e9"/>
         <axis    xyz = "0 1 0"/>
     </joint>

Commit message: added Spot EAP2 to URDF

File: spot_description/urdf/spot.urdf.xacro (robot description, xacro)
@@ -6,4 +6,6 @@
     <xacro:arg name="has_arm" default="False" />
     <xacro:arg name="has_eap" default="False" />
+    <xacro:arg name="has_eap_2" default="False" />
+    <xacro:arg name="has_realsense" default="False" />
     <!-- Fixed links -->
     <link name="body">
@@ -538,4 +540,24 @@
         </xacro:VLP-16>
     </xacro:if>
+    <!-- Updated Spot Enhanced Autonomy Package (EAP2) -->
+    <xacro:if value="$(arg has_eap_2)">
+        <link name="eap_2_assembly">
+            <visual>
+                <geometry>
+                    <mesh filename="package://spot_description/meshes/accessories/eap2_lidar.stl" />
+                </geometry>
+            </visual>
+            <collision>
+                <geometry>
+                    <mesh filename="package://spot_description/meshes/accessories/eap2_lidar.stl" />
+                </geometry>
+            </collision>
+        </link>
+        <joint name="lidar_mount" type="fixed">
+            <origin xyz="-0.03 0.0 0.0" rpy="0 0 0" />
+            <parent link="rear_rail" />
+            <child link="lidar_assembly" />
+        </joint>
+    </xacro:if>
     <!-- Optional custom includes. -->
     <xacro:include filename="$(optenv SPOT_URDF_EXTRAS empty.urdf)" />

Commit message: fixed bugs with EAP2 setup

File: spot_description/urdf/spot.urdf.xacro (robot description, xacro)
@@ -554,8 +554,8 @@
             </collision>
         </link>
-        <joint name="lidar_mount" type="fixed">
+        <joint name="eap_2_mount" type="fixed">
             <origin xyz="-0.03 0.0 0.0" rpy="0 0 0" />
             <parent link="rear_rail" />
-            <child link="lidar_assembly" />
+            <child link="eap_2_assembly" />
         </joint>
     </xacro:if>

Commit message: Updated EAP2 visuals and collisions

File: spot_description/urdf/spot.urdf.xacro (robot description, xacro)
@@ -545,10 +545,10 @@
             <visual>
                 <geometry>
-                    <mesh filename="package://spot_description/meshes/accessories/eap2_lidar.stl" />
+                    <mesh filename="package://spot_description/meshes/accessories/EAP2.dae" />
                 </geometry>
             </visual>
             <collision>
                 <geometry>
-                    <mesh filename="package://spot_description/meshes/accessories/eap2_lidar.stl" />
+                    <mesh filename="package://spot_description/meshes/accessories/EAP2_compressed.stl" />
                 </geometry>
             </collision>

Commit message: fixed issues with EAP2 config

File: spot_description/urdf/spot.urdf.xacro (robot description, xacro)
@@ -555,5 +555,5 @@
         </link>
         <joint name="eap_2_mount" type="fixed">
-            <origin xyz="-0.03 0.0 0.0" rpy="0 0 0" />
+	    <origin xyz="0.015 0.0 0.0" rpy="0 0 ${pi/2}" />
             <parent link="rear_rail" />
             <child link="eap_2_assembly" />

Commit message: EAP config fixes

File: spot_description/urdf/spot.urdf.xacro (robot description, xacro)
@@ -555,5 +555,5 @@
         </link>
         <joint name="eap_2_mount" type="fixed">
-            <origin xyz="-0.03 0.0 0.0" rpy="0 0 0" />
+            <origin xyz="0.015 0.0 0.0" rpy="0 0 ${pi/2}" />
             <parent link="rear_rail" />
             <child link="eap_2_assembly" />

Commit message: Updated urdf to have optional kinematic models

File: spot_description/urdf/spot.urdf.xacro (robot description, xacro)
@@ -4,38 +4,67 @@
          published by the driver (see spot_driver package) during runtime, so that the transforms
          include calibration adjustments. -->
-    <xacro:arg name="has_arm" default="False" />
-    <xacro:arg name="has_eap" default="False" />
-    <xacro:arg name="has_eap_2" default="False" />
-    <xacro:arg name="has_realsense" default="False" />
+    <xacro:arg name="has_arm" default="False"/>
+    <xacro:arg name="has_eap" default="False"/>
+    <xacro:arg name="has_eap_2" default="False"/>
+    <xacro:arg name="has_realsense" default="False"/>
+    <xacro:arg name="kinematic_model" default="default"/>
+    <xacro:property name="kinematic_model" value="$(arg kinematic_model)"/>
     <!-- Virtual links -->
     <link name="base_footprint"/>
-    <link name="body_height"/>
-    <link name="body_with_yaw"/>
-    <link name="body_with_pitch_and_yaw"/>
     <!-- Virtual Joints -->
-    <joint name="body_height_joint" type="prismatic">
-        <parent link = "base_footprint"/>
-        <child  link = "body_height"/>
-        <axis xyz = "0 0 1"/>
-        <limit lower = "0.37" upper = "0.60" velocity="0.1" effort="1e9"/>
-    </joint>
-    <joint name="body_yaw_joint" type="revolute">
-        <parent link = "body_height"/>
-        <child  link = "body_with_yaw"/>
-        <limit lower = "${-pi/9}" upper = "${pi/9}" velocity="0.1" effort="1e9"/>
-        <axis    xyz = "0 0 1"/>
-    </joint>
-    <joint name="body_pitch_joint" type="revolute">
-        <parent link = "body_with_yaw"/>
-        <child  link = "body_with_pitch_and_yaw"/>
-        <limit lower = "${-pi/12}" upper = "${pi/12}"  velocity="0.1" effort="1e9"/>
-        <axis    xyz = "0 1 0"/>
-    </joint>
-    <joint name="body_roll_joint" type="revolute">
-        <parent link = "body_with_pitch_and_yaw"/>
-        <child  link = "body"/>
-        <limit lower = "${-pi/18}" upper = "${pi/18}"  velocity="0.1" effort="1e9"/>
-        <axis    xyz = "1 0 0"/>
-    </joint>
+    <xacro:if value="${kinematic_model == 'body_assist'}"/>
+        <link name="body_height"/>
+        <link name="body_with_yaw"/>
+        <link name="body_with_pitch_and_yaw"/>
+        <joint name="body_height_joint" type="prismatic">
+            <parent link = "base_footprint"/>
+            <child  link = "body_height"/>
+            <axis xyz = "0 0 1"/>
+            <limit lower = "0.37" upper = "0.60" velocity="0.1" effort="1e9"/>
+        </joint>
+        <joint name="body_yaw_joint" type="revolute">
+            <parent link = "body_height"/>
+            <child  link = "body_with_yaw"/>
+            <limit lower = "${-pi/9}" upper = "${pi/9}" velocity="0.1" effort="1e9"/>
+            <axis    xyz = "0 0 1"/>
+        </joint>
+        <joint name="body_pitch_joint" type="revolute">
+            <parent link = "body_with_yaw"/>
+            <child  link = "body_with_pitch_and_yaw"/>
+            <limit lower = "${-pi/12}" upper = "${pi/12}"  velocity="0.1" effort="1e9"/>
+            <axis    xyz = "0 1 0"/>
+        </joint>
+        <joint name="body_roll_joint" type="revolute">
+            <parent link = "body_with_pitch_and_yaw"/>
+            <child  link = "body"/>
+            <limit lower = "${-pi/18}" upper = "${pi/18}"  velocity="0.1" effort="1e9"/>
+            <axis    xyz = "1 0 0"/>
+        </joint>
+    </xacro:if>
+    <xacro:if value="${kinematic_model == 'mobile_manipulation'}">
+        <!-- Virtual Base Movement links -->
+        <link name="body_x"/>
+        <link name="body_y"/>
+        <!-- Virtual Joints -->
+        <joint name="body_x" type="prismatic">
+            <parent link = "base_footprint"/>
+            <child  link = "body_x"/>
+            <axis xyz = "1 0 0"/>
+            <limit lower = "-10.0" upper = "10.0" velocity="0.1" effort="1e9"/>
+        </joint>
+        <joint name="body_y" type="prismatic">
+            <parent link = "body_x"/>
+            <child  link = "body_y"/>
+            <axis xyz = "0 1 0"/>
+            <limit lower = "-10.0" upper = "10.0" velocity="0.1" effort="1e9"/>
+        </joint>
+        <joint name="body_or" type="revolute">
+            <parent link = "body_y"/>
+            <child  link = "body"/>
+            <limit lower = "0" upper = "${2*pi}" velocity="0.1" effort="1e9"/>
+            <axis    xyz = "0 0 1"/>
+        </joint>
+        <!-- EOF Virtual Base Movement Links-->
+    </xacro:if>
     <!-- Fixed links -->
     <link name="body">

Commit message: Updated urdf to work with both kinematic models

File: spot_description/urdf/spot.urdf.xacro (robot description, xacro)
@@ -8,10 +8,9 @@
     <xacro:arg name="has_eap_2" default="False"/>
     <xacro:arg name="has_realsense" default="False"/>
-    <xacro:arg name="kinematic_model" default="default"/>
+    <xacro:arg name="kinematic_model" default="body_assist"/>
     <xacro:property name="kinematic_model" value="$(arg kinematic_model)"/>
-    <!-- Virtual links -->
     <link name="base_footprint"/>
     <!-- Virtual Joints -->
-    <xacro:if value="${kinematic_model == 'body_assist'}"/>
+    <xacro:if value="${kinematic_model == 'body_assist'}">
         <link name="body_height"/>
         <link name="body_with_yaw"/>
@@ -46,4 +45,5 @@
         <link name="body_x"/>
         <link name="body_y"/>
+        <link name="body_or"/>
         <!-- Virtual Joints -->
         <joint name="body_x" type="prismatic">
@@ -61,7 +61,12 @@
         <joint name="body_or" type="revolute">
             <parent link = "body_y"/>
-            <child  link = "body"/>
+            <child  link = "body_or"/>
             <limit lower = "0" upper = "${2*pi}" velocity="0.1" effort="1e9"/>
             <axis    xyz = "0 0 1"/>
+        </joint>
+        <joint name="ground_to_body" type="fixed">
+            <parent link = "body_or"/>
+            <child  link = "body"/>
+            <origin xyz="0 0 0.52"/>
         </joint>
         <!-- EOF Virtual Base Movement Links-->

Commit message: Added velodyne link and fixed alignment

File: spot_description/urdf/spot.urdf.xacro (robot description, xacro)
@@ -623,4 +623,11 @@
             <child link="eap_2_assembly" />
         </joint>
+        <link name="velodyne"/>
+        <joint name="eap2_to_velodyne_joint" type="fixed">
+            <parent link = "eap_2_assembly"/>
+            <child  link = "velodyne"/>
+            <!-- These values were found by trial and error and may be slightly inaccurate -->
+            <origin xyz="0 0.035 0.11" rpy="0 0 -0.95"/>
+        </joint>
     </xacro:if>
     <!-- Optional custom includes. -->

Commit message: Added URDF code for RL mounting kit

File: spot_description/urdf/spot.urdf.xacro (robot description, xacro)
@@ -7,4 +7,5 @@
     <xacro:arg name="has_eap" default="False"/>
     <xacro:arg name="has_eap_2" default="False"/>
+    <xacro:arg name="has_rl_kit" default="False"/>
     <xacro:arg name="has_realsense" default="False"/>
     <xacro:arg name="kinematic_model" default="body_assist"/>
@@ -106,4 +107,10 @@
         <parent link="body" />
         <child link="rear_rail" />
+    </joint>
+    <link name="payload_mount_reference_frame"/>
+    <joint name="payload_mount_reference_frame_joint" type="fixed">
+        <parent link = "base_link"/>
+        <child  link = "payload_mount_reference_frame"/>
+        <origin xyz = "0.2075 0.0 0.0805"/>
     </joint>
     <!-- Front Left -->
@@ -631,4 +638,9 @@
         </joint>
     </xacro:if>
+    <!-- Spot Reinforcement Learning Research Kit Mount with Nvidia Jetson Orin AGX -->
+    <xacro:if value="$(arg has_rl_kit)">
+        <xacro:include filename="$(find spot_description)/urdf/accessories/rl_kit.xacro"/>
+        <xacro:rl_kit/>
+    </xacro:if>
     <!-- Optional custom includes. -->
     <xacro:include filename="$(optenv SPOT_URDF_EXTRAS empty.urdf)" />

Commit message: make default kinematic model empty

File: spot_description/urdf/spot.urdf.xacro (robot description, xacro)
@@ -9,5 +9,5 @@
     <xacro:arg name="has_rl_kit" default="False"/>
     <xacro:arg name="has_realsense" default="False"/>
-    <xacro:arg name="kinematic_model" default="body_assist"/>
+    <xacro:arg name="kinematic_model" default="none"/>
     <xacro:property name="kinematic_model" value="$(arg kinematic_model)"/>
     <link name="base_footprint"/>
@@ -72,4 +72,11 @@
         </joint>
         <!-- EOF Virtual Base Movement Links-->
+    </xacro:if>
+    <xacro:if value="${kinematic_model == 'none'}">
+        <joint name="ground_to_body" type="fixed">
+            <parent link = "base_footprint"/>
+            <child  link = "body"/>
+            <origin xyz="0 0 0.52"/>
+        </joint>
     </xacro:if>
     <!-- Fixed links -->

Commit message: Fixed the EAP2 location by measuring mesh coordinates in blender

File: spot_description/urdf/spot.urdf.xacro (robot description, xacro)
@@ -641,6 +641,5 @@
             <parent link = "eap_2_assembly"/>
             <child  link = "velodyne"/>
-            <!-- These values were found by trial and error and may be slightly inaccurate -->
-            <origin xyz="0 0.035 0.11" rpy="0 0 -0.95"/>
+            <origin  xyz = "0 0.02775 0.1091" rpy="0 0 -0.9486"/>
         </joint>
     </xacro:if>

Commit message: Fixed improper transform when kinematic model is 'none'

File: spot_description/urdf/spot.urdf.xacro (robot description, xacro)
@@ -11,5 +11,7 @@
     <xacro:arg name="kinematic_model" default="none"/>
     <xacro:property name="kinematic_model" value="$(arg kinematic_model)"/>
-    <link name="base_footprint"/>
+    <xacro:unless value="${kinematic_model == 'none'}">
+        <link name="base_footprint"/>
+    </xacro:unless>
     <!-- Virtual Joints -->
     <xacro:if value="${kinematic_model == 'body_assist'}">
@@ -72,11 +74,4 @@
         </joint>
         <!-- EOF Virtual Base Movement Links-->
-    </xacro:if>
-    <xacro:if value="${kinematic_model == 'none'}">
-        <joint name="ground_to_body" type="fixed">
-            <parent link = "base_footprint"/>
-            <child  link = "body"/>
-            <origin xyz="0 0 0.52"/>
-        </joint>
     </xacro:if>
     <!-- Fixed links -->

Commit message: add visual fallbacks for accessories and enable prop mesh selection

File: spot_description/urdf/spot.urdf.xacro (robot description, xacro)
@@ -10,4 +10,5 @@
     <xacro:arg name="has_realsense" default="False"/>
     <xacro:arg name="kinematic_model" default="none"/>
+    <xacro:arg name="use_proprietary_meshes" default="false" />
     <xacro:property name="kinematic_model" value="$(arg kinematic_model)"/>
     <xacro:unless value="${kinematic_model == 'none'}">
@@ -592,14 +593,30 @@
     <xacro:if value="$(arg has_eap)">
         <link name="lidar_assembly">
+          <xacro:if value="$(arg use_proprietary_meshes)">
             <visual>
-                <geometry>
-                    <mesh filename="package://spot_description/meshes/accessories/eap_lidar.stl" />
-                </geometry>
+              <geometry>
+                <mesh filename="package://spot_propriety_description/meshes/accessories/eap_lidar.stl"/>
+              </geometry>
             </visual>
             <collision>
-                <geometry>
-                    <mesh filename="package://spot_description/meshes/accessories/eap_lidar.stl" />
-                </geometry>
+              <geometry>
+                <mesh filename="package://spot_propriety_description/meshes/accessories/eap_lidar.stl"/>
+              </geometry>
             </collision>
+          </xacro:if>
+          <xacro:unless value="$(arg use_proprietary_meshes)">
+            <visual>
+              <geometry>
+                <cylinder radius="0.1" length="0.17"/>
+              </geometry>
+              <origin xyz="0 0 0"/>
+            </visual>
+            <collision>
+              <geometry>
+                <cylinder radius="0.1" length="0.17"/>
+              </geometry>
+              <origin xyz="0 0 0"/>
+            </collision>
+          </xacro:unless>
         </link>
         <joint name="lidar_mount" type="fixed">
@@ -616,14 +633,46 @@
     <xacro:if value="$(arg has_eap_2)">
         <link name="eap_2_assembly">
+          <xacro:if value="$(arg use_proprietary_meshes)">
             <visual>
-                <geometry>
-                    <mesh filename="package://spot_description/meshes/accessories/EAP2.dae" />
-                </geometry>
+              <geometry>
+                <mesh filename="package://spot_propriety_description/meshes/accessories/EAP2.dae" />
+              </geometry>
             </visual>
             <collision>
-                <geometry>
-                    <mesh filename="package://spot_description/meshes/accessories/EAP2_compressed.stl" />
-                </geometry>
+              <geometry>
+                <mesh filename="package://spot_propriety_description/meshes/accessories/EAP2_compressed.stl" />
+              </geometry>
             </collision>
+          </xacro:if>
+          <xacro:unless value="$(arg use_proprietary_meshes)">
+            <!-- Base Box (computer) -->
+            <visual name="eap2_base">
+              <geometry>
+                <box size="0.224 0.173 0.064"/>
+              </geometry>
+              <origin xyz="0 0 0.032" rpy="0 0 0"/>
+            </visual>
+            <!-- LIDAR Cylinder -->
+            <visual name="eap2_lidar">
+              <geometry>
+                <cylinder radius="0.0735" length="0.182"/>
+              </geometry>
+              <origin xyz="0 0 0.155" rpy="0 0 0"/> <!-- base_z/2 + lidar_z/2 -->
+            </visual>
+            <!-- Base collision -->
+            <collision name="eap2_base_col">
+              <geometry>
+                <box size="0.224 0.173 0.064"/>
+              </geometry>
+              <origin xyz="0 0 0.032" rpy="0 0 0"/>
+            </collision>
+            <!-- LIDAR collision -->
+            <collision name="eap2_lidar_col">
+              <geometry>
+                <cylinder radius="0.0735" length="0.182"/>
+              </geometry>
+              <origin xyz="0 0 0.155" rpy="0 0 0"/>
+            </collision>
+          </xacro:unless>
         </link>
         <joint name="eap_2_mount" type="fixed">

Commit message: make accessory material black

File: spot_description/urdf/spot.urdf.xacro (robot description, xacro)
@@ -616,4 +616,7 @@
               </geometry>
               <origin xyz="0 0 0"/>
+              <material name="black">
+                <color rgba="0 0 0 1"/>
+              </material>
             </visual>
             <collision>
@@ -657,4 +660,7 @@
               </geometry>
               <origin xyz="0 0 0.032" rpy="0 0 0"/>
+              <material name="black">
+                <color rgba="0 0 0 1"/>
+              </material>
             </visual>
             <!-- LIDAR Cylinder -->
@@ -664,4 +670,7 @@
               </geometry>
               <origin xyz="0 0 0.155" rpy="0 0 0"/> <!-- base_z/2 + lidar_z/2 -->
+              <material name="black">
+                <color rgba="0 0 0 1"/>
+              </material>
             </visual>
             <!-- Base collision -->

Commit message: fix EAP visual and collision origin

File: spot_description/urdf/spot.urdf.xacro (robot description, xacro)
@@ -615,5 +615,5 @@
                 <cylinder radius="0.1" length="0.17"/>
               </geometry>
-              <origin xyz="0 0 0"/>
+	      <origin xyz="0 0 ${0.17/2}"/>
               <material name="black">
                 <color rgba="0 0 0 1"/>
@@ -624,5 +624,5 @@
                 <cylinder radius="0.1" length="0.17"/>
               </geometry>
-              <origin xyz="0 0 0"/>
+	      <origin xyz="0 0 ${0.17/2}"/>
             </collision>
           </xacro:unless>
