Commit message: adjust EAP2 Lidar visual and collision geometry

File: spot_description/urdf/spot.urdf.xacro (robot description, xacro)
@@ -657,7 +657,7 @@
             <visual name="eap2_base">
               <geometry>
-                <box size="0.224 0.173 0.064"/>
-              </geometry>
-              <origin xyz="0 0 0.032" rpy="0 0 0"/>
+                <box size="0.173 0.264 0.064"/>
+              </geometry>
+              <origin xyz="0 -0.01 0.032" rpy="0 0 0"/>
               <material name="black">
                 <color rgba="0 0 0 1"/>
@@ -667,7 +667,7 @@
             <visual name="eap2_lidar">
               <geometry>
-                <cylinder radius="0.0735" length="0.182"/>
-              </geometry>
-              <origin xyz="0 0 0.155" rpy="0 0 0"/> <!-- base_z/2 + lidar_z/2 -->
+                <cylinder radius="0.0765" length="0.182"/>
+              </geometry>
+              <origin xyz="0 0.03 0.155" rpy="0 0 0"/> <!-- base_z/2 + lidar_z/2 -->
               <material name="black">
                 <color rgba="0 0 0 1"/>
@@ -677,14 +677,14 @@
             <collision name="eap2_base_col">
               <geometry>
-                <box size="0.224 0.173 0.064"/>
-              </geometry>
-              <origin xyz="0 0 0.032" rpy="0 0 0"/>
+                <box size="0.173 0.264 0.064"/>
+              </geometry>
+              <origin xyz="0 -0.01 0.032" rpy="0 0 0"/>
             </collision>
             <!-- LIDAR collision -->
             <collision name="eap2_lidar_col">
               <geometry>
-                <cylinder radius="0.0735" length="0.182"/>
-              </geometry>
-              <origin xyz="0 0 0.155" rpy="0 0 0"/>
+                <cylinder radius="0.0765" length="0.182"/>
+              </geometry>
+              <origin xyz="0 0.03 0.155" rpy="0 0 0"/>
             </collision>
           </xacro:unless>

Commit message: adjust eap visual and collision dim

File: spot_description/urdf/spot.urdf.xacro (robot description, xacro)
@@ -613,5 +613,5 @@
             <visual>
               <geometry>
-                <cylinder radius="0.1" length="0.17"/>
+                <cylinder radius="0.12" length="0.17"/>
               </geometry>
 	      <origin xyz="0 0 ${0.17/2}"/>
@@ -622,5 +622,5 @@
             <collision>
               <geometry>
-                <cylinder radius="0.1" length="0.17"/>
+                <cylinder radius="0.12" length="0.17"/>
               </geometry>
 	      <origin xyz="0 0 ${0.17/2}"/>

Commit message: Removed simulation related tags since we do not have a functional simulation

File: spot_description/urdf/spot.urdf.xacro (robot description, xacro)
@@ -134,8 +134,4 @@
             </geometry>
         </collision>
-        <inertial>
-            <mass value="1.5" />
-    	    <inertia  ixx="0.0605" ixy="0.0"  ixz="0.0"  iyy="0.0"  iyz="0.0"  izz="0.0" />
-    	</inertial>
     </link>
     <joint name="front_left_hip_x" type="revolute">
@@ -144,17 +140,6 @@
         <parent link="body" />
         <child link="front_left_hip" />
-        <dynamics damping="0.1" friction="0.1"/>
         <limit effort="1000" velocity="1000.00" lower="-0.78539816339744827899" upper="0.78539816339744827899" />
     </joint>
-    <transmission name="front_left_hip_x_trans">
-	    <type>transmission_interface/SimpleTransmission</type>
-	    <joint name="front_left_hip_x">
-            <hardwareInterface>EffortJointInterface</hardwareInterface>
-        </joint>
-	    <actuator name="front_left_hip_x">
-          	<mechanicalReduction>50</mechanicalReduction>
-          	<hardwareInterface>EffortJointInterface</hardwareInterface>
-	    </actuator>
-    </transmission>
     <link name="front_left_upper_leg">
         <visual>
@@ -168,8 +153,4 @@
             </geometry>
         </collision>
-        <inertial>
-            <mass value="1.5" />
-    	    <inertia  ixx="0.0" ixy="0.0"  ixz="0.0"  iyy="0.05"  iyz="0.0"  izz="0.0" />
-    	</inertial>
     </link>
     <joint name="front_left_hip_y" type="revolute">
@@ -178,17 +159,6 @@
         <parent link="front_left_hip" />
         <child link="front_left_upper_leg" />
-        <dynamics damping="0.1" friction="0.1"/>
         <limit effort="1000" velocity="1000.00" lower="-0.89884456477707963539" upper="2.2951079663725435509" />
     </joint>
-    <transmission name="front_left_hip_y_trans">
-        <type>transmission_interface/SimpleTransmission</type>
-        <joint name="front_left_hip_y">
-            <hardwareInterface>EffortJointInterface</hardwareInterface>
-        </joint>
-        <actuator name="front_left_hip_y">
-            <mechanicalReduction>50</mechanicalReduction>
-            <hardwareInterface>EffortJointInterface</hardwareInterface>
-        </actuator>
-    </transmission>
     <link name="front_left_lower_leg">
         <visual>
@@ -202,8 +172,4 @@
             </geometry>
         </collision>
-        <inertial>
-            <mass value="1.0" />
-    	    <inertia  ixx="0.0" ixy="0.0"  ixz="0.0"  iyy="0.045"  iyz="0.0"  izz="0.0" />
-    	</inertial>
     </link>
     <joint name="front_left_knee" type="revolute">
@@ -212,29 +178,6 @@
         <parent link="front_left_upper_leg" />
         <child link="front_left_lower_leg" />
-        <dynamics damping="0.1" friction="0.1"/>
         <limit effort="1000" velocity="1000.00" lower="-2.7929" upper="-0.254801" />
     </joint>
-    <gazebo reference="front_left_lower_leg">
-        <sensor name="front_left_lower_leg_contactsensor_sensor" type="contact">
-        <always_on>true</always_on>
-        <contact>
-            <collision>front_left_lower_leg_fixed_joint_lump__front_bump_sensor_collision</collision>
-        </contact>
-        <plugin filename="libgazebo_ros_bumper.so" name="front_left_lower_leg_plugin">
-            <bumperTopicName>front_left_lower_leg_contact</bumperTopicName>
-            <frameName>front_left_lower_leg</frameName>
-        </plugin>
-        </sensor>
-    </gazebo>
-    <transmission name="front_left_knee_trans">
-	  <type>transmission_interface/SimpleTransmission</type>
-	  <joint name="front_left_knee">
-          	<hardwareInterface>EffortJointInterface</hardwareInterface>
-      </joint>
-	  <actuator name="front_left_knee">
-          	<mechanicalReduction>50</mechanicalReduction>
-          	<hardwareInterface>EffortJointInterface</hardwareInterface>
-	  </actuator>
-    </transmission>
     <!-- Front Right -->
     <link name="front_right_hip">
@@ -249,8 +192,4 @@
             </geometry>
         </collision>
-        <inertial>
-            <mass value="1.5" />
-    	    <inertia  ixx="0.0605" ixy="0.0"  ixz="0.0"  iyy="0.0"  iyz="0.0"  izz="0.0" />
-    	</inertial>
     </link>
     <joint name="front_right_hip_x" type="revolute">
@@ -259,17 +198,6 @@
         <parent link="body" />
         <child link="front_right_hip" />
-        <dynamics damping="0.1" friction="0.1"/>
         <limit effort="1000" velocity="1000.00" lower="-0.78539816339744827899" upper="0.78539816339744827899" />
     </joint>
-    <transmission name="front_right_hip_x_trans">
-	  <type>transmission_interface/SimpleTransmission</type>
-	  <joint name="front_right_hip_x">
-          	<hardwareInterface>EffortJointInterface</hardwareInterface>
-      </joint>
-	  <actuator name="front_right_hip_x">
-          	<mechanicalReduction>50</mechanicalReduction>
-          	<hardwareInterface>EffortJointInterface</hardwareInterface>
-	  </actuator>
-    </transmission>
     <link name="front_right_upper_leg">
         <visual>
@@ -283,8 +211,4 @@
             </geometry>
         </collision>
-        <inertial>
-            <mass value="1.5" />
-    	    <inertia  ixx="0.0" ixy="0.0"  ixz="0.0"  iyy="0.05"  iyz="0.0"  izz="0.0" />
-    	</inertial>
     </link>
     <joint name="front_right_hip_y" type="revolute">
@@ -293,17 +217,6 @@
         <parent link="front_right_hip" />
         <child link="front_right_upper_leg" />
-        <dynamics damping="0.1" friction="0.1"/>
         <limit effort="1000" velocity="1000.00" lower="-0.89884456477707963539" upper="2.2951079663725435509" />
     </joint>
-    <transmission name="front_right_hip_y_trans">
-        <type>transmission_interface/SimpleTransmission</type>
-        <joint name="front_right_hip_y">
-            <hardwareInterface>EffortJointInterface</hardwareInterface>
-        </joint>
-        <actuator name="front_right_hip_y">
-            <mechanicalReduction>50</mechanicalReduction>
-            <hardwareInterface>EffortJointInterface</hardwareInterface>
-        </actuator>
-    </transmission>
     <link name="front_right_lower_leg">
         <visual>
@@ -317,8 +230,4 @@
             </geometry>
         </collision>
-        <inertial>
-            <mass value="1.0" />
-    	    <inertia  ixx="0.0" ixy="0.0"  ixz="0.0"  iyy="0.045"  iyz="0.0"  izz="0.0" />
-    	</inertial>
     </link>
     <joint name="front_right_knee" type="revolute">
@@ -327,29 +236,6 @@
         <parent link="front_right_upper_leg" />
         <child link="front_right_lower_leg" />
-        <dynamics damping="0.1" friction="0.1"/>
         <limit effort="1000" velocity="1000.00" lower="-2.7929" upper="-0.247563" />
     </joint>
-    <gazebo reference="front_right_lower_leg">
-        <sensor name="front_right_lower_leg_contactsensor_sensor" type="contact">
-        <always_on>true</always_on>
-        <contact>
-            <collision>front_right_lower_leg_fixed_joint_lump__front_bump_sensor_collision</collision>
-        </contact>
-        <plugin filename="libgazebo_ros_bumper.so" name="front_right_lower_leg_plugin">
-            <bumperTopicName>front_right_lower_leg_contact</bumperTopicName>
-            <frameName>front_right_lower_leg</frameName>
-        </plugin>
-        </sensor>
-    </gazebo>
-    <transmission name="front_right_knee_trans">
-        <type>transmission_interface/SimpleTransmission</type>
-        <joint name="front_right_knee">
-            <hardwareInterface>EffortJointInterface</hardwareInterface>
-        </joint>
-        <actuator name="front_right_knee">
-            <mechanicalReduction>50</mechanicalReduction>
-            <hardwareInterface>EffortJointInterface</hardwareInterface>
-        </actuator>
-    </transmission>
     <!-- Rear Left -->
     <link name="rear_left_hip">
@@ -364,8 +250,4 @@
             </geometry>
         </collision>
-        <inertial>
-            <mass value="1.5" />
-    	    <inertia  ixx="0.0605" ixy="0.0"  ixz="0.0"  iyy="0.0"  iyz="0.0"  izz="0.0" />
-    	</inertial>
     </link>
     <joint name="rear_left_hip_x" type="revolute">
@@ -374,17 +256,6 @@
         <parent link="body" />
         <child link="rear_left_hip" />
-        <dynamics damping="0.1" friction="0.1"/>
         <limit effort="1000" velocity="1000.00" lower="-0.78539816339744827899" upper="0.78539816339744827899" />
     </joint>
-    <transmission name="rear_left_hip_x_trans">
-        <type>transmission_interface/SimpleTransmission</type>
-        <joint name="rear_left_hip_x">
-            <hardwareInterface>EffortJointInterface</hardwareInterface>
-        </joint>
-        <actuator name="rear_left_hip_x">
-            <mechanicalReduction>50</mechanicalReduction>
-            <hardwareInterface>EffortJointInterface</hardwareInterface>
-        </actuator>
-    </transmission>
     <link name="rear_left_upper_leg">
         <visual>
@@ -398,8 +269,4 @@
             </geometry>
         </collision>
-        <inertial>
-           <mass value="1.5" />
-    	   <inertia  ixx="0.0" ixy="0.0"  ixz="0.0"  iyy="0.05"  iyz="0.0"  izz="0.0" />
-    	</inertial>
     </link>
     <joint name="rear_left_hip_y" type="revolute">
@@ -408,17 +275,6 @@
         <parent link="rear_left_hip" />
         <child link="rear_left_upper_leg" />
-        <dynamics damping="0.1" friction="0.1"/>
         <limit effort="1000" velocity="1000.00" lower="-0.89884456477707963539" upper="2.2951079663725435509" />
     </joint>
-    <transmission name="rear_left_hip_y_trans">
-        <type>transmission_interface/SimpleTransmission</type>
-        <joint name="rear_left_hip_y">
-            <hardwareInterface>EffortJointInterface</hardwareInterface>
-        </joint>
-        <actuator name="rear_left_hip_y">
-            <mechanicalReduction>50</mechanicalReduction>
-            <hardwareInterface>EffortJointInterface</hardwareInterface>
-        </actuator>
-    </transmission>
     <link name="rear_left_lower_leg">
         <visual>
@@ -432,8 +288,4 @@
             </geometry>
         </collision>
-        <inertial>
-            <mass value="1.0" />
-    	    <inertia  ixx="0.0" ixy="0.0"  ixz="0.0"  iyy="0.045"  iyz="0.0"  izz="0.0" />
-    	</inertial>
     </link>
     <joint name="rear_left_knee" type="revolute">
@@ -442,29 +294,6 @@
         <parent link="rear_left_upper_leg" />
         <child link="rear_left_lower_leg" />
-        <dynamics damping="0.1" friction="0.1"/>
         <limit effort="1000" velocity="1000.00" lower="-2.7929" upper="-0.267153" />
     </joint>
-    <gazebo reference="rear_left_lower_leg">
-        <sensor name="rear_left_lower_leg_contactsensor_sensor" type="contact">
-        <always_on>true</always_on>
-        <contact>
-            <collision>rear_left_lower_leg_fixed_joint_lump__rear_bump_sensor_collision</collision>
-        </contact>
-        <plugin filename="libgazebo_ros_bumper.so" name="rear_left_lower_leg_plugin">
-            <bumperTopicName>rear_left_lower_leg_contact</bumperTopicName>
-            <frameName>rear_left_lower_leg</frameName>
-        </plugin>
-        </sensor>
-    </gazebo>
-    <transmission name="rear_left_knee_trans">
-        <type>transmission_interface/SimpleTransmission</type>
-        <joint name="rear_left_knee">
-             <hardwareInterface>EffortJointInterface</hardwareInterface>
-        </joint>
-        <actuator name="rear_left_knee">
-            <mechanicalReduction>50</mechanicalReduction>
-            <hardwareInterface>EffortJointInterface</hardwareInterface>
-        </actuator>
-    </transmission>
     <!-- Rear Right -->
     <link name="rear_right_hip">
@@ -479,8 +308,4 @@
             </geometry>
         </collision>
-        <inertial>
-            <mass value="1.5" />
-    	    <inertia  ixx="0.0605" ixy="0.0"  ixz="0.0"  iyy="0.0"  iyz="0.0"  izz="0.0" />
-    	</inertial>
     </link>
     <joint name="rear_right_hip_x" type="revolute">
@@ -489,17 +314,6 @@
         <parent link="body" />
         <child link="rear_right_hip" />
-        <dynamics damping="0.1" friction="0.1"/>
         <limit effort="1000" velocity="1000.00" lower="-0.78539816339744827899" upper="0.78539816339744827899" />
     </joint>
-    <transmission name="rear_right_hip_x_trans">
-        <type>transmission_interface/SimpleTransmission</type>
-        <joint name="rear_right_hip_x">
-            <hardwareInterface>EffortJointInterface</hardwareInterface>
-        </joint>
-        <actuator name="rear_right_hip_x">
-            <mechanicalReduction>50</mechanicalReduction>
-            <hardwareInterface>EffortJointInterface</hardwareInterface>
-        </actuator>
-    </transmission>
     <link name="rear_right_upper_leg">
         <visual>
@@ -513,8 +327,4 @@
             </geometry>
         </collision>
-        <inertial>
-            <mass value="1.5" />
-    	    <inertia  ixx="0.0" ixy="0.0"  ixz="0.0"  iyy="0.05"  iyz="0.0"  izz="0.0" />
-    	</inertial>
     </link>
     <joint name="rear_right_hip_y" type="revolute">
@@ -523,17 +333,6 @@
         <parent link="rear_right_hip" />
         <child link="rear_right_upper_leg" />
-        <dynamics damping="0.1" friction="0.1"/>
         <limit effort="1000" velocity="1000.00" lower="-0.89884456477707963539" upper="2.2951079663725435509" />
     </joint>
-    <transmission name="rear_right_hip_y_trans">
-        <type>transmission_interface/SimpleTransmission</type>
-        <joint name="rear_right_hip_y">
-            <hardwareInterface>EffortJointInterface</hardwareInterface>
-            </joint>
-        <actuator name="rear_right_hip_y">
-            <mechanicalReduction>50</mechanicalReduction>
-            <hardwareInterface>EffortJointInterface</hardwareInterface>
-        </actuator>
-    </transmission>
     <link name="rear_right_lower_leg">
         <visual>
@@ -547,8 +346,4 @@
             </geometry>
         </collision>
-        <inertial>
-            <mass value="1.0" />
-    	    <inertia  ixx="0.0" ixy="0.0"  ixz="0.0"  iyy="0.045"  iyz="0.0"  izz="0.0" />
-    	</inertial>
     </link>
     <joint name="rear_right_knee" type="revolute">
@@ -557,32 +352,6 @@
         <parent link="rear_right_upper_leg" />
         <child link="rear_right_lower_leg" />
-        <dynamics damping="0.1" friction="0.1"/>
         <limit effort="1000" velocity="1000.00" lower="-2.7929" upper="-0.257725" />
     </joint>
-    <gazebo reference="rear_right_lower_leg">
-        <sensor name="rear_right_lower_leg_contactsensor_sensor" type="contact">
-        <always_on>true</always_on>
-        <contact>
-            <collision>rear_right_lower_leg_fixed_joint_lump__rear_bump_sensor_collision</collision>
-        </contact>
-        <plugin filename="libgazebo_ros_bumper.so" name="rear_right_lower_leg_plugin">
-            <bumperTopicName>rear_right_lower_leg_contact</bumperTopicName>
-            <frameName>rear_right_lower_leg</frameName>
-        </plugin>
-        </sensor>
-    </gazebo>
-    <transmission name="rear_right_knee_trans">
-        <type>transmission_interface/SimpleTransmission</type>
-        <joint name="rear_right_knee">
-            <hardwareInterface>EffortJointInterface</hardwareInterface>
-            </joint>
-        <actuator name="rear_right_knee">
-            <mechanicalReduction>50</mechanicalReduction>
-            <hardwareInterface>EffortJointInterface</hardwareInterface>
-        </actuator>
-    </transmission>
-    <gazebo>
-    	<plugin name="gazebo_ros_control" filename="libgazebo_ros_control.so"/>
-    </gazebo>
     <!-- Spot Arm -->
     <xacro:if value="$(arg has_arm)">

Commit message: Added auto-detect for spot_proprietary_description

File: spot_description/urdf/spot.urdf.xacro (robot description, xacro)
@@ -11,5 +11,5 @@
     <xacro:arg name="kinematic_model" default="none"/>
     <xacro:arg name="use_proprietary_meshes" default="false" />
-    <xacro:arg name="proprietary_pkg" default="spot_propreity_description" />
+    <xacro:arg name="proprietary_pkg" default="spot_proprietary_description" />
     <xacro:arg name="proprietary_mesh_format" default="dae" />
     <xacro:property name="kinematic_model" value="$(arg kinematic_model)"/>

Commit message: make body_or joint continuous instead of revolute

File: spot_description/urdf/spot.urdf.xacro (robot description, xacro)
@@ -68,8 +68,8 @@
             <limit lower = "-10.0" upper = "10.0" velocity="0.1" effort="1e9"/>
         </joint>
-        <joint name="body_or" type="revolute">
+        <joint name="body_or" type="continuous">
             <parent link = "body_y"/>
             <child  link = "body_or"/>
-            <limit lower = "0" upper = "${2*pi}" velocity="0.1" effort="1e9"/>
+            <limit velocity="0.1" effort="1e9"/>
             <axis    xyz = "0 0 1"/>
         </joint>
