Commit message: enable prop mesh selection with visual primitive fallbacks

File: spot_description/urdf/accessories/rl_kit_velodyne_mount.xacro (robot description, xacro)
@@ -2,28 +2,48 @@
 <robot name="rl_kit_velodyne_mount" xmlns:xacro="http://www.ros.org/wiki/xacro">
     <xacro:include filename="$(find velodyne_description)/urdf/VLP-16.urdf.xacro"/>
+    <xacro:arg name="use_proprietary_meshes" default="false" />
     <link name="rl_kit_velodyne_mounting_plate">
+      <xacro:if value="$(arg use_proprietary_meshes)">
         <visual>
-            <geometry>
-                <mesh filename="package://spot_description/meshes/accessories/rl_kit_velodyne_mount.dae"/>
-            </geometry>
+          <geometry>
+            <mesh filename="package://spot_propriety_description/meshes/accessories/rl_kit_velodyne_mount.dae"/>
+          </geometry>
         </visual>
-        <collision>
-            <geometry>
-                <box size="0.19 0.18 0.013"/>
-            </geometry>
-        </collision>
+      </xacro:if>
+      <xacro:unless value="$(arg use_proprietary_meshes)">
+        <visual>
+          <geometry>
+          <box size="0.19 0.18 0.013"/>
+          </geometry>
+        </visual>
+      </xacro:unless>
+      <collision>
+        <geometry>
+          <box size="0.19 0.18 0.013"/>
+        </geometry>
+      </collision>
     </link>
     <link name="velodyne_cage">
+      <xacro:if value="$(arg use_proprietary_meshes)">
         <visual>
-            <geometry>
-                <mesh filename="package://spot_description/meshes/accessories/velodyne_cage.dae"/>
-            </geometry>
+          <geometry>
+            <mesh filename="package://spot_propriety_description/meshes/accessories/velodyne_cage.dae"/>
+          </geometry>
         </visual>
-        <collision>
-            <geometry>
-                <cylinder length="0.08" radius="0.08"/>
-            </geometry>
-            <origin xyz="0 0 0.04"/>
-        </collision>
+      </xacro:if>
+      <xacro:unless value="$(arg use_proprietary_meshes)">
+        <visual>
+          <geometry>
+          <cylinder length="0.08" radius="0.08"/>
+          </geometry>
+        <origin xyz="0 0 0.04"/>
+        </visual>
+      </xacro:unless>
+      <collision>
+        <geometry>
+          <cylinder length="0.08" radius="0.08"/>
+        </geometry>
+        <origin xyz="0 0 0.04"/>
+      </collision>
     </link>
     <joint name="velodyne_cage_link" type="fixed">

Commit message: update to use prop pkg name and extension args

File: spot_description/urdf/accessories/rl_kit_velodyne_mount.xacro (robot description, xacro)
@@ -3,9 +3,14 @@
     <xacro:include filename="$(find velodyne_description)/urdf/VLP-16.urdf.xacro"/>
     <xacro:arg name="use_proprietary_meshes" default="false" />
+    <xacro:arg name="proprietary_pkg" default="spot_propreity_description" />
+    <xacro:arg name="proprietary_format" default="dae" />
+    <!-- Determine mesh source -->
+  <xacro:property name="mesh_pkg" value="$(eval proprietary_pkg if use_proprietary_meshes else 'spot_description')"/>
+  <xacro:property name="mesh_ext" value="$(eval proprietary_format if use_proprietary_meshes else 'obj')" />
     <link name="rl_kit_velodyne_mounting_plate">
       <xacro:if value="$(arg use_proprietary_meshes)">
         <visual>
           <geometry>
-            <mesh filename="package://spot_propriety_description/meshes/accessories/rl_kit_velodyne_mount.dae"/>
+            <mesh filename="package://${mesh_pkg}/meshes/accessories/rl_kit_velodyne_mount.${mesh_ext}"/>
           </geometry>
         </visual>
@@ -28,5 +33,5 @@
         <visual>
           <geometry>
-            <mesh filename="package://spot_propriety_description/meshes/accessories/velodyne_cage.dae"/>
+            <mesh filename="package://${mesh_pkg}/meshes/accessories/velodyne_cage.${mesh_ext}"/>
           </geometry>
         </visual>
