Commit message: Added GXP to rl_kit accessory

File: spot_description/urdf/accessories/rl_kit.xacro (robot description, xacro)
@@ -48,4 +48,16 @@
             <origin xyz = "-0.078 0.0 0.0"/>
         </joint>
+        <link name="rl_kit_gxp_interface">
+            <visual>
+                <geometry>
+                    <mesh filename="package://spot_description/meshes/accessories/gxp.dae"/>
+                </geometry>
+            </visual>
+        </link>
+        <joint name="rl_kit_gxp_joint" type="fixed">
+            <parent link = "rl_kit_reference_frame"/>
+            <child  link = "rl_kit_gxp_interface"/>
+            <origin xyz = "0.13 0.0 -0.056"/>
+        </joint>
     </xacro:macro>
 </robot>

Commit message: Updated URDF with visual models for rl kit

File: spot_description/urdf/accessories/rl_kit.xacro (robot description, xacro)
@@ -11,9 +11,7 @@
             <visual>
                 <geometry>
-                    <box size="${2*0.076} ${2*0.103} ${2*0.033}"/>
+                    <mesh filename="package://spot_description/meshes/accessories/rl_kit_wire_housing_box.dae"/>
                 </geometry>
-                <material name="black_color">
-                    <color rgba="0.1 0.1 0.1 1"/>
-                </material>
+                <origin xyz="-0.025 0 -0.03" rpy="0 0 ${pi/2}"/>
             </visual>
             <collision>
@@ -29,11 +27,15 @@
         </joint>
         <link name="rl_kit_jetson_housing_box">
-            <visual>
+            <visual name="housing">
                 <geometry>
-                    <box size="${2*0.078} ${2*0.103} ${2*0.056}"/>
+                    <mesh filename="package://spot_description/meshes/accessories/rl_kit_jetson_housing_box.dae"/>
                 </geometry>
-                <material name="black_color">
-                    <color rgba="0.1 0.1 0.1 1"/>
-                </material>
+                <origin xyz="0.02 0 -0.056"/>
+            </visual>
+            <visual name="jetson">
+                <geometry>
+                    <mesh filename="package://spot_description/meshes/accessories/jetson_orin_dev_kit.dae"/>
+                </geometry>
+                <origin xyz="0 0 -0.056" rpy="0 0 ${pi/2}"/>
             </visual>
             <collision>

File: spot_description/urdf/accessories/rl_kit_velodyne_mount.xacro (robot description, xacro)
@@ -38,5 +38,5 @@
         <parent link = "rl_kit_jetson_housing_box"/>
         <child  link = "rl_kit_velodyne_mounting_plate"/>
-        <origin xyz="-0.045 0.0 0.056"/>
+        <origin xyz="-0.03 0.0 0.06"/>
     </joint>
 </robot>

Commit message: add visual fallback for gpx and enable propriety mesh selection for rl kit

File: spot_description/urdf/accessories/rl_kit.xacro (robot description, xacro)
@@ -2,4 +2,5 @@
 <robot name="rl_kit" xmlns:xacro="http://www.ros.org/wiki/xacro">
     <xacro:macro name="rl_kit">
+    <xacro:arg name="use_proprietary_meshes" default="false" />
         <link name="rl_kit_reference_frame"/>
         <joint name="rl_kit_base_mount_to_body"  type="fixed">
@@ -9,10 +10,20 @@
         </joint>
         <link name="rl_kit_wire_housing_box">
+	<xacro:if value="$(arg use_proprietary_meshes)">
             <visual>
                 <geometry>
-                    <mesh filename="package://spot_description/meshes/accessories/rl_kit_wire_housing_box.dae"/>
+                    <mesh filename="package://spot_propriety_description/meshes/accessories/rl_kit_wire_housing_box.dae"/>
                 </geometry>
                 <origin xyz="-0.025 0 -0.03" rpy="0 0 ${pi/2}"/>
             </visual>
+        </xacro:if>
+	<xacro:unless value="$(arg use_proprietary_meshes)">
+            <visual>
+                <geometry>
+                    <box size="${2*0.076} ${2*0.103} ${2*0.033}"/>
+                </geometry>
+                <origin xyz="-0.025 0 -0.03" rpy="0 0 ${pi/2}"/>
+            </visual>
+        </xacro:unless>
             <collision>
                 <geometry>
@@ -27,7 +38,8 @@
         </joint>
         <link name="rl_kit_jetson_housing_box">
+	<xacro:if value="$(arg use_proprietary_meshes)">
             <visual name="housing">
                 <geometry>
-                    <mesh filename="package://spot_description/meshes/accessories/rl_kit_jetson_housing_box.dae"/>
+                    <mesh filename="package://spot_propriety_description/meshes/accessories/rl_kit_jetson_housing_box.dae"/>
                 </geometry>
                 <origin xyz="0.02 0 -0.056"/>
@@ -35,8 +47,17 @@
             <visual name="jetson">
                 <geometry>
-                    <mesh filename="package://spot_description/meshes/accessories/jetson_orin_dev_kit.dae"/>
+                    <mesh filename="package://spot_propriety_description/meshes/accessories/jetson_orin_dev_kit.dae"/>
                 </geometry>
                 <origin xyz="0 0 -0.056" rpy="0 0 ${pi/2}"/>
             </visual>
+        </xacro:if>
+	<xacro:unless value="$(arg use_proprietary_meshes)">
+          <visual name="housing_and_jetson">
+            <geometry>
+              <box size="${2*0.078} ${2*0.103} ${2*0.056}"/>
+            </geometry>
+            <origin xyz="0.02 0 -0.056"/>
+          </visual>
+        </xacro:unless>
             <collision>
                 <geometry>
@@ -51,9 +72,18 @@
         </joint>
         <link name="rl_kit_gxp_interface">
+          <xacro:if value="$(arg use_proprietary_meshes)">
             <visual>
-                <geometry>
-                    <mesh filename="package://spot_description/meshes/accessories/gxp.dae"/>
-                </geometry>
+              <geometry>
+                <mesh filename="package://spot_propriety_description/meshes/accessories/gxp.dae"/>
+              </geometry>
             </visual>
+          </xacro:if>
+          <xacro:unless value="$(arg use_proprietary_meshes)">
+            <visual>
+              <geometry>
+                <box size="0.1905 0.04445 0.0635"/>
+              </geometry>
+            </visual>
+          </xacro:unless>
         </link>
         <joint name="rl_kit_gxp_joint" type="fixed">

Commit message: add collision geometry for gpx interface

File: spot_description/urdf/accessories/rl_kit.xacro (robot description, xacro)
@@ -84,6 +84,12 @@
                 <box size="0.1905 0.04445 0.0635"/>
               </geometry>
+	      <origin xyz="0 0 0"/>
             </visual>
           </xacro:unless>
+	  <collision>
+            <geometry>
+              <box size="0.1905 0.04445 0.0635"/>
+            </geometry>
+          </collision>
         </link>
         <joint name="rl_kit_gxp_joint" type="fixed">

Commit message: fix wrong dims and misalignment of rl-kit visual geometries

File: spot_description/urdf/accessories/rl_kit.xacro (robot description, xacro)
@@ -21,12 +21,12 @@
             <visual>
                 <geometry>
-                    <box size="${2*0.076} ${2*0.103} ${2*0.033}"/>
+                    <box size="${2*0.103} 0.130 0.0635"/>
                 </geometry>
-                <origin xyz="-0.025 0 -0.03" rpy="0 0 ${pi/2}"/>
+                <origin xyz="0.0 0.0 0.0" rpy="0 0 ${pi/2}"/>
             </visual>
         </xacro:unless>
             <collision>
                 <geometry>
-                    <box size="${2*0.076} ${2*0.103} ${2*0.033}"/>
+                    <box size="${2*0.103} 0.130 0.0635}"/>
                 </geometry>
             </collision>
@@ -57,5 +57,5 @@
               <box size="${2*0.078} ${2*0.103} ${2*0.056}"/>
             </geometry>
-            <origin xyz="0.02 0 -0.056"/>
+            <origin xyz="0.01 0.0 0.0"/>
           </visual>
         </xacro:unless>
@@ -64,4 +64,5 @@
                     <box size="${2*0.078} ${2*0.103} ${2*0.056}"/>
                 </geometry>
+            <origin xyz="0.01 0.0 0.0"/>
             </collision>
         </link>
@@ -82,13 +83,14 @@
             <visual>
               <geometry>
-                <box size="0.1905 0.04445 0.0635"/>
+                <box size=" 0.04445 0.1905 0.0635"/>
               </geometry>
-	      <origin xyz="0 0 0"/>
+	      <origin xyz="${0.0445/2 + 0.01} 0 ${0.0635/2}"/>
             </visual>
           </xacro:unless>
 	  <collision>
             <geometry>
-              <box size="0.1905 0.04445 0.0635"/>
+              <box size=" 0.04445 0.1905 0.0635"/>
             </geometry>
+	      <origin xyz="${0.0445/2 + 0.01} 0 ${0.0635/2}"/>
           </collision>
         </link>

Commit message: fix typo in wire housing box collision geometry

File: spot_description/urdf/accessories/rl_kit.xacro (robot description, xacro)
@@ -28,6 +28,7 @@
             <collision>
                 <geometry>
-                    <box size="${2*0.103} 0.130 0.0635}"/>
+                    <box size="${2*0.103} 0.130 0.0635"/>
                 </geometry>
+                <origin xyz="0.0 0.0 0.0" rpy="0 0 ${pi/2}"/>
             </collision>
         </link>

Commit message: rename proprietary_format arg to proprietary_mesh_format

File: spot_description/urdf/accessories/rl_kit.xacro (robot description, xacro)
@@ -3,4 +3,9 @@
     <xacro:macro name="rl_kit">
     <xacro:arg name="use_proprietary_meshes" default="false" />
+    <xacro:arg name="proprietary_pkg" default="spot_proprietary_description" />
+    <xacro:arg name="proprietary_mesh_format" default="dae" />
+    <!-- Determine mesh source -->
+  <xacro:property name="mesh_pkg" value="$(eval proprietary_pkg if use_proprietary_meshes else 'spot_description')"/>
+  <xacro:property name="mesh_ext" value="$(eval proprietary_mesh_format if use_proprietary_meshes else 'obj')" />
         <link name="rl_kit_reference_frame"/>
         <joint name="rl_kit_base_mount_to_body"  type="fixed">
@@ -13,5 +18,5 @@
             <visual>
                 <geometry>
-                    <mesh filename="package://spot_propriety_description/meshes/accessories/rl_kit_wire_housing_box.dae"/>
+                    <mesh filename="package://${mesh_pkg}/meshes/accessories/rl_kit_wire_housing_box.${mesh_ext}"/>
                 </geometry>
                 <origin xyz="-0.025 0 -0.03" rpy="0 0 ${pi/2}"/>
@@ -42,5 +47,5 @@
             <visual name="housing">
                 <geometry>
-                    <mesh filename="package://spot_propriety_description/meshes/accessories/rl_kit_jetson_housing_box.dae"/>
+                    <mesh filename="package://${mesh_pkg}/meshes/accessories/rl_kit_jetson_housing_box.${mesh_ext}"/>
                 </geometry>
                 <origin xyz="0.02 0 -0.056"/>
@@ -48,5 +53,5 @@
             <visual name="jetson">
                 <geometry>
-                    <mesh filename="package://spot_propriety_description/meshes/accessories/jetson_orin_dev_kit.dae"/>
+                    <mesh filename="package://${mesh_pkg}/meshes/accessories/jetson_orin_dev_kit.${mesh_ext}"/>
                 </geometry>
                 <origin xyz="0 0 -0.056" rpy="0 0 ${pi/2}"/>
@@ -77,5 +82,5 @@
             <visual>
               <geometry>
-                <mesh filename="package://spot_propriety_description/meshes/accessories/gxp.dae"/>
+                <mesh filename="package://${mesh_pkg}/meshes/accessories/gxp.${mesh_ext}"/>
               </geometry>
             </visual>

File: spot_description/urdf/accessories/rl_kit_velodyne_mount.xacro (robot description, xacro)
@@ -3,9 +3,9 @@
     <xacro:include filename="$(find velodyne_description)/urdf/VLP-16.urdf.xacro"/>
     <xacro:arg name="use_proprietary_meshes" default="false" />
-    <xacro:arg name="proprietary_pkg" default="spot_propreity_description" />
-    <xacro:arg name="proprietary_format" default="dae" />
+    <xacro:arg name="proprietary_pkg" default="spot_proprietary_description" />
+    <xacro:arg name="proprietary_mesh_format" default="dae" />
     <!-- Determine mesh source -->
   <xacro:property name="mesh_pkg" value="$(eval proprietary_pkg if use_proprietary_meshes else 'spot_description')"/>
-  <xacro:property name="mesh_ext" value="$(eval proprietary_format if use_proprietary_meshes else 'obj')" />
+  <xacro:property name="mesh_ext" value="$(eval proprietary_mesh_format if use_proprietary_meshes else 'obj')" />
     <link name="rl_kit_velodyne_mounting_plate">
       <xacro:if value="$(arg use_proprietary_meshes)">

File: spot_description/urdf/arm/spot_arm.urdf.xacro (robot description, xacro)
@@ -4,9 +4,9 @@
     <xacro:arg name="has_realsense" default="False" />
     <xacro:arg name="use_proprietary_meshes" default="false" />
-    <xacro:arg name="proprietary_pkg" default="spot_propreity_description" />
-    <xacro:arg name="proprietary_format" default="dae" />
+    <xacro:arg name="proprietary_pkg" default="spot_proprietary_description" />
+    <xacro:arg name="proprietary_mesh_format" default="dae" />
     <!-- Determine mesh source -->
   <xacro:property name="mesh_pkg" value="$(eval proprietary_pkg if use_proprietary_meshes else 'spot_description')"/>
-  <xacro:property name="mesh_ext" value="$(eval proprietary_format if use_proprietary_meshes else 'obj')" />
+  <xacro:property name="mesh_ext" value="$(eval proprietary_mesh_format if use_proprietary_meshes else 'obj')" />
     <link name="${name}_base_link">
         <visual>

File: spot_description/urdf/spot.urdf.xacro (robot description, xacro)
@@ -12,9 +12,9 @@
     <xacro:arg name="use_proprietary_meshes" default="false" />
     <xacro:arg name="proprietary_pkg" default="spot_propreity_description" />
-    <xacro:arg name="proprietary_format" default="dae" />
+    <xacro:arg name="proprietary_mesh_format" default="dae" />
     <xacro:property name="kinematic_model" value="$(arg kinematic_model)"/>
     <!-- Determine mesh source -->
     <xacro:property name="mesh_pkg" value="$(eval proprietary_pkg if use_proprietary_meshes else 'spot_description')"/>
-    <xacro:property name="mesh_ext" value="$(eval proprietary_format if use_proprietary_meshes else 'obj')" />
+    <xacro:property name="mesh_ext" value="$(eval proprietary_mesh_format if use_proprietary_meshes else 'obj')" />
     <xacro:unless value="${kinematic_model == 'none'}">
         <link name="base_footprint"/>

Commit message: add arm0_base_link visual and make visual color black

File: spot_description/urdf/accessories/rl_kit.xacro (robot description, xacro)
@@ -29,4 +29,7 @@
                 </geometry>
                 <origin xyz="0.0 0.0 0.0" rpy="0 0 ${pi/2}"/>
+                <material name="black">
+                  <color rgba="0 0 0 1"/>
+                </material>
             </visual>
         </xacro:unless>
@@ -64,4 +67,7 @@
             </geometry>
             <origin xyz="0.01 0.0 0.0"/>
+            <material name="black">
+              <color rgba="0 0 0 1"/>
+            </material>
           </visual>
         </xacro:unless>
@@ -92,4 +98,7 @@
               </geometry>
 	      <origin xyz="${0.0445/2 + 0.01} 0 ${0.0635/2}"/>
+              <material name="black">
+                <color rgba="0 0 0 1"/>
+              </material>
             </visual>
           </xacro:unless>

File: spot_description/urdf/arm/spot_arm.urdf.xacro (robot description, xacro)
@@ -10,4 +10,5 @@
   <xacro:property name="mesh_ext" value="$(eval proprietary_mesh_format if use_proprietary_meshes else 'obj')" />
     <link name="${name}_base_link">
+	<xacro:if value="$(arg use_proprietary_meshes)">
         <visual>
             <geometry>
@@ -17,4 +18,16 @@
             <origin xyz="-0.001 0.0002 -0.116" rpy="0 0.03 0"/>
         </visual>
+        </xacro:if>
+	<xacro:unless value="$(arg use_proprietary_meshes)">
+        <visual>
+            <geometry>
+                <cylinder radius="0.08" length="0.05"/>
+            </geometry>
+            <origin xyz="-0.02 0 -0.08"/>
+            <material name="black">
+              <color rgba="0 0 0 1"/>
+            </material>
+        </visual>
+        </xacro:unless>
         <collision>
             <geometry>

Commit message: adjust rl_kit visual and collision dims to match meshes

File: spot_description/urdf/accessories/rl_kit.xacro (robot description, xacro)
@@ -26,7 +26,7 @@
             <visual>
                 <geometry>
-                    <box size="${2*0.103} 0.130 0.0635"/>
+                    <box size="${2*0.103} 0.09 0.0635"/>
                 </geometry>
-                <origin xyz="0.0 0.0 0.0" rpy="0 0 ${pi/2}"/>
+                <origin xyz="-0.025 0.0 0.0" rpy="0 0 ${pi/2}"/>
                 <material name="black">
                   <color rgba="0 0 0 1"/>
@@ -36,7 +36,7 @@
             <collision>
                 <geometry>
-                    <box size="${2*0.103} 0.130 0.0635"/>
+                    <box size="${2*0.103} 0.09 0.0635"/>
                 </geometry>
-                <origin xyz="0.0 0.0 0.0" rpy="0 0 ${pi/2}"/>
+                <origin xyz="-0.025 0.0 0.0" rpy="0 0 ${pi/2}"/>
             </collision>
         </link>
@@ -64,5 +64,5 @@
           <visual name="housing_and_jetson">
             <geometry>
-              <box size="${2*0.078} ${2*0.103} ${2*0.056}"/>
+              <box size="${2*0.068} ${2*0.1} ${2*0.056}"/>
             </geometry>
             <origin xyz="0.01 0.0 0.0"/>
@@ -74,5 +74,5 @@
             <collision>
                 <geometry>
-                    <box size="${2*0.078} ${2*0.103} ${2*0.056}"/>
+                    <box size="${2*0.068} ${2*0.1} ${2*0.056}"/>
                 </geometry>
             <origin xyz="0.01 0.0 0.0"/>
@@ -97,5 +97,5 @@
                 <box size=" 0.04445 0.1905 0.0635"/>
               </geometry>
-	      <origin xyz="${0.0445/2 + 0.01} 0 ${0.0635/2}"/>
+	      <origin xyz="${0.0445/2 - 0.02} 0 ${0.0635/2}"/>
               <material name="black">
                 <color rgba="0 0 0 1"/>
@@ -107,5 +107,5 @@
               <box size=" 0.04445 0.1905 0.0635"/>
             </geometry>
-	      <origin xyz="${0.0445/2 + 0.01} 0 ${0.0635/2}"/>
+	      <origin xyz="${0.0445/2 - 0.02} 0 ${0.0635/2}"/>
           </collision>
         </link>
